File: design/mackerel_08/mackerel_08.kicad_sch (KiCad schematic)
At the start: 24 parts, among them J1 Conn_02x20_Odd_Even, J2 Conn_02x10_Odd_Even, U1 MC68008FN, U2 GAL16V8, U3 74HC595, U4 GAL16V8, U5 NE555P, X1 CXO_DIP14

Commit message: Double DUART board with independent interrupt channels
Connections:
- net BOOT: now also U4.2 (I2); no longer U4.1 (I1/CLK)
- net ~{AS}: now also U4.1 (I1/CLK); no longer U4.2 (I2)
Other:
- note added: "TODO: Making a priority encoder on a GAL is really ugly Find a better way"
- note removed: "TODO: Move the IACK decoding to the peripheral boards"
Changed lines of the file:
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@@
-    (stroke (width 0) (type default) (color 0 0 0 0))
-  )
-  (wire (pts (xy 127.635 94.615) (xy 133.35 94.615))
     (stroke (width 0) (type default) (color 0 0 0 0))
   )
@@
     (stroke (width 0) (type default) (color 0 0 0 0))
   )
+  (wire (pts (xy 133.35 97.155) (xy 127.635 97.155))
+    (stroke (width 0) (type default) (color 0 0 0 0))
+  )
   (wire (pts (xy 84.455 74.93) (xy 89.535 74.93))
     (stroke (width 0) (type default) (color 0 0 0 0))
@@
     (stroke (width 0) (type default) (color 0 0 0 0))
   )
-  (wire (pts (xy 127.635 94.615) (xy 127.635 80.01))
+  (wire (pts (xy 127.635 80.01) (xy 127.635 97.155))
     (stroke (width 0) (type default) (color 0 0 0 0))
   )
@@
     (stroke (width 0) (type default) (color 0 0 0 0))
   )
+  (text "TODO: Making a priority encoder on a GAL is really ugly\nFind a better way"
+    (at 85.725 193.04 0)
+    (effects (font (size 1.27 1.27)) (justify left bottom))
+  )
   (text "Address Decoder" (at 159.385 119.38 0)
     (effects (font (size 1.27 1.27)) (justify left bottom))
@@
     (effects (font (size 1.27 1.27)) (justify left bottom))
   )
-  (text "TODO: Move the IACK decoding to the peripheral boards\n"
-    (at 132.08 143.51 0)
-    (effects (font (size 1.27 1.27)) (justify left bottom))
-  )
   (label "A5" (at 84.455 46.99 0)
     (effects (font (size 1.27 1.27)) (justify left bottom))
@@
     (effects (font (size 1.27 1.27)) (justify right bottom))
   )
-  (label "~{IACK1}" (at 167.64 147.955 0)
-    (effects (font (size 1.27 1.27)) (justify left bottom))
-  )
   (label "A0" (at 222.25 74.295 180)
     (effects (font (size 1.27 1.27)) (justify right bottom))
@@
     (effects (font (size 1.27 1.27)) (justify left bottom))
   )
-  (label "~{IACK4}" (at 167.64 155.575 0)
-    (effects (font (size 1.27 1.27)) (justify left bottom))
-  )
   (label "A21" (at 84.455 87.63 0)
     (effects (font (size 1.27 1.27)) (justify left bottom))
@@
     (effects (font (size 1.27 1.27)) (justify right bottom))
   )
-  (label "~{IACK3}" (at 167.64 153.035 0)
-    (effects (font (size 1.27 1.27)) (justify left bottom))
-  )
   (label "A8" (at 84.455 54.61 0)
     (effects (font (size 1.27 1.27)) (justify left bottom))
@@
     (effects (font (size 1.27 1.27)) (justify right bottom))
   )
-  (label "~{IACK5}" (at 167.64 158.115 0)
-    (effects (font (size 1.27 1.27)) (justify left bottom))
-  )
   (label "D7" (at 84.455 110.49 0)
     (effects (font (size 1.27 1.27)) (justify left bottom))
@@
     (effects (font (size 1.27 1.27)) (justify right bottom))
   )
-  (label "A3" (at 161.925 153.035 180)
-    (effects (font (size 1.27 1.27)) (justify right bottom))
-  )
   (label "A1" (at 234.95 74.295 0)
     (effects (font (size 1.27 1.27)) (justify left bottom))
@@
     (effects (font (size 1.27 1.27)) (justify left bottom))
   )
-  (label "~{AS}" (at 133.35 97.155 180)
+  (label "~{AS}" (at 133.35 94.615 180)
     (effects (font (size 1.27 1.27)) (justify right bottom))
   )
@@
     (effects (font (size 1.27 1.27)) (justify left bottom))
   )
-  (label "A1" (at 161.925 147.955 180)
-    (effects (font (size 1.27 1.27)) (justify right bottom))
-  )
   (label "A22" (at 222.25 123.825 180)
     (effects (font (size 1.27 1.27)) (justify right bottom))
@@
     (effects (font (size 1.27 1.27)) (justify right bottom))
   )
-  (label "A2" (at 161.925 150.495 180)
-    (effects (font (size 1.27 1.27)) (justify right bottom))
-  )
   (label "~{IRQ7}" (at 234.95 133.985 0)
     (effects (font (size 1.27 1.27)) (justify left bottom))
   )
-  (label "IACK" (at 161.29 157.48 180)
-    (effects (font (size 1.27 1.27)) (justify right bottom))
-  )
   (label "RST_IN" (at 222.25 136.525 180)
     (effects (font (size 1.27 1.27)) (justify right bottom))
@@
     (effects (font (size 1.27 1.27)) (justify right bottom))
   )
-  (label "~{IACK2}" (at 167.64 150.495 0)
-    (effects (font (size 1.27 1.27)) (justify left bottom))
-  )
   (label "D7" (at 234.95 71.755 0)
     (effects (font (size 1.27 1.27)) (justify left bottom))
   )
-  (label "~{IACK7}" (at 167.64 163.195 0)
-    (effects (font (size 1.27 1.27)) (justify left bottom))
-  )
   (label "A16" (at 222.25 116.205 180)
     (effects (font (size 1.27 1.27)) (justify right bottom))
@@
     (effects (font (size 1.27 1.27)) (justify left bottom))
   )
-  (label "BOOT" (at 133.35 94.615 180)
+  (label "BOOT" (at 133.35 97.155 180)
     (effects (font (size 1.27 1.27)) (justify right bottom))
   )
@@
     (effects (font (size 1.27 1.27)) (justify right bottom))
   )
-  (label "~{IACK6}" (at 167.64 160.655 0)
-    (effects (font (size 1.27 1.27)) (justify left bottom))
-  )
   (label "~{IRQ1}" (at 234.95 126.365 0)
