File: design/mackerel-08-v1/mackerel-08-v1.kicad_pcb (KiCad board)
At the start: 2 copper layers, 100 x 100 mm, 13 parts, among them U1 MC68008, U2 7410, U3 74HC595, U4 SST39SF040, X1 CXO_DIP14

Commit message: simplifying schematic
Parts:
- added C1: C_Polarized, Capacitor_THT:CP_Radial_D5.0mm_P2.50mm, F.Cu at (-156.7, 197.6)
- added C2: C_Polarized, Capacitor_THT:CP_Radial_D8.0mm_P3.80mm, F.Cu at (62.7, 30.5)
- added D1: LED, LED_THT:LED_D5.0mm, F.Cu at (-188.5, 183.4)
- added D2: LED, LED_THT:LED_D5.0mm, F.Cu at (-186.7, 211.6)
- added J2: DC_Jack, Connector_BarrelJack:BarrelJack_GCT_DCJ200-10-A_Horizontal, F.Cu at (51.8, 33.6)
- added J3: Conn_01x06, Connector_PinHeader_2.54mm:PinHeader_1x06_P2.54mm_Vertical, F.Cu at (-129.7, 111.9)
- added J4: Conn_01x06, Connector_PinHeader_2.54mm:PinHeader_1x06_P2.54mm_Vertical, F.Cu at (-134.3, 111.9)
- added J5: Conn_02x20_Odd_Even, Connector_PinHeader_2.54mm:PinHeader_2x20_P2.54mm_Vertical, F.Cu at (75.9, 172.2)
- added R10: R, Resistor_SMD:R_1206_3216Metric_Pad1.30x1.75mm_HandSolder, F.Cu at (-179.3, 170.7)
- added R11: R, Resistor_SMD:R_1206_3216Metric_Pad1.30x1.75mm_HandSolder, F.Cu at (-185.7, 204.7)
- added R12: R, Resistor_SMD:R_1206_3216Metric_Pad1.30x1.75mm_HandSolder, F.Cu at (-144.0, 196.1)
- added R13: R, Resistor_SMD:R_1206_3216Metric_Pad1.30x1.75mm_HandSolder, F.Cu at (-132.1, 178.1)
- added R9: R, Resistor_SMD:R_1206_3216Metric_Pad1.30x1.75mm_HandSolder, F.Cu at (-11.9, 71.1)
- added SW1: SW_Push, Button_Switch_THT:SW_PUSH_6mm_H5mm, F.Cu at (-152.1, 182.2)
- added U10: 74HC595, Package_DIP:DIP-16_W7.62mm_Socket_LongPads, F.Cu at (-115.1, 76.2)
- added U11: 74HC10, Package_DIP:DIP-14_W7.62mm_Socket_LongPads, F.Cu at (89.2, 141.7)
- added U12: GAL16V8, Package_DIP:DIP-20_W7.62mm_Socket_LongPads, F.Cu at (-99.5, 58.3)
- added U13: GAL16V8, Package_DIP:DIP-20_W7.62mm_Socket_LongPads, F.Cu at (92.5, 127.2)
- added U14: NE555P, Package_DIP:DIP-8_W7.62mm, F.Cu at (-167.1, 178.8)
- added U5: AS7C4096A, Package_SO:SOJ-36_10.16x23.49mm_P1.27mm, F.Cu at (108.0, 97.3)
- added U6: AS7C4096A, Package_SO:SOJ-36_10.16x23.49mm_P1.27mm, F.Cu at (124.0, 97.3)
- added U7: AS7C4096A, Package_SO:SOJ-36_10.16x23.49mm_P1.27mm, F.Cu at (140.0, 97.3)
- added U8: SST39SF040, Package_DIP:DIP-32_W15.24mm_Socket_LongPads, F.Cu at (119.9, 154.2)
- added U9: XR68C681, Package_LCC:PLCC-44_THT-Socket, F.Cu at (126.7, 62.5)
- added X2: CXO_DIP8, Oscillator:Oscillator_DIP-8, F.Cu at (-48.6, 67.1)
- R1, R2, R3, R4, R5, R6, R7, R8: footprint Resistor_THT:R_Axial_DIN0207_L6.3mm_D2.5mm_P7.62mm_Horizontal -> Resistor_SMD:R_1206_3216Metric_Pad1.30x1.75mm_HandSolder
- U2: value 7410 -> AS7C4096A; footprint Package_DIP:DIP-14_W7.62mm -> Package_SO:SOJ-36_10.16x23.49mm_P1.27mm
- U3: value 74HC595 -> AS7C4096A; footprint Package_DIP:DIP-16_W7.62mm -> Package_SO:SOJ-36_10.16x23.49mm_P1.27mm
- U4: value SST39SF040 -> AS7C4096A; footprint Socket:DIP_Socket-32_W11.9_W12.7_W15.24_W17.78_W18.5_3M_232-1285-00-0602J -> Package_SO:SOJ-36_10.16x23.49mm_P1.27mm
- X1: value CXO_DIP14 -> CXO_DIP8; footprint Oscillator:Oscillator_DIP-14 -> Oscillator:Oscillator_DIP-8
- moved R2 295.8 mm to (-133.7, 128.5)
- moved R7 268.2 mm to (-107.9, 126.7)
- moved X1 224.5 mm to (-85.6, 117.2)
- moved R1 219.1 mm to (-113.8, 126.7)
- moved R3 209.4 mm to (-97.7, 102.0)
- moved R8 178.2 mm to (-28.7, 65.3)
- moved R5 164.2 mm to (-61.6, 105.5)
- moved R6 157.8 mm to (-21.2, 57.8)
- moved R4 130.9 mm to (-22.1, 76.2)
- moved U1 114.7 mm to (69.1, 146.8), turned to -90 degrees
- moved U4 93.4 mm to (92.0, 97.3)
- moved U2 79.7 mm to (60.0, 97.3)
- moved U3 71.6 mm to (76.0, 97.3), turned to 0 degrees
Connections:
- R1 pad 1: +5V -> GND
- R1 pad 2: Net-(R1-Pad2) -> /DTACK
- R2 pad 1: +5V -> /IACK_DUART
- R2 pad 2: Net-(R2-Pad2) -> +5V
- R3 pad 2: Net-(R3-Pad2) -> /IPL0
- R4 pad 2: Net-(R4-Pad2) -> /IPL1
- R5 pad 1: Net-(R5-Pad1) -> +5V
- R5 pad 2: GND -> /IPL2
- R6 pad 1: +5V -> VPA
- R6 pad 2: /IPL0 -> +5V
- R7 pad 1: +5V -> Net-(R7-Pad1)
- R7 pad 2: /IPL1 -> +5V
- R8 pad 1: +5V -> Net-(R8-Pad1)
- R8 pad 2: /IPL2 -> +5V
- U1 pad 1: unconnected-(U1-Pad1) -> A2
- U1 pad 10: unconnected-(U1-Pad10) -> A11
- U1 pad 11: unconnected-(U1-Pad11) -> A12
- U1 pad 12: unconnected-(U1-Pad12) -> A13
- U1 pad 13: unconnected-(U1-Pad13) -> A21
- U1 pad 14: unconnected-(U1-Pad14) -> A14
- U1 pad 16: unconnected-(U1-Pad16) -> A15
- U1 pad 18: unconnected-(U1-Pad18) -> A16
- U1 pad 19: unconnected-(U1-Pad19) -> A17
- U1 pad 2: unconnected-(U1-Pad2) -> A3
- U1 pad 20: unconnected-(U1-Pad20) -> A18
- U1 pad 21: unconnected-(U1-Pad21) -> A19
- U1 pad 22: unconnected-(U1-Pad22) -> A20
- U1 pad 23: unconnected-(U1-Pad23) -> D7
- U1 pad 24: unconnected-(U1-Pad24) -> D6
- U1 pad 25: unconnected-(U1-Pad25) -> D5
- U1 pad 26: unconnected-(U1-Pad26) -> D4
- U1 pad 27: unconnected-(U1-Pad27) -> D3
- U1 pad 28: unconnected-(U1-Pad28) -> D2
- U1 pad 29: unconnected-(U1-Pad29) -> D1
- U1 pad 3: unconnected-(U1-Pad3) -> A4
- U1 pad 30: unconnected-(U1-Pad30) -> D0
- U1 pad 31: unconnected-(U1-Pad31) -> /AS
- U1 pad 32: unconnected-(U1-Pad32) -> /DS
- U1 pad 33: unconnected-(U1-Pad33) -> /RW
- U1 pad 34: Net-(R5-Pad1) -> /DTACK
- U1 pad 36: Net-(R3-Pad2) -> Net-(R8-Pad1)
- U1 pad 37: Net-(R4-Pad2) -> Net-(R7-Pad1)
- U1 pad 38: CPU_CLK -> Net-(U1-Pad38)
- U1 pad 4: unconnected-(U1-Pad4) -> A5
- U1 pad 42: unconnected-(U1-Pad42) -> E
- U1 pad 43: Net-(R1-Pad2) -> VPA
- U1 pad 44: Net-(R2-Pad2) -> Net-(R9-Pad1)
- U1 pad 48: Net-(U1-Pad48) -> FC2
- U1 pad 49: Net-(U1-Pad49) -> FC1
- U1 pad 5: unconnected-(U1-Pad5) -> A6
- U1 pad 50: Net-(U1-Pad50) -> FC0
- U1 pad 51: unconnected-(U1-Pad51) -> A0
- U1 pad 52: unconnected-(U1-Pad52) -> A1
- U1 pad 6: unconnected-(U1-Pad6) -> A7
- U1 pad 7: unconnected-(U1-Pad7) -> A8
- U1 pad 8: unconnected-(U1-Pad8) -> A9
- U1 pad 9: unconnected-(U1-Pad9) -> A10
- U2 pad 1: Net-(U1-Pad48) -> A0
- U2 pad 11: GND -> D2
- U2 pad 12: /IACK -> D3
- U2 pad 13: Net-(U1-Pad50) -> /RW
- U2 pad 14: +5V -> A5
- U2 pad 2: Net-(U1-Pad49) -> A1
- U2 pad 3: GND -> A2
- U2 pad 4: GND -> A3
- U2 pad 5: GND -> A4
- U2 pad 6: unconnected-(U2-Pad6) -> RAM_EN0
- U2 pad 7: GND -> D0
- U2 pad 8: unconnected-(U2-Pad8) -> D1
- U2 pad 9: GND -> +5V
- U3 pad 1: unconnected-(U3-Pad1) -> A0
- U3 pad 10: unconnected-(U3-Pad10) -> GND
- U3 pad 11: unconnected-(U3-Pad11) -> D2
- U3 pad 12: unconnected-(U3-Pad12) -> D3
- U3 pad 13: unconnected-(U3-Pad13) -> /RW
- U3 pad 14: unconnected-(U3-Pad14) -> A5
- U3 pad 15: unconnected-(U3-Pad15) -> A6
- U3 pad 16: +5V -> A7
- U3 pad 2: unconnected-(U3-Pad2) -> A1
- U3 pad 3: unconnected-(U3-Pad3) -> A2
- U3 pad 4: unconnected-(U3-Pad4) -> A3
- U3 pad 5: unconnected-(U3-Pad5) -> A4
- U3 pad 6: unconnected-(U3-Pad6) -> RAM_EN1
- U3 pad 7: unconnected-(U3-Pad7) -> D0
- U3 pad 8: GND -> D1
- U3 pad 9: unconnected-(U3-Pad9) -> +5V
- U4 pad 1: unconnected-(U4-Pad1) -> A0
- U4 pad 10: unconnected-(U4-Pad10) -> GND
- U4 pad 11: unconnected-(U4-Pad11) -> D2
- U4 pad 12: unconnected-(U4-Pad12) -> D3
- U4 pad 13: unconnected-(U4-Pad13) -> /RW
- U4 pad 14: unconnected-(U4-Pad14) -> A5
- U4 pad 15: unconnected-(U4-Pad15) -> A6
- U4 pad 16: GND -> A7
- U4 pad 17: unconnected-(U4-Pad17) -> A8
- U4 pad 18: unconnected-(U4-Pad18) -> A9
- U4 pad 2: unconnected-(U4-Pad2) -> A1
- U4 pad 20: unconnected-(U4-Pad20) -> A10
- U4 pad 21: unconnected-(U4-Pad21) -> A11
- U4 pad 22: unconnected-(U4-Pad22) -> A12
- U4 pad 23: unconnected-(U4-Pad23) -> A13
- U4 pad 24: unconnected-(U4-Pad24) -> A14
- U4 pad 25: unconnected-(U4-Pad25) -> D4
- U4 pad 26: unconnected-(U4-Pad26) -> D5
- U4 pad 27: unconnected-(U4-Pad27) -> +5V
- U4 pad 28: unconnected-(U4-Pad28) -> GND
- U4 pad 29: unconnected-(U4-Pad29) -> D6
- U4 pad 3: unconnected-(U4-Pad3) -> A2
- U4 pad 30: unconnected-(U4-Pad30) -> D7
- U4 pad 31: unconnected-(U4-Pad31) -> GND
- U4 pad 32: +5V -> A15
- U4 pad 4: unconnected-(U4-Pad4) -> A3
- U4 pad 5: unconnected-(U4-Pad5) -> A4
- U4 pad 6: unconnected-(U4-Pad6) -> RAM_EN2
- U4 pad 7: unconnected-(U4-Pad7) -> D0
- U4 pad 8: unconnected-(U4-Pad8) -> D1
- U4 pad 9: unconnected-(U4-Pad9) -> +5V
- X1 pad 8: CPU_CLK -> +5V
Other:
- board outline removed
- copper layers 2 -> 4

Commit message: Full interrupt and IACK decoding in PLD
Parts:
- removed C1: C_Polarized, Capacitor_THT:CP_Radial_D5.0mm_P2.50mm
- removed C2: C_Polarized, Capacitor_THT:CP_Radial_D8.0mm_P3.80mm
- removed D1, D2: LED, LED_THT:LED_D5.0mm
- removed J2: DC_Jack, Connector_BarrelJack:BarrelJack_GCT_DCJ200-10-A_Horizontal
- removed J3, J4: Conn_01x06, Connector_PinHeader_2.54mm:PinHeader_1x06_P2.54mm_Vertical
- removed J5: Conn_02x20_Odd_Even, Connector_PinHeader_2.54mm:PinHeader_2x20_P2.54mm_Vertical
- removed R1, R10, R11, R12, R13, R2, R3, R4, R5, R6, R7, R8, R9: R, Resistor_SMD:R_1206_3216Metric_Pad1.30x1.75mm_HandSolder
- removed SW1: SW_Push, Button_Switch_THT:SW_PUSH_6mm_H5mm
- removed U1: MC68008, Package_LCC:PLCC-52_THT-Socket
- removed U10: 74HC595, Package_DIP:DIP-16_W7.62mm_Socket_LongPads
- removed U11: 74HC10, Package_DIP:DIP-14_W7.62mm_Socket_LongPads
- removed U12, U13: GAL16V8, Package_DIP:DIP-20_W7.62mm_Socket_LongPads
- removed U14: NE555P, Package_DIP:DIP-8_W7.62mm
- removed U2, U3, U4, U5, U6, U7: AS7C4096A, Package_SO:SOJ-36_10.16x23.49mm_P1.27mm
- removed U8: SST39SF040, Package_DIP:DIP-32_W15.24mm_Socket_LongPads
- removed U9: XR68C681, Package_LCC:PLCC-44_THT-Socket
- removed X1, X2: CXO_DIP8, Oscillator:Oscillator_DIP-8

Commit message: Mackerel-08 mostly routed
Parts:
- added C1: C_Polarized, Capacitor_THT:CP_Radial_D5.0mm_P2.50mm, F.Cu at (160.0, 99.1)
- added C2: C_Polarized, Capacitor_THT:CP_Radial_D8.0mm_P3.80mm, F.Cu at (30.5, 93.5)
- added D1: LED, LED_THT:LED_D5.0mm, F.Cu at (146.1, 114.3)
- added D2: LED, LED_THT:LED_D5.0mm, F.Cu at (132.1, 114.3)
- added J1: Conn_02x20_Odd_Even, Connector_PinSocket_2.54mm:PinSocket_2x20_P2.54mm_Horizontal, F.Cu at (30.5, 114.3)
- added J2: DC_Jack, Connector_BarrelJack:BarrelJack_GCT_DCJ200-10-A_Horizontal, F.Cu at (34.5, 104.1)
- added J3: Conn_02x10_Odd_Even, Connector_PinSocket_2.54mm:PinSocket_2x10_P2.54mm_Horizontal, F.Cu at (96.5, 114.3)
- added J4: Conn_02x10_Odd_Even, Connector_PinSocket_2.54mm:PinSocket_2x10_P2.54mm_Horizontal, F.Cu at (26.7, 30.5)
- added J5: Conn_01x06, Connector_PinSocket_2.54mm:PinSocket_1x06_P2.54mm_Horizontal, F.Cu at (24.1, 61.0)
- added J6: Conn_01x06, Connector_PinSocket_2.54mm:PinSocket_1x06_P2.54mm_Horizontal, F.Cu at (24.1, 81.3)
- added R10: R, Resistor_SMD:R_1206_3216Metric_Pad1.30x1.75mm_HandSolder, B.Cu at (147.7, 124.3)
- added R11: R, Resistor_SMD:R_1206_3216Metric_Pad1.30x1.75mm_HandSolder, B.Cu at (136.3, 122.2)
- added R12: R, Resistor_SMD:R_1206_3216Metric_Pad1.30x1.75mm_HandSolder, B.Cu at (171.6, 105.8)
- added R13: R, Resistor_SMD:R_1206_3216Metric_Pad1.30x1.75mm_HandSolder, B.Cu at (163.6, 105.8)
- added R2: R, Resistor_SMD:R_1206_3216Metric_Pad1.30x1.75mm_HandSolder, B.Cu at (54.9, 38.0)
- added R3: R, Resistor_SMD:R_1206_3216Metric_Pad1.30x1.75mm_HandSolder, B.Cu at (92.9, 24.2)
- added R4: R, Resistor_SMD:R_1206_3216Metric_Pad1.30x1.75mm_HandSolder, B.Cu at (106.2, 44.7)
- added R5: R, Resistor_SMD:R_1206_3216Metric_Pad1.30x1.75mm_HandSolder, B.Cu at (99.1, 24.1)
- added R6: R, Resistor_SMD:R_1206_3216Metric_Pad1.30x1.75mm_HandSolder, B.Cu at (112.9, 44.5)
- added R7: R, Resistor_SMD:R_1206_3216Metric_Pad1.30x1.75mm_HandSolder, B.Cu at (115.6, 25.8)
- added R8: R, Resistor_SMD:R_1206_3216Metric_Pad1.30x1.75mm_HandSolder, B.Cu at (105.1, 24.0)
- added R9: R, Resistor_SMD:R_1206_3216Metric_Pad1.30x1.75mm_HandSolder, B.Cu at (105.7, 41.4)
- added SW1: SW_Push, Button_Switch_THT:SW_PUSH_6mm_H5mm, F.Cu at (167.6, 115.6)
- added U1: MC68008, Package_LCC:PLCC-52_THT-Socket, F.Cu at (99.1, 40.6)
- added U10: XR68C681, Package_LCC:PLCC-44_THT-Socket, F.Cu at (53.3, 33.0)
- added U11: 74HC595, Package_DIP:DIP-16_W7.62mm_Socket_LongPads, F.Cu at (132.1, 50.8)
- added U12: ATF22V10C, Package_DIP:DIP-24_W7.62mm_Socket_LongPads, F.Cu at (78.7, 104.1)
- added U13: 74HC10, Package_DIP:DIP-14_W7.62mm_Socket_LongPads, F.Cu at (134.6, 35.6)
- added U14: ATF22V10C, Package_DIP:DIP-24_W7.62mm_Socket_LongPads, F.Cu at (121.9, 104.1)
- added U15: NE555P, Package_DIP:DIP-8_W7.62mm_Socket_LongPads, F.Cu at (167.6, 96.5)
- added U2: AS7C4096A, Package_SO:SOJ-36_10.16x23.49mm_P1.27mm, F.Cu at (48.8, 76.5)
- added U3: AS7C4096A, Package_SO:SOJ-36_10.16x23.49mm_P1.27mm, F.Cu at (64.0, 76.5)
- added U4: AS7C4096A, Package_SO:SOJ-36_10.16x23.49mm_P1.27mm, F.Cu at (79.3, 76.5)
- added U5: AS7C4096A, Package_SO:SOJ-36_10.16x23.49mm_P1.27mm, F.Cu at (94.5, 76.5)
- added U6: AS7C4096A, Package_SO:SOJ-36_10.16x23.49mm_P1.27mm, F.Cu at (109.8, 76.5)
- added U7: AS7C4096A, Package_SO:SOJ-36_10.16x23.49mm_P1.27mm, F.Cu at (125.0, 76.5)
- added U8: AS7C4096A, Package_SO:SOJ-36_10.16x23.49mm_P1.27mm, F.Cu at (140.2, 76.5)
- added U9: SST39SF040, Socket:DIP_Socket-32_W11.9_W12.7_W15.24_W17.78_W18.5_3M_232-1285-00-0602J, F.Cu at (160.0, 43.2)
- added X1: CXO_DIP8, Oscillator:Oscillator_DIP-8, F.Cu at (76.2, 38.1)
- added X2: CXO_DIP8, Oscillator:Oscillator_DIP-8, F.Cu at (76.2, 53.3)
Routing:
- net /A1: track 0.00 -> 328.3 mm, vias 0 -> 6
- net /A2: track 0.00 -> 315.7 mm, vias 0 -> 6
- net /A3: track 0.00 -> 299.6 mm, vias 0 -> 5
- net //RESET: track 0.00 -> 285.7 mm, vias 0 -> 3
- net /D3: track 0.00 -> 259.1 mm, vias 0 -> 5
- net /A4: track 0.00 -> 250.9 mm, vias 0 -> 5
- net /D4: track 0.00 -> 243.6 mm, vias 0 -> 3
- net /D5: track 0.00 -> 242.9 mm, vias 0 -> 4
- net /A7: track 0.00 -> 238.4 mm, vias 0 -> 3
- net /D7: track 0.00 -> 235.4 mm, vias 0 -> 5
- net /D2: track 0.00 -> 235.0 mm, vias 0 -> 3
- net /D1: track 0.00 -> 233.6 mm, vias 0 -> 3
- net /D6: track 0.00 -> 233.4 mm, vias 0 -> 5
- net /A8: track 0.00 -> 232.8 mm, vias 0 -> 3
- net /A5: track 0.00 -> 232.1 mm, vias 0 -> 3
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- added copper zone on In2.Cu, net +5V
- added copper zone on In1.Cu, net GND
Other:
- board outline added: 160 x 99.1 mm
