File: design/mackerel-08-v1/mackerel-08-v1.kicad_pcb (KiCad board)
At the start: 4 copper layers, 180 x 130 mm, 83 parts, among them J1 Conn_02x04_Odd_Even, J2 DC_Jack, J3 Conn_02x20_Odd_Even, J4 Conn_02x04_Odd_Even, J5 DB9_Male_MountingHoles, J6 DB9_Male_MountingHoles, J7 Conn_02x04_Odd_Even, J8 Conn_01x03, J9 Conn_01x12, SW1 SW_Push, SW2 SW_SPDT, U1 MC68008, U10 XR68C681, U11 74HC595, U12 ATF22V10C, U13 MAX3232, U14 ATF22V10C, U15 NE555P, U16 MAX3232, U17 ATF22V10C, U2 AS6C4008-55PCN, U3 SST39SF040, U4 AS6C4008-55PCN, U5 AS6C4008-55PCN, U6 AS6C4008-55PCN, U7 AS6C4008-55PCN, U8 AS6C4008-55PCN, U9 AS6C4008-55PCN, X1 CXO_DIP8, X2 CXO_DIP8

Commit message: Clean up the schematic, ready for final routing
Parts:
- removed the C20 at (93.9, 45.1)
- removed the C21 at (68.6, 45.2)
- removed the C22 at (100.0, 45.1)
- removed the C23 at (74.7, 45.2)
- removed the C24 at (90.3, 45.1)
- removed the C26 at (64.9, 45.2)
- removed the C27 at (83.2, 45.2)
- removed the J5 at (178.0, 42.0)
- removed the J6 at (134.0, 42.0)
- removed J8: Conn_01x03, Connector_PinHeader_2.54mm:PinHeader_1x03_P2.54mm_Vertical
- removed the J9 at (197.6, 65.0)
- removed the U13 at (89.3, 41.0)
- removed U16: MAX3232, Package_DIP:DIP-16_W7.62mm
- added J2: Conn_01x06, Connector_PinSocket_2.54mm:PinSocket_1x06_P2.54mm_Horizontal, F.Cu at (-24.5, 34.2)
- added J3: Conn_01x06, Connector_PinSocket_2.54mm:PinSocket_1x06_P2.54mm_Horizontal, F.Cu at (-11.2, 34.2)
- added JP1: Jumper_2_Open, Connector_PinHeader_2.54mm:PinHeader_1x02_P2.54mm_Vertical, F.Cu at (-57.5, 39.4)
- added R18: R, Resistor_THT:R_Axial_DIN0207_L6.3mm_D2.5mm_P7.62mm_Horizontal, F.Cu at (-69.0, 39.1)
- added R19: R, Resistor_THT:R_Axial_DIN0207_L6.3mm_D2.5mm_P7.62mm_Horizontal, F.Cu at (-69.0, 43.1)
- added R20: R, Resistor_THT:R_Axial_DIN0207_L6.3mm_D2.5mm_P7.62mm_Horizontal, F.Cu at (-69.0, 47.2)
- added R21: R, Resistor_THT:R_Axial_DIN0207_L6.3mm_D2.5mm_P7.62mm_Horizontal, F.Cu at (-69.0, 51.2)
- added R22: R, Resistor_THT:R_Axial_DIN0207_L6.3mm_D2.5mm_P7.62mm_Horizontal, F.Cu at (-69.0, 55.3)
- added R23: R, Resistor_THT:R_Axial_DIN0207_L6.3mm_D2.5mm_P7.62mm_Horizontal, F.Cu at (-69.0, 59.4)
- added R24: R, Resistor_THT:R_Axial_DIN0207_L6.3mm_D2.5mm_P7.62mm_Horizontal, F.Cu at (-69.0, 63.4)
- added R25: R, Resistor_THT:R_Axial_DIN0207_L6.3mm_D2.5mm_P7.62mm_Horizontal, F.Cu at (-69.0, 67.5)
- added R26: R, Resistor_THT:R_Axial_DIN0207_L6.3mm_D2.5mm_P7.62mm_Horizontal, F.Cu at (-69.0, 71.5)
- added R27: R, Resistor_THT:R_Axial_DIN0207_L6.3mm_D2.5mm_P7.62mm_Horizontal, F.Cu at (-69.0, 75.5)
- added R28: R, Resistor_THT:R_Axial_DIN0207_L6.3mm_D2.5mm_P7.62mm_Horizontal, F.Cu at (-34.0, 51.2)
- added R29: R, Resistor_THT:R_Axial_DIN0207_L6.3mm_D2.5mm_P7.62mm_Horizontal, F.Cu at (-34.0, 55.2)
- C25: value C_Polarized_US -> C_Polarized; footprint Capacitor_THT:CP_Radial_D5.0mm_P2.50mm -> Capacitor_THT:CP_Radial_D10.0mm_P5.00mm
- moved C30 130.8 mm to (-48.2, 105.5)
- moved C11 83.6 mm to (-22.7, 105.6), turned to -90 degrees
- moved U6 80.0 mm to (60.0, 100.0)
- moved U7 80.0 mm to (80.0, 100.0)
- moved U12 60.0 mm to (180.0, 100.0)
- moved C22 48.9 mm to (39.3, 47.1), turned to 0 degrees
- moved U10 40.0 mm to (140.0, 100.0)
- moved U8 40.0 mm to (100.0, 100.0)
- moved U9 40.0 mm to (120.0, 100.0)
- moved C25 21.9 mm to (104.7, 66.7)
- moved U11 20.0 mm to (160.0, 100.0)
- moved R1 9.39 mm to (99.4, 55.5)
- moved R3 9.39 mm to (99.4, 52.0)
- moved R2 9.39 mm to (99.4, 58.8)
- moved C10 0.25 mm to (33.9, 50.6)
- renumbered C28 to C10, C2 to C11, C3 to C12, C4 to C13, C5 to C14, C6 to C15, C7 to C16, C8 to C17, C9 to C18, C10 to C19, C11 to C20, C12 to C21, C29 to C22, C13 to C23, C14 to C24, C15 to C26, C16 to C27, C17 to C28, C18 to C29, C19 to C30, C1 to C9, D3 to D1, D1 to D2, D2 to D3, J3 to J1, J1 to J5, J4 to J6, J2 to J9, R3 to R1, R16 to R10, R17 to R11, R1 to R12, R15 to R13, R12 to R14, R11 to R15, R10 to R16, R13 to R17, R4 to R2, R5 to R3, R6 to R4, R7 to R5, R8 to R6, R9 to R7, R2 to R8, R14 to R9, U4 to U10, U8 to U11, U5 to U12, U3 to U13, U10 to U15, U15 to U17, U11 to U2, U12 to U3, U14 to U4, U17 to U5, U2 to U8
Connections:
- net CLK_CPU renamed /CLK_CPU
- net /IRQ2 renamed /IRQ_EXP
- C25 pad 1: GND -> +5V
- C25 pad 2: Net-(U13-VS-) -> GND
- J1 pad 37: /DTACK2 -> /DTACK_EXP
- J1 pad 38: /IACK2 -> /IACK_EXP
- U4 pad 17: unconnected-(U14-IO3-Pad17) -> AS
- U4 pad 18: /IACK2 -> /IACK_EXP
- U4 pad 7: unconnected-(U14-IN6-Pad7) -> Net-(U4-IN6)
- U4 pad 8: unconnected-(U14-IN7-Pad8) -> Net-(U4-IN7)
- U4 pad 9: unconnected-(U14-IN8-Pad9) -> Net-(U4-IN8)
- U5 pad 1: /DTACK_DUART -> AS
- U5 pad 10: /IN9 -> Net-(U5-IN9)
- U5 pad 11: /IN10 -> Net-(U5-IN10)
- U5 pad 13: /IN11 -> Net-(U5-IN11)
- U5 pad 14: /IO0 -> unconnected-(U5-IO0-Pad14)
- U5 pad 15: /IO1 -> unconnected-(U5-IO1-Pad15)
- U5 pad 16: /IO2 -> unconnected-(U5-IO2-Pad16)
- U5 pad 17: /IO3 -> unconnected-(U5-IO3-Pad17)
- U5 pad 18: /IO4 -> unconnected-(U5-IO4-Pad18)
- U5 pad 19: /IO5 -> unconnected-(U5-IO5-Pad19)
- U5 pad 2: /DTACK2 -> /ROM
- U5 pad 20: /IO6 -> unconnected-(U5-IO6-Pad20)
- U5 pad 21: /IO7 -> unconnected-(U5-IO7-Pad21)
- U5 pad 22: /IO8 -> unconnected-(U5-IO8-Pad22)
- U5 pad 23: /DTACK_CPU -> Net-(JP1-A)
- U5 pad 3: /AS -> /DUART
- U5 pad 4: /DS -> Net-(U5-IN3/PD)
- U5 pad 5: /IACK -> /EXP
- U5 pad 6: /IACK_DUART -> /DTACK_DUART
- U5 pad 7: /IACK2 -> /DTACK_EXP
- U5 pad 8: /DUART -> /IACK_EXP
- U5 pad 9: /EXP -> /IACK_DUART
Routing:
- net /IRQ_DUART: track 149.2 -> 0.00 mm, vias 3 -> 0
- net RXA: track 112.2 -> 0.00 mm
- net TXA: track 106.0 -> 0.00 mm
- net /DUART: track 94.2 -> 0.00 mm
- net /IRQ_EXP: track 91.2 -> 0.00 mm, vias 2 -> 0
- net Net-(U13-R1IN): track 87.7 -> 0.00 mm, vias 2 -> 0
- net /IACK2: track 86.6 -> 0.00 mm, vias 2 -> 0
- net Net-(U13-T1OUT): track 85.1 -> 0.00 mm
- net Net-(U16-R1IN): track 78.2 -> 0.00 mm
- net Net-(U13-T2OUT): track 76.3 -> 0.00 mm
- net /CTSA: track 71.2 -> 0.00 mm, vias 1 -> 0
- net Net-(U13-R2IN): track 69.2 -> 0.00 mm
- net Net-(U16-T1OUT): track 66.6 -> 0.00 mm
- net Net-(U16-T2OUT): track 63.9 -> 0.00 mm, vias 1 -> 0
- net /RTSA: track 61.7 -> 0.00 mm
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
Commit message: Mackerel-08 v1 is fully routed, needs graphics, labels, and cleanup
Parts:
- removed C30, C9: C, Capacitor_THT:C_Disc_D4.3mm_W1.9mm_P5.00mm
- removed R21, R22, R23, R24, R25, R26, R27: R, Resistor_THT:R_Axial_DIN0207_L6.3mm_D2.5mm_P7.62mm_Horizontal
- added JP2: Jumper_2_Open, Connector_PinHeader_2.54mm:PinHeader_1x02_P2.54mm_Vertical, F.Cu at (64.5, 43.0)
- added JP3: Jumper_2_Open, Connector_PinHeader_2.54mm:PinHeader_1x02_P2.54mm_Vertical, F.Cu at (64.5, 49.8)
- moved R19 239.7 mm to (165.4, 93.0)
- moved R20 239.5 mm to (165.4, 96.2)
- moved JP1 199.1 mm to (140.5, 60.5), turned to -90 degrees
- moved R18 198.7 mm to (129.7, 42.5)
- moved J2 109.7 mm to (84.0, 50.5), turned to -90 degrees
- moved R13 98.4 mm to (29.2, 143.3), turned to 90 degrees
- moved R28 89.7 mm to (52.4, 75.0)
- moved R29 89.4 mm to (52.4, 78.2)
- moved D3 86.3 mm to (24.2, 125.8)
- moved R14 82.0 mm to (22.2, 143.3), turned to 90 degrees
- moved R17 80.2 mm to (25.8, 143.3), turned to 90 degrees
- moved J3 73.0 mm to (60.0, 50.5), turned to -90 degrees
- moved D2 71.2 mm to (24.2, 101.5)
- moved D1 67.2 mm to (24.2, 113.8)
- moved C11 65.2 mm to (33.2, 72.2)
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Connections:
- J2 pad 3: +5V -> Net-(J2-Pin_3)
- J3 pad 3: +5V -> Net-(J3-Pin_3)
- U4 pad 7: Net-(U4-IN6) -> GND
- U4 pad 8: Net-(U4-IN7) -> GND
- U4 pad 9: Net-(U4-IN8) -> GND
- U5 pad 10: Net-(U5-IN9) -> GND
- U5 pad 11: Net-(U5-IN10) -> GND
- U5 pad 13: Net-(U5-IN11) -> GND
- U5 pad 4: Net-(U5-IN3/PD) -> GND
Routing:
- net SPI_INT1: track 0.00 -> 174.2 mm, vias 0 -> 4
- net /DTACK_DUART: track 0.00 -> 157.5 mm, vias 0 -> 1
- net /IACK_DUART: track 0.00 -> 157.1 mm, vias 0 -> 5
- net SPI_INT0: track 0.00 -> 144.4 mm, vias 0 -> 2
- net /RAM0: track 0.00 -> 144.0 mm, vias 0 -> 3
- net /DUART: track 0.00 -> 134.0 mm, vias 0 -> 3
- net /RAM1: track 0.00 -> 124.9 mm, vias 0 -> 3
- net /IRQ_DUART: track 0.00 -> 122.9 mm, vias 0 -> 1
- net SPI_DO: track 46.2 -> 163.3 mm, vias 0 -> 4
- net SPI_CS1: track 0.00 -> 116.3 mm, vias 0 -> 2
- net /RAM2: track 0.00 -> 103.7 mm, vias 0 -> 3
- net /IRQ_EXP: track 0.00 -> 90.9 mm, vias 0 -> 2
- net /DTACK_EXP: track 0.00 -> 89.2 mm, vias 0 -> 1
- net /IACK_EXP: track 0.00 -> 88.3 mm, vias 0 -> 1
- net /RESET: track 208.9 -> 293.5 mm
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Other:
- board size 180 x 130 mm -> 180 x 120 mm
- board text added: "/IRQ2"
- board text added: "RTSA"
- board text added: "RTSB"
- board text added: "RXA"
- board text added: "RXB"
- board text added: "TXA"
- board text added: "TXB"
- board text removed: "/INT2"
- board text removed: "ON"
- board text removed: "RESET"

Commit message: Mackerel-08 SVC v1 labeled and ready for final checks
Parts:
- added REF**: OSHW-Logo2_7.3x6mm_SilkScreen, Symbol:OSHW-Logo2_7.3x6mm_SilkScreen, F.Cu at (166.8, 48.8)
- added REF**: KiCad-Logo2_5mm_SilkScreen, Symbol:KiCad-Logo2_5mm_SilkScreen, F.Cu at (182.8, 48.8)
- moved C22 6.76 mm to (38.2, 59.6), turned to -90 degrees
- moved SW1 4.50 mm to (23.0, 78.0)
- moved SW2 4.33 mm to (21.6, 68.0)
- moved R15 3.69 mm to (27.0, 92.2)
- moved R16 3.69 mm to (23.5, 92.2)
- moved C25 3.50 mm to (99.0, 85.1)
- moved R28 2.12 mm to (51.2, 76.8)
- moved R29 2.12 mm to (51.2, 80.0)
- moved JP2 0.75 mm to (64.5, 43.8)
- moved JP3 0.25 mm to (64.5, 49.5)
Routing:
- net /CTSB: track 24.6 -> 26.8 mm
- net /CTSA: track 22.2 -> 24.1 mm
- net Net-(U17-THR): track 30.9 -> 32.4 mm
- net AS: track 24.1 -> 25.6 mm
- net Net-(J9-VCC): track 11.8 -> 12.6 mm
- net /AS: track 142.1 -> 142.8 mm
Other:
- outline, holes or cut-outs redrawn
- board text added: "555"
- board text added: "5V ONLY"
- board text added: "ADDRESS DECODER"
- board text added: "BOOT SIGNAL"
- board text added: "C. Maykish - 2024"
- board text added: "CPU CLOCK"
- board text added: "DTACK GENERATOR"
- board text added: "DUART CLK"
- board text added: "INTERRUPT DECODER"
- board text added: "MACKEREL-08 SBC v1 github.com/crmaykish/mackerel-68k"
- board text added: "MC68008 CPU"
- board text added: "Mackerel-08 SBC v1 Designed by Colin Maykish - July 2024 github.com/crmaykish/mackerel-68k"
- board text added: "OFF"
- board text added: "ON"
- board text added: "Open: DTACK Grounded Closed: DTACK Gen"
- board text added: "RAM0"
- board text added: "RAM1"
- board text added: "RAM2"
- board text added: "RAM3"
- board text added: "RAM4"
- board text added: "RAM5"
- board text added: "RAM6"
- board text added: "RESET"
- board text added: "ROM"
- board text added: "UART 5V"
- board text added: "UART A"
- board text added: "UART B"
- board text added: "XR68C681 DUART"
