File: design/mackerel-08-v1/mackerel-08-v1.kicad_sch (KiCad schematic)
At the start: 75 parts, among them J1 Conn_01x08, J2 DC_Jack, J3 Conn_02x20_Counter_Clockwise, J4 Conn_02x20_Counter_Clockwise, J5 DB9_Male_MountingHoles, J6 DB9_Male_MountingHoles, SW1 SW_Push, SW2 SW_SPDT, U1 MC68008, U10 XR68C681, U11 74HC595, U12 ATF22V10C, U13 MAX3232, U14 ATF22V10C, U15 NE555P, U16 MAX3232, U2 AS6C4008-55PCN, U3 AS6C4008-55PCN, U4 AS6C4008-55PCN, U5 AS6C4008-55PCN, U6 AS6C4008-55PCN, U7 AS6C4008-55PCN, U8 AS6C4008-55PCN, U9 SST39SF040, X1 CXO_DIP8, X2 CXO_DIP8

Commit message: Mackerel-08 PCB Rev1 mostly routed
Parts:
- removed J1: Conn_01x08, Connector_PinSocket_2.54mm:PinSocket_1x08_P2.54mm_Vertical, symbol Connector_Generic:Conn_01x08
- added C29, C30: C, Capacitor_THT:C_Disc_D4.3mm_W1.9mm_P5.00mm, symbol Device:C
- added J1, J10, J9: Conn_02x04_Counter_Clockwise, Connector_PinSocket_2.54mm:PinSocket_2x04_P2.54mm_Vertical, symbol Connector_Generic:Conn_02x04_Counter_Clockwise
- added J8: Conn_01x03, Connector_PinHeader_2.54mm:PinHeader_1x03_P2.54mm_Vertical, symbol Connector_Generic:Conn_01x03
- added R16: R, Resistor_THT:R_Axial_DIN0207_L6.3mm_D2.5mm_P7.62mm_Horizontal, symbol Device:R
- added U17: ATF22V10C, Package_DIP:DIP-24_W7.62mm, symbol mackerel-68k-symbols:ATF22V10C
- C10, C11, C12, C13, C14, C15, C16, C17, C18, C19, C3, C4, C5, C6, C7, C8, C9: footprint Capacitor_THT:C_Disc_D3.0mm_W2.0mm_P2.50mm -> Capacitor_THT:C_Disc_D4.3mm_W1.9mm_P5.00mm
- C2: footprint Capacitor_THT:CP_Radial_D8.0mm_P3.80mm -> Capacitor_THT:CP_Radial_D10.0mm_P5.00mm
- C20, C21, C22, C23, C24, C25, C26, C27: footprint Capacitor_THT:CP_Radial_Tantal_D4.5mm_P5.00mm -> Capacitor_THT:CP_Radial_D5.0mm_P2.50mm
- H1, H2, H3, H4: footprint MountingHole:MountingHole_3.7mm_Pad_Via -> MountingHole:MountingHole_3.2mm_M3_Pad
- J3: footprint (none) -> Connector_IDC:IDC-Header_2x20_P2.54mm_Vertical
- U9: footprint Package_DIP:DIP-32_W15.24mm -> Socket:DIP_Socket-32_W11.9_W12.7_W15.24_W17.78_W18.5_3M_232-1285-00-0602J
- renumbered D2 to D1, D1 to D2, U7 to U2, U6 to U4, U8 to U6, U4 to U7, U2 to U8
Connections:
- net SD_CD is gone; now on net SPI_DO: U10.40 (IP2)
- net /DUART0 is gone; now on net /RAM6: U12.15 (IO1)
- net /IRQ1 is gone; now on net FC0: U14.1 (CLK/IN0)
- net +5V: now also SW2.1 (A), C29.1, C30.1, R16.2, U17.24 (vcc); no longer J2.1 (VCC)
- net A1: now also U14.10 (IN9); no longer U14.9 (IN8)
- net A13: now also U12.4 (IN3/PD)
- net A14: now also U12.5 (IN4)
- net A15: now also U12.6 (IN5)
- net A2: now also U14.11 (IN10); no longer U14.10 (IN9)
- net A3: now also U14.13 (IN11); no longer U14.11 (IN10)
- net FC0: no longer U14.4 (IN3/PD)
- net FC1: now also U14.2 (IN1); no longer U14.5 (IN4)
- net FC2: now also U14.3 (IN2); no longer U14.6 (IN5)
- net GND: now also U9.16 (GND), U9.24 (/OE), C29.2, C30.2, J8.1 (Pin_1), U17.12 (GND)
- net RXA: now also J8.3 (Pin_3)
- net RXB: now also U16.12 (R1OUT)
- net SPI_DO: no longer U10.3 (IP3)
- net TXA: now also J8.2 (Pin_2)
- net TXB: now also U16.11 (T1IN)
- net /AS: now also U14.4 (IN3/PD); no longer U14.13 (IN11)
- net /CTSB: now also U16.9 (R2OUT)
- net /DTACK_CPU: now also U17.23 (IO9)
- net /DUART: now also U12.23 (IO9)
- net /IACK: now also U14.23 (IO9); no longer U14.19 (IO5)
- net /IACK2: now also U14.18 (IO4); no longer U14.15 (IO1)
- net /IACK_DUART: now also U14.19 (IO5)
- net /INT_DUART: now also U14.5 (IN4)
- net /IPL0: now also U14.22 (IO8); no longer U14.21 (IO7)
- net /IPL1: now also U14.21 (IO7); no longer U14.22 (IO8)
- net /IPL2: now also U14.20 (IO6); no longer U14.23 (IO9)
- net /IRQ2: now also U14.6 (IN5); no longer U14.2 (IN1)
- net /RAM0: now also U12.21 (IO7), U2.22 (CE#); no longer U12.23 (IO9), U8.22 (CE#)
- net /RAM1: now also U12.20 (IO6); no longer U12.22 (IO8)
- net /RAM2: now also U12.19 (IO5), U4.22 (CE#); no longer U12.21 (IO7), U7.22 (CE#)
- net /RAM3: now also U12.18 (IO4); no longer U12.20 (IO6)
- net /RAM4: now also U12.17 (IO3), U6.22 (CE#); no longer U12.19 (IO5), U2.22 (CE#)
- net /RAM5: now also U12.16 (IO2), U7.22 (CE#); no longer U12.18 (IO4), U4.22 (CE#)
- net /RAM6: now also U8.22 (CE#); no longer U12.17 (IO3), U6.22 (CE#)
- net /RTSB: now also U16.10 (T2IN)
- net /IACK4: now reaches U14.16 (IO2)
- net /IACK3: now reaches U14.17 (IO3)
- net /IRQ3: now reaches U14.7 (IN6)
- net /IRQ4: now reaches U14.8 (IN7)
- net at SW2.2 (B): now also J2.1 (VCC)
- net LED_U0: no longer names the net of R1.1, U10.17 (OP7)
- net /CS_IO renamed /IO
- net /IACK1: no longer names the net of U14.14 (IO0)
- net /ROM0 renamed /ROM
- net /ROM: now also U12.22 (IO8); no longer U12.16 (IO2)
- new net: R16.1, U10.3 (IP3)
- new net /DTACK0: U17.2 (IN1)
- new net /DTACK1: U17.3 (IN2)
- new net /DTACK2: U17.4 (IN3/PD)
- new net /IACK5: U14.15 (IO1)
- new net /IRQ5: U14.9 (IN8)
Other:
- note added: "Address Decoder"
- note added: "TODO: Figure out IACK/DTACK relationship"
- note added: "TODO: add interrupt pins"
- note added: "TODO: include SPI interrupts"
- note added: "TODO: pullups on SPI lines"
- note added: "TODO: what goes into DTACK generation?"
- note removed: "IACK factors into DTACK"
- note removed: "TODO: do something with DTACK"
- moved on the sheet: J2, R14, R15, SW2, U12, U14
