File: design/mackerel-08-v1/mackerel-08-duart.kicad_sch (KiCad schematic)
At the start: 25 parts, among them J1 Conn_02x04_Odd_Even, J4 Conn_02x04_Odd_Even, J5 DB9_Male_MountingHoles, J6 DB9_Male_MountingHoles, J7 Conn_02x04_Odd_Even, J8 Conn_01x03, U10 XR68C681, U13 MAX3232, U16 MAX3232, X2 CXO_DIP8

Commit message: Clean up the schematic, ready for final routing
Parts:
- removed C20, C21, C22, C23, C24, C25, C26, C27: C_Polarized_US, Capacitor_THT:CP_Radial_D5.0mm_P2.50mm, symbol Device:C_Polarized_US
- removed J5, J6: DB9_Male_MountingHoles, Connector_Dsub:DSUB-9_Male_Horizontal_P2.77x2.84mm_EdgePinOffset7.70mm_Housed_MountingHolesOffset9.12mm, symbol Connector:DB9_Male_MountingHoles
- removed J8: Conn_01x03, Connector_PinHeader_2.54mm:PinHeader_1x03_P2.54mm_Vertical, symbol Connector_Generic:Conn_01x03
- removed U13, U16: MAX3232, Package_DIP:DIP-16_W7.62mm, symbol Interface_UART:MAX3232
- added J2, J3: Conn_01x06, Connector_PinSocket_2.54mm:PinSocket_1x06_P2.54mm_Horizontal, symbol Connector_Generic:Conn_01x06
- added R28, R29: R, Resistor_THT:R_Axial_DIN0207_L6.3mm_D2.5mm_P7.62mm_Horizontal, symbol Device:R
- renumbered D3 to D1, J1 to J5, J4 to J6, R16 to R10, R17 to R11, R1 to R12, R15 to R13, R2 to R8, R14 to R9, U10 to U15
Connections:
- net +5V: now also J2.3 (Pin_3), J3.3 (Pin_3)
- net GND: now also J2.1 (Pin_1), J3.1 (Pin_1), R28.1, R29.1
- net RXA: now also J2.4 (Pin_4)
- net RXB: now also J3.4 (Pin_4)
- net TXA: now also J2.5 (Pin_5)
- net TXB: now also J3.5 (Pin_5)
- net /CTSA: now also R28.2
- net /CTSB: now also R29.2
- net /RTSA: now also J2.2 (Pin_2)
- net /RTSB: now also J3.2 (Pin_2)
- no-connect marks 11 -> 5
Other:
- note added: "SPI Headers"
- note added: "SPI interrupts are assumed active-low"
- note added: "UART Headers"
- note added: "XR68C681 DUART"
- note removed: "TODO: check the pinout of CTS/RTS and the DB-9 connector"
- note removed: "TODO: pullups/downs on CTS inputs"
- company: (none) -> Colin Maykish
- title: (none) -> Mackerel-08 SBC v1
- moved on the sheet: D1, J5, J6, J7, R10, R11, R12, R13, R8, R9, U15, X2

Commit message: Mackerel-08 v1 is fully routed, needs graphics, labels, and cleanup
Parts:
- added JP2, JP3: Jumper_2_Open, Connector_PinHeader_2.54mm:PinHeader_1x02_P2.54mm_Vertical, symbol Jumper:Jumper_2_Open
Connections:
- net +5V: now also JP2.1 (A), JP3.1 (A); no longer J2.3 (Pin_3), J3.3 (Pin_3)
- new net: J2.3 (Pin_3), JP2.2 (B)
- new net: J3.3 (Pin_3), JP3.2 (B)
Other:
- moved on the sheet: J2, J3
