File: design/mackerel-30-itx/mackerel-30-itx.kicad_sch (KiCad schematic)
At the start: 10 parts, among them J1 DE9_Plug_MountingHoles, J2 DE9_Plug_MountingHoles, J3 Conn_02x20_Odd_Even, J4 ATX-24, J5 RJ45, J6 DIN-5

Commit message: Final touches on Mackerel-08 v1
Parts:
- J5: footprint Connector_RJ:RJ45_Amphenol_54602-x08_Horizontal -> Connector_RJ:RJ45_Bel_SI-60062-F
Changed lines of the file:
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@@
 			)
 		)
-		(property "Footprint" "Connector_RJ:RJ45_Amphenol_54602-x08_Horizontal"
+		(property "Footprint" "Connector_RJ:RJ45_Bel_SI-60062-F"
 			(at 39.37 47.625 90)
 			(effects
