File: hardware/mackerel-10-v1/mackerel-10-v1.kicad_pcb (KiCad board)
At the start: 2 copper layers, 160 x 100 mm, 40 parts, among them J1 Conn_02x05_Odd_Even, J2 DIN41612_02x32_AC, J3 DE9_Plug_MountingHoles, J4 Conn_01x06, J5 Conn_01x06, J6 DC_Jack, J7 DE9_Plug_MountingHoles, SW1 SW_Push, U1 68010D, U12 NE555P, U3 SST39SF040, U4 KM62256CLP, U5 SST39SF040, U6 KM62256CLP, U7 XR68C681, U8 MAX3232, U9 MAX3232, X1 50 MHz, X2 3.6864 MHz

Commit message: More progress on Mackerel-10 schematic and PCB
Parts:
- removed C2, C3: C_Polarized, Capacitor_THT:CP_Radial_D10.0mm_P5.00mm
- removed J3: DE9_Plug_MountingHoles, Connector_Dsub:DSUB-9_Male_Horizontal_P2.77x2.84mm_EdgePinOffset7.70mm_Housed_MountingHolesOffset9.12mm
- removed J6: DC_Jack, Connector_BarrelJack:BarrelJack_GCT_DCJ200-10-A_Horizontal
- removed U8, U9: MAX3232, Package_DIP:DIP-16_W7.62mm
- added C4: 1000uF, Capacitor_THT:CP_Radial_D10.0mm_P5.00mm, F.Cu at (24.7, 40.9)
- added H1: MountingHole_Pad, MountingHole:MountingHole_3.2mm_M3_Pad, F.Cu at (25.0, 25.0)
- added H2: MountingHole_Pad, MountingHole:MountingHole_3.2mm_M3_Pad, F.Cu at (215.0, 25.0)
- added H3: MountingHole_Pad, MountingHole:MountingHole_3.2mm_M3_Pad, F.Cu at (25.0, 155.0)
- added H4: MountingHole_Pad, MountingHole:MountingHole_3.2mm_M3_Pad, F.Cu at (215.0, 155.0)
- added J8: Barrel_Jack_MountingPin, Connector_BarrelJack:BarrelJack_Horizontal, F.Cu at (36.6, 34.4)
- added U10: ~, Package_LCC:PLCC-84_THT-Socket, F.Cu at (127.5, 99.8)
- added U11: ~, mackerel:SIMM-30, F.Cu at (159.4, 44.2)
- added U13: ~, mackerel:SIMM-30, F.Cu at (189.6, 44.2)
- added U14: ~, mackerel:SIMM-30, F.Cu at (204.7, 44.2)
- added U15: NE555P, Package_DIP:DIP-8_W7.62mm, F.Cu at (121.2, -81.8)
- added U16: 74HC245, Package_DIP:DIP-20_W7.62mm, F.Cu at (152.7, 143.0)
- added U17: 74HC245, Package_DIP:DIP-20_W7.62mm, F.Cu at (183.6, 143.0)
- J2: footprint Connector_DIN:DIN41612_C_2x32_Male_Horizontal_THT -> Connector_DIN:DIN41612_C_2x32_Female_Vertical_THT
- J7: value DE9_Plug_MountingHoles -> Conn_02x20_Odd_Even; footprint Connector_Dsub:DSUB-9_Male_Horizontal_P2.77x2.84mm_EdgePinOffset7.70mm_Housed_MountingHolesOffset9.12mm -> Connector_IDC:IDC-Header_2x20_P2.54mm_Vertical
- U12: value NE555P -> ~; footprint Package_DIP:DIP-8_W7.62mm -> mackerel:SIMM-30
- U4, U6: value KM62256CLP -> AS6C4008-55PCN; footprint Package_DIP:DIP-28_W15.24mm -> Package_DIP:DIP-32_W15.24mm
- moved X2 346.3 mm to (137.4, 32.3)
- moved X1 345.7 mm to (137.7, 48.3)
- moved D1 269.3 mm to (223.9, -86.7)
- moved J5 262.9 mm to (94.7, 31.1), turned to -90 degrees
- moved R12 250.8 mm to (221.0, -78.5)
- moved J4 237.5 mm to (66.5, 31.1), turned to -90 degrees
- moved D2 231.9 mm to (192.3, -86.9)
- moved U7 230.0 mm to (121.9, 30.2)
- moved U12 228.7 mm to (174.5, 44.2), turned to 90 degrees
- moved R13 221.4 mm to (189.7, -78.5)
- moved C1 163.3 mm to (124.0, -89.9)
- moved U5 158.4 mm to (33.2, 96.8), turned to 0 degrees
- moved JP1 155.7 mm to (-80.8, -98.6)
- moved JP2 155.7 mm to (-76.2, -98.6)
- moved SW1 148.7 mm to (108.0, -80.5)
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Connections:
- C1 pad 2: Net-(U12-THR) -> Net-(U15-THR)
- R10 pad 2: Net-(U12-R) -> Net-(U15-R)
- R11 pad 1: Net-(U12-THR) -> Net-(U15-THR)
- SW1 pad 2: Net-(U12-R) -> Net-(U15-R)
- U12 pad 1: GND -> +5V
- U12 pad 2: Net-(U12-THR) -> /DRAM_CAS1
- U12 pad 3: /RESET -> D8
- U12 pad 4: Net-(U12-R) -> DRAM_A0
- U12 pad 5: unconnected-(U12-CV-Pad5) -> DRAM_A1
- U12 pad 6: Net-(U12-THR) -> D9
- U12 pad 7: unconnected-(U12-DIS-Pad7) -> DRAM_A2
- U12 pad 8: +5V -> DRAM_A3
- U2 pad 10: /ODDROM -> /ROM_LOWER
- U2 pad 12: /EXP -> /DTACK_DUART
- U2 pad 15: /DTACK_DUART -> /IRQ_DUART
- U2 pad 16: /DTACK_EXP -> /IACK_DUART
- U2 pad 17: /IRQ1 -> unconnected-(U2-IO-Pad17)
- U2 pad 18: /IRQ2 -> unconnected-(U2-IO-Pad18)
- U2 pad 20: /IRQ3 -> unconnected-(U2-IO-Pad20)
- U2 pad 21: /IACK1 -> unconnected-(U2-IO-Pad21)
- U2 pad 22: /IACK2 -> unconnected-(U2-IO-Pad22)
- U2 pad 24: /IACK3 -> unconnected-(U2-IO-Pad24)
- U2 pad 6: /EVENRAM -> /SRAM_UPPER
- U2 pad 8: /ODDRAM -> /SRAM_LOWER
- U2 pad 9: /EVENROM -> /ROM_UPPER
- U3 pad 22: unconnected-(U3-CE-Pad22) -> /ROM_UPPER
- U3 pad 24: unconnected-(U3-OE-Pad24) -> GND
- U4 pad 1: A15 -> A19
- U4 pad 10: A1 -> A3
- U4 pad 11: D8 -> A2
- U4 pad 12: D9 -> A1
- U4 pad 13: D10 -> D8
- U4 pad 14: GND -> D9
- U4 pad 15: D11 -> D10
- U4 pad 16: D12 -> GND
- U4 pad 17: D13 -> D11
- U4 pad 18: D14 -> D12
- U4 pad 19: D15 -> D13
- U4 pad 2: A13 -> A17
- U4 pad 20: unconnected-(U4-~{CS}-Pad20) -> D14
- U4 pad 21: A11 -> D15
- U4 pad 22: unconnected-(U4-~{OE}-Pad22) -> /SRAM_UPPER
- U4 pad 23: A12 -> A11
- U4 pad 24: A10 -> GND
- U4 pad 25: A9 -> A12
- U4 pad 26: A14 -> A10
- U4 pad 27: unconnected-(U4-~{WE}-Pad27) -> A9
- U4 pad 28: +5V -> A14
- U4 pad 3: A8 -> A15
- U4 pad 4: A7 -> A13
- U4 pad 5: A6 -> A8
- U4 pad 6: A5 -> A7
- U4 pad 7: A4 -> A6
- U4 pad 8: A3 -> A5
- U4 pad 9: A2 -> A4
- U5 pad 22: unconnected-(U5-CE-Pad22) -> /ROM_LOWER
- U5 pad 24: unconnected-(U5-OE-Pad24) -> GND
- U6 pad 1: A15 -> A19
- U6 pad 10: A1 -> A3
- U6 pad 11: D0 -> A2
- U6 pad 12: D1 -> A1
- U6 pad 13: D2 -> D0
- U6 pad 14: GND -> D1
- U6 pad 15: D3 -> D2
- U6 pad 16: D4 -> GND
- U6 pad 17: D5 -> D3
- U6 pad 18: D6 -> D4
- U6 pad 19: D7 -> D5
- U6 pad 2: A13 -> A17
- U6 pad 20: unconnected-(U6-~{CS}-Pad20) -> D6
- U6 pad 21: A11 -> D7
- U6 pad 22: unconnected-(U6-~{OE}-Pad22) -> /SRAM_LOWER
- U6 pad 23: A12 -> A11
- U6 pad 24: A10 -> GND
- U6 pad 25: A9 -> A12
- U6 pad 26: A14 -> A10
- U6 pad 27: unconnected-(U6-~{WE}-Pad27) -> A9
- U6 pad 28: +5V -> A14
- U6 pad 3: A8 -> A15
- U6 pad 4: A7 -> A13
- U6 pad 5: A6 -> A8
- U6 pad 6: A5 -> A7
- U6 pad 7: A4 -> A6
- U6 pad 8: A3 -> A5
- U6 pad 9: A2 -> A4
- U7 pad 10: unconnected-(U7-/DTACK-Pad10) -> /DTACK_DUART
- U7 pad 11: unconnected-(U7-RXDB-Pad11) -> RXB
- U7 pad 13: unconnected-(U7-TXDB-Pad13) -> TXB
- U7 pad 14: unconnected-(U7-OP1-Pad14) -> /RTSB
- U7 pad 24: unconnected-(U7-INTR-Pad24) -> /IRQ_DUART
- U7 pad 32: unconnected-(U7-OP0-Pad32) -> /RTSA
- U7 pad 33: unconnected-(U7-TXDA-Pad33) -> TXA
- U7 pad 35: unconnected-(U7-RXDA-Pad35) -> RXA
- U7 pad 38: unconnected-(U7-/RESET-Pad38) -> /RESET
- U7 pad 39: unconnected-(U7-CS-Pad39) -> /DUART
- U7 pad 41: unconnected-(U7-/IACK-Pad41) -> /IACK_DUART
- U7 pad 9: unconnected-(U7-/RW-Pad9) -> R/W
Other:
- board size 160 x 100 mm -> 200 x 140 mm

Commit message: Rough layout of simplified Mack-10 prototype
Parts:
- removed J7: Conn_02x20_Odd_Even, Connector_IDC:IDC-Header_2x20_P2.54mm_Vertical
- removed JP1, JP2: Jumper_2_Open, Connector_PinHeader_2.54mm:PinHeader_1x02_P2.54mm_Vertical
- removed U10: ~, Package_LCC:PLCC-84_THT-Socket
- removed U11, U12, U13, U14: ~, mackerel:SIMM-30
- removed U16, U17: 74HC245, Package_DIP:DIP-20_W7.62mm
- added J3: Conn_02x20_Odd_Even, Connector_IDC:IDC-Header_2x20_P2.54mm_Vertical, F.Cu at (40.2, 133.6)
- J2: value DIN41612_02x32_AC -> Conn_02x20_Odd_Even; footprint Connector_DIN:DIN41612_C_2x32_Female_Vertical_THT -> Connector_IDC:IDC-Header_2x20_P2.54mm_Vertical
- moved U6 123.9 mm to (159.0, 35.0)
- moved J1 111.1 mm to (40.8, 108.6), turned to 180 degrees
- moved U4 110.7 mm to (158.5, 81.0)
- moved U3 102.3 mm to (134.0, 35.8)
- moved U5 101.5 mm to (133.5, 81.3)
- moved U2 56.9 mm to (75.5, 80.8)
- moved U7 53.6 mm to (70.5, 45.5)
- moved X1 52.1 mm to (88.8, 66.2)
- moved X2 51.4 mm to (88.4, 47.8)
- moved H4 44.7 mm to (175.0, 135.0)
- moved H2 40.0 mm to (175.0, 25.0)
- moved J5 34.5 mm to (60.2, 30.5)
- moved U1 33.1 mm to (105.4, 35.2)
- moved J2 23.7 mm to (110.4, 133.2), turned to 90 degrees
- moved H3 20.0 mm to (25.0, 135.0)
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Connections:
- net Net-(U1-BGACK) renamed /BGACK
- net Net-(U1-BR) renamed /BR
- J4 pad 3: Net-(J4-Pin_3) -> unconnected-(J4-Pin_3-Pad3)
- J5 pad 3: Net-(J5-Pin_3) -> unconnected-(J5-Pin_3-Pad3)
- R3 pad 2: IPL2 -> /IPL2
- R4 pad 2: IPL1 -> /IPL1
- R5 pad 2: IPL0 -> /IPL0
- U1 pad 11: unconnected-(U1-BG-Pad11) -> /BG
- U1 pad 23: IPL2 -> /IPL2
- U1 pad 24: IPL1 -> /IPL1
- U1 pad 25: IPL0 -> /IPL0
Other:
- board size 200 x 140 mm -> 160 x 120 mm

Commit message: Mack-10 proto routed except for expansion headers
Parts:
- removed D2: LED, LED_THT:LED_D5.0mm
- removed J4, J5: Conn_01x06, Connector_PinSocket_2.54mm:PinSocket_1x06_P2.54mm_Horizontal
- removed J8: Barrel_Jack_MountingPin, Connector_BarrelJack:BarrelJack_Horizontal
- removed U15: NE555P, Package_DIP:DIP-8_W7.62mm
- added C10: 0.1uF, Capacitor_THT:C_Disc_D4.7mm_W2.5mm_P5.00mm, F.Cu at (148.3, 110.5)
- added C11: 0.1uF, Capacitor_THT:C_Disc_D4.7mm_W2.5mm_P5.00mm, F.Cu at (156.0, 87.6)
- added C12: 0.1uF, Capacitor_THT:C_Disc_D4.7mm_W2.5mm_P5.00mm, F.Cu at (145.8, 69.8)
- added C13: 0.1uF, Capacitor_THT:C_Disc_D4.7mm_W2.5mm_P5.00mm, F.Cu at (115.6, 56.1)
- added C14: 0.1uF, Capacitor_THT:C_Disc_D4.7mm_W2.5mm_P5.00mm, F.Cu at (38.2, 65.4)
- added C15: 0.1uF, Capacitor_THT:C_Disc_D4.7mm_W2.5mm_P5.00mm, F.Cu at (60.2, 64.8)
- added C16: 0.1uF, Capacitor_THT:C_Disc_D4.7mm_W2.5mm_P5.00mm, F.Cu at (82.2, 65.0)
- added C17: 0.1uF, Capacitor_THT:C_Disc_D4.7mm_W2.5mm_P5.00mm, F.Cu at (104.2, 64.9)
- added C18: 0.1uF, Capacitor_THT:C_Disc_D4.7mm_W2.5mm_P5.00mm, F.Cu at (131.1, 23.5)
- added C19: 0.1uF, Capacitor_THT:C_Disc_D4.7mm_W2.5mm_P5.00mm, F.Cu at (139.1, 56.1)
- added C2: 0.1uF, Capacitor_THT:C_Disc_D4.7mm_W2.5mm_P5.00mm, F.Cu at (62.0, 29.8)
- added C20: 0.1uF, Capacitor_THT:C_Disc_D4.7mm_W2.5mm_P5.00mm, F.Cu at (166.1, 37.5)
- added C3: C_Polarized, Capacitor_THT:CP_Radial_D5.0mm_P2.50mm, F.Cu at (164.8, 32.6)
- added C5: 0.1uF, Capacitor_THT:C_Disc_D4.7mm_W2.5mm_P5.00mm, F.Cu at (133.1, 69.8)
- added C6: 0.1uF, Capacitor_THT:C_Disc_D4.7mm_W2.5mm_P5.00mm, F.Cu at (122.9, 69.8)
- added C7: 0.1uF, Capacitor_THT:C_Disc_D4.7mm_W2.5mm_P5.00mm, F.Cu at (115.2, 95.2)
- added C8: 0.1uF, Capacitor_THT:C_Disc_D4.7mm_W2.5mm_P5.00mm, F.Cu at (128.0, 110.5)
- added C9: 0.1uF, Capacitor_THT:C_Disc_D4.7mm_W2.5mm_P5.00mm, F.Cu at (135.6, 110.5)
- added D3: LED, LED_THT:LED_D5.0mm, F.Cu at (162.9, 104.5)
- added J10: Conn_01x06, Connector_PinHeader_2.54mm:PinHeader_1x06_P2.54mm_Vertical, F.Cu at (93.6, 22.6)
- added J6: Barrel_Jack_MountingPin, Connector_BarrelJack:BarrelJack_Horizontal, F.Cu at (156.5, 34.0)
- added J9: Conn_01x06, Connector_PinHeader_2.54mm:PinHeader_1x06_P2.54mm_Vertical, F.Cu at (113.5, 22.6)
- added R14: R, Resistor_THT:R_Axial_DIN0204_L3.6mm_D1.6mm_P5.08mm_Horizontal, F.Cu at (144.0, 32.5)
- added U9: NE555P, Package_DIP:DIP-8_W7.62mm, F.Cu at (158.5, 40.9)
- C1: value C_Polarized -> 1000uF; footprint Capacitor_THT:CP_Radial_D5.0mm_P2.50mm -> Capacitor_THT:CP_Radial_D10.0mm_P5.00mm
- C4: value 1000uF -> 0.1uF; footprint Capacitor_THT:CP_Radial_D10.0mm_P5.00mm -> Capacitor_THT:C_Disc_D4.7mm_W2.5mm_P5.00mm
- R10, R11, R12, R13: footprint Resistor_THT:R_Axial_DIN0207_L6.3mm_D2.5mm_P7.62mm_Horizontal -> Resistor_THT:R_Axial_DIN0204_L3.6mm_D1.6mm_P5.08mm_Horizontal
- X2: value 3.6864 MHz -> 3.6864MHz
- moved R9 242.1 mm to (161.9, 97.8)
- moved R8 242.1 mm to (161.9, 95.3)
- moved R7 242.0 mm to (161.8, 92.9)
- moved R6 241.9 mm to (161.8, 90.4)
- moved D1 211.0 mm to (162.8, 115.2)
- moved R10 210.5 mm to (159.4, 117.8), turned to 90 degrees
- moved R5 201.6 mm to (113.9, 40.1), turned to 180 degrees
- moved R4 201.5 mm to (113.9, 37.6), turned to 180 degrees
- moved R3 201.3 mm to (113.9, 35.1), turned to 180 degrees
- moved R13 188.0 mm to (159.5, 107.0), turned to 90 degrees
- moved R11 156.1 mm to (164.9, 53.7), turned to 180 degrees
- moved SW1 147.4 mm to (159.1, 57.8)
- moved R12 141.4 mm to (164.9, 51.3), turned to 180 degrees
- moved C1 134.6 mm to (146.5, 42.8)
- moved R2 131.6 mm to (49.9, 64.8), turned to 180 degrees
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Connections:
- C1 pad 2: Net-(U15-THR) -> GND
- D1 pad 1: /RESET -> GND
- R10 pad 2: Net-(U15-R) -> Net-(D1-A)
- R11 pad 1: Net-(U15-THR) -> +5V
- R11 pad 2: GND -> Net-(U9-R)
- R12 pad 1: +5V -> Net-(U9-THR)
- R12 pad 2: Net-(D1-A) -> GND
- SW1 pad 2: Net-(U15-R) -> Net-(U9-R)
- U2 pad 10: /ROM_LOWER -> A16
- U2 pad 11: /DUART -> A17
- U2 pad 12: /DTACK_DUART -> A15
- U2 pad 15: /IRQ_DUART -> A18
- U2 pad 16: /IACK_DUART -> A14
- U2 pad 17: unconnected-(U2-IO-Pad17) -> R/W
- U2 pad 18: unconnected-(U2-IO-Pad18) -> A4
- U2 pad 2: unconnected-(U2-OE2/GCLK2-Pad2) -> GND
- U2 pad 20: unconnected-(U2-IO-Pad20) -> A3
- U2 pad 21: unconnected-(U2-IO-Pad21) -> A2
- U2 pad 22: unconnected-(U2-IO-Pad22) -> /SRAM_LOWER
- U2 pad 24: unconnected-(U2-IO-Pad24) -> A1
- U2 pad 25: FC0 -> D7
- U2 pad 27: FC1 -> D0
- U2 pad 28: FC2 -> D6
- U2 pad 29: /VPA -> D1
- U2 pad 30: /BERR -> D5
- U2 pad 31: /DTACK -> D2
- U2 pad 33: A16 -> D3
- U2 pad 34: A17 -> D4
- U2 pad 35: A18 -> /SRAM_UPPER
- U2 pad 36: A19 -> /ROM_LOWER
- U2 pad 37: A20 -> /ROM_UPPER
- U2 pad 39: A21 -> unconnected-(U2-IO-Pad39)
- U2 pad 4: CLK_CPU -> /IPL2
- U2 pad 40: A22 -> unconnected-(U2-IO-Pad40)
- U2 pad 41: A23 -> unconnected-(U2-IO-Pad41)
- U2 pad 5: /RESET -> /BERR
- U2 pad 58: unconnected-(U2-IO-Pad58) -> /IRQ_DUART
- U2 pad 6: /SRAM_UPPER -> /VPA
- U2 pad 60: unconnected-(U2-IO-Pad60) -> /DTACK_DUART
- U2 pad 61: unconnected-(U2-IO-Pad61) -> /IACK_DUART
- U2 pad 63: unconnected-(U2-IO-Pad63) -> /DUART
- U2 pad 64: unconnected-(U2-IO-Pad64) -> A20
- U2 pad 65: unconnected-(U2-IO-Pad65) -> A21
- U2 pad 67: unconnected-(U2-IO-Pad67) -> A22
- U2 pad 68: unconnected-(U2-IO-Pad68) -> A23
- U2 pad 69: unconnected-(U2-IO-Pad69) -> /AS
- U2 pad 70: unconnected-(U2-IO-Pad70) -> /UDS
- U2 pad 73: unconnected-(U2-IO-Pad73) -> /LDS
- U2 pad 74: /AS -> /DTACK
- U2 pad 75: /UDS -> CLK_CPU
- U2 pad 76: /LDS -> FC0
- U2 pad 77: R/W -> FC1
- U2 pad 79: /IPL0 -> FC2
- U2 pad 8: /SRAM_LOWER -> /RESET
- U2 pad 80: /IPL1 -> /IPL0
- U2 pad 81: /IPL2 -> /IPL1
- U2 pad 9: /ROM_UPPER -> A19
- U7 pad 14: /RTSB -> unconnected-(U7-OP1-Pad14)
- U7 pad 32: /RTSA -> unconnected-(U7-OP0-Pad32)
Routing:
- net D5: track 0.00 -> 272.4 mm, vias 0 -> 4
- net D6: track 0.00 -> 270.3 mm, vias 0 -> 4
- net D4: track 0.00 -> 265.2 mm, vias 0 -> 3
- net D2: track 0.00 -> 259.5 mm, vias 0 -> 3
- net D7: track 0.00 -> 256.2 mm, vias 0 -> 4
- net D3: track 0.00 -> 253.6 mm, vias 0 -> 3
- net D0: track 0.00 -> 247.1 mm, vias 0 -> 3
- net D1: track 0.00 -> 242.8 mm, vias 0 -> 3
- net A1: track 0.00 -> 201.5 mm, vias 0 -> 2
- net A2: track 0.00 -> 197.1 mm, vias 0 -> 2
- net /RESET: track 0.00 -> 196.7 mm, vias 0 -> 3
- net R/W: track 0.00 -> 196.6 mm, vias 0 -> 4
- net A3: track 0.00 -> 185.2 mm, vias 0 -> 2
- net A4: track 0.00 -> 174.1 mm, vias 0 -> 2
- net A21: track 0.00 -> 157.7 mm, vias 0 -> 1
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- added copper zone on In2.Cu, net +5V
- added copper zone on In1.Cu, net GND
Other:
- board size 160 x 120 mm -> 150 x 120 mm
- copper layers 2 -> 4
- board text added: "5V"
- board text added: "MACKEREL-10 SBC Proto"
- board text added: "RAM LOWER"
- board text added: "RAM UPPER"
- board text added: "ROM LOWER"
- board text added: "ROM UPPER"
- board text added: "RST"
- board text added: "github.com/crmaykish/mackerel-68k Colin Maykish - 2024"

Commit message: Mack-10 proto fully routed
Parts:
- added C21: 1000uF, Capacitor_THT:CP_Radial_D8.0mm_P3.50mm, F.Cu at (22.9, 120.0)
- added C22: 1000uF, Capacitor_THT:CP_Radial_D8.0mm_P3.50mm, F.Cu at (92.3, 124.7)
- moved H3 6.00 mm to (24.0, 130.0)
- moved H4 6.00 mm to (166.0, 130.0)
- moved J2 6.00 mm to (35.0, 126.0)
- moved J3 6.00 mm to (105.0, 126.0)
Connections:
- net /BGACK renamed Net-(U1-BGACK)
- net /BR renamed Net-(U1-BR)
- J2 pad 1: unconnected-(J2-Pin_1-Pad1) -> +5V
- J2 pad 10: unconnected-(J2-Pin_10-Pad10) -> D13
- J2 pad 11: unconnected-(J2-Pin_11-Pad11) -> D14
- J2 pad 12: unconnected-(J2-Pin_12-Pad12) -> D15
- J2 pad 13: unconnected-(J2-Pin_13-Pad13) -> A1
- J2 pad 14: unconnected-(J2-Pin_14-Pad14) -> A2
- J2 pad 15: unconnected-(J2-Pin_15-Pad15) -> A3
- J2 pad 16: unconnected-(J2-Pin_16-Pad16) -> A4
- J2 pad 17: unconnected-(J2-Pin_17-Pad17) -> A5
- J2 pad 18: unconnected-(J2-Pin_18-Pad18) -> A6
- J2 pad 19: unconnected-(J2-Pin_19-Pad19) -> A7
- J2 pad 2: unconnected-(J2-Pin_2-Pad2) -> +5V
- J2 pad 20: unconnected-(J2-Pin_20-Pad20) -> A8
- J2 pad 21: unconnected-(J2-Pin_21-Pad21) -> GND
- J2 pad 22: unconnected-(J2-Pin_22-Pad22) -> GND
- J2 pad 23: unconnected-(J2-Pin_23-Pad23) -> A23
- J2 pad 24: unconnected-(J2-Pin_24-Pad24) -> A22
- J2 pad 25: unconnected-(J2-Pin_25-Pad25) -> A21
- J2 pad 26: unconnected-(J2-Pin_26-Pad26) -> A20
- J2 pad 27: unconnected-(J2-Pin_27-Pad27) -> A9
- J2 pad 28: unconnected-(J2-Pin_28-Pad28) -> A10
- J2 pad 29: unconnected-(J2-Pin_29-Pad29) -> A11
- J2 pad 3: unconnected-(J2-Pin_3-Pad3) -> GND
- J2 pad 30: unconnected-(J2-Pin_30-Pad30) -> A12
- J2 pad 31: unconnected-(J2-Pin_31-Pad31) -> A13
- J2 pad 32: unconnected-(J2-Pin_32-Pad32) -> A14
- J2 pad 33: unconnected-(J2-Pin_33-Pad33) -> A15
- J2 pad 34: unconnected-(J2-Pin_34-Pad34) -> A16
- J2 pad 35: unconnected-(J2-Pin_35-Pad35) -> A17
- J2 pad 36: unconnected-(J2-Pin_36-Pad36) -> A18
- J2 pad 37: unconnected-(J2-Pin_37-Pad37) -> A19
- J2 pad 39: unconnected-(J2-Pin_39-Pad39) -> GND
- J2 pad 4: unconnected-(J2-Pin_4-Pad4) -> GND
- J2 pad 40: unconnected-(J2-Pin_40-Pad40) -> GND
- J2 pad 5: unconnected-(J2-Pin_5-Pad5) -> D8
- J2 pad 6: unconnected-(J2-Pin_6-Pad6) -> D9
- J2 pad 7: unconnected-(J2-Pin_7-Pad7) -> D10
- J2 pad 8: unconnected-(J2-Pin_8-Pad8) -> D11
- J2 pad 9: unconnected-(J2-Pin_9-Pad9) -> D12
- J3 pad 1: unconnected-(J3-Pin_1-Pad1) -> +5V
- J3 pad 10: unconnected-(J3-Pin_10-Pad10) -> D5
- J3 pad 11: unconnected-(J3-Pin_11-Pad11) -> D6
- J3 pad 12: unconnected-(J3-Pin_12-Pad12) -> D7
- J3 pad 13: unconnected-(J3-Pin_13-Pad13) -> /AS
- J3 pad 14: unconnected-(J3-Pin_14-Pad14) -> R/W
- J3 pad 15: unconnected-(J3-Pin_15-Pad15) -> /UDS
- J3 pad 16: unconnected-(J3-Pin_16-Pad16) -> /LDS
- J3 pad 17: unconnected-(J3-Pin_17-Pad17) -> /BERR
- J3 pad 18: unconnected-(J3-Pin_18-Pad18) -> /VPA
- J3 pad 19: unconnected-(J3-Pin_19-Pad19) -> /EXP
- J3 pad 2: unconnected-(J3-Pin_2-Pad2) -> +5V
- J3 pad 20: unconnected-(J3-Pin_20-Pad20) -> /IRQ_EXP
- J3 pad 21: unconnected-(J3-Pin_21-Pad21) -> /DTACK_EXP
- J3 pad 22: unconnected-(J3-Pin_22-Pad22) -> /IACK_EXP
- J3 pad 23: unconnected-(J3-Pin_23-Pad23) -> GND
- J3 pad 24: unconnected-(J3-Pin_24-Pad24) -> GND
- J3 pad 25: unconnected-(J3-Pin_25-Pad25) -> GPIO_0
- J3 pad 26: unconnected-(J3-Pin_26-Pad26) -> GPIO_1
- J3 pad 27: unconnected-(J3-Pin_27-Pad27) -> GPIO_2
- J3 pad 28: unconnected-(J3-Pin_28-Pad28) -> GPIO_3
- J3 pad 29: unconnected-(J3-Pin_29-Pad29) -> GPIO_4
- J3 pad 3: unconnected-(J3-Pin_3-Pad3) -> GND
- J3 pad 30: unconnected-(J3-Pin_30-Pad30) -> GPIO_5
- J3 pad 31: unconnected-(J3-Pin_31-Pad31) -> GPIO_6
- J3 pad 32: unconnected-(J3-Pin_32-Pad32) -> GPIO_7
- J3 pad 33: unconnected-(J3-Pin_33-Pad33) -> GND
- J3 pad 34: unconnected-(J3-Pin_34-Pad34) -> GND
- J3 pad 35: unconnected-(J3-Pin_35-Pad35) -> CLK_CPU
- J3 pad 36: unconnected-(J3-Pin_36-Pad36) -> CLK_SRC
- J3 pad 37: unconnected-(J3-Pin_37-Pad37) -> /RESET
- J3 pad 38: unconnected-(J3-Pin_38-Pad38) -> /RESET
- J3 pad 39: unconnected-(J3-Pin_39-Pad39) -> GND
- J3 pad 4: unconnected-(J3-Pin_4-Pad4) -> GND
- J3 pad 40: unconnected-(J3-Pin_40-Pad40) -> GND
- J3 pad 5: unconnected-(J3-Pin_5-Pad5) -> D0
- J3 pad 6: unconnected-(J3-Pin_6-Pad6) -> D1
- J3 pad 7: unconnected-(J3-Pin_7-Pad7) -> D2
- J3 pad 8: unconnected-(J3-Pin_8-Pad8) -> D3
- J3 pad 9: unconnected-(J3-Pin_9-Pad9) -> D4
- U1 pad 11: /BG -> unconnected-(U1-BG-Pad11)
- U2 pad 39: unconnected-(U2-IO-Pad39) -> /IRQ_EXP
- U2 pad 40: unconnected-(U2-IO-Pad40) -> /EXP
- U2 pad 41: unconnected-(U2-IO-Pad41) -> /IACK_EXP
- U2 pad 44: unconnected-(U2-IO-Pad44) -> /DTACK_EXP
- U2 pad 45: unconnected-(U2-IO-Pad45) -> GPIO_1
- U2 pad 46: unconnected-(U2-IO-Pad46) -> GPIO_0
- U2 pad 48: unconnected-(U2-IO-Pad48) -> GPIO_2
- U2 pad 49: unconnected-(U2-IO-Pad49) -> GPIO_3
- U2 pad 50: unconnected-(U2-IO-Pad50) -> GPIO_4
- U2 pad 51: unconnected-(U2-IO-Pad51) -> GPIO_5
- U2 pad 52: unconnected-(U2-IO-Pad52) -> GPIO_6
- U2 pad 54: unconnected-(U2-IO-Pad54) -> GPIO_7
- U2 pad 83: /CLK_SRC -> CLK_SRC
- X1 pad 5: /CLK_SRC -> CLK_SRC
Routing:
- net CLK_SRC: track 0.00 -> 82.4 mm
- net /AS: track 145.7 -> 227.4 mm, vias 0 -> 1
- net /UDS: track 137.2 -> 217.7 mm, vias 0 -> 1
- net A20: track 152.1 -> 232.3 mm
- net A21: track 157.7 -> 236.5 mm
- net A23: track 150.9 -> 228.9 mm
- net /LDS: track 133.3 -> 208.0 mm, vias 0 -> 1
- net A22: track 156.1 -> 230.9 mm
- net /BERR: track 61.2 -> 128.9 mm, vias 0 -> 1
- net /VPA: track 65.7 -> 128.5 mm, vias 0 -> 1
- net A19: track 148.1 -> 208.2 mm, vias 1 -> 2
- net A15: track 149.5 -> 208.5 mm, vias 4 -> 5
- net CLK_CPU: track 98.1 -> 156.8 mm
- net A13: track 116.3 -> 174.5 mm, vias 1 -> 2
- net A17: track 147.6 -> 204.9 mm, vias 1 -> 2
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Other:
- board size 150 x 120 mm -> 150 x 114 mm
- board text added: "5VDC"
- board text added: "GND"
- board text added: "RXA"
- board text added: "RXB"
- board text added: "TXA"
- board text added: "TXB"
