File: hardware/mackerel-10-v1/mackerel-10-v1.kicad_pcb (KiCad board)
At the start: 2 copper layers, 170 x 170 mm, 58 parts, among them J1 Conn_02x05_Odd_Even, J2 Conn_01x06, J3 Conn_01x06, J4 Conn_01x10, J5 Conn_02x05_Odd_Even, J6 Conn_02x20_Odd_Even, SW1 SW_Push, U1 68010D, U12 74HC245, U13 74HC245, U3 SST39SF040, U4 AS6C4008-55PCN, U5 SST39SF040, U6 AS6C4008-55PCN, U7 XR68C681, U8 NE555P, X1 50MHz, X2 3.6864MHz

Commit message: Rough layout of components on PCB
Parts:
- removed R33, R34, R35, R36: R, Resistor_THT:R_Axial_DIN0207_L6.3mm_D2.5mm_P7.62mm_Horizontal
- added C10: 0.1uF, Capacitor_THT:C_Disc_D4.7mm_W2.5mm_P5.00mm, F.Cu at (-30.7, 174.6)
- added C11: 1000uF, Capacitor_THT:CP_Radial_D8.0mm_P3.50mm, F.Cu at (-20.0, 11.0)
- added C12: 1000uF, Capacitor_THT:CP_Radial_D8.0mm_P3.50mm, F.Cu at (-20.0, 20.5)
- added C9: C_Polarized, Capacitor_THT:CP_Radial_D5.0mm_P2.50mm, F.Cu at (-102.8, 241.0)
- added HS1: Heatsink, Heatsink:Heatsink_Stonecold_HS-S02_13.21x9.53mm, F.Cu at (53.0, -25.4)
- added J10: Conn_02x20_Odd_Even, Connector_IDC:IDC-Header_2x20_P2.54mm_Vertical, F.Cu at (41.9, 162.6)
- added J11: Conn_02x20_Odd_Even, Connector_IDC:IDC-Header_2x20_P2.54mm_Vertical, F.Cu at (107.5, 162.1)
- added J12: DE9_Receptacle_MountingHoles, Connector_Dsub:DSUB-9_Female_Horizontal_P2.77x2.84mm_EdgePinOffset7.70mm_Housed_MountingHolesOffset9.12mm, F.Cu at (32.3, 78.2)
- added J13: DE9_Receptacle_MountingHoles, Connector_Dsub:DSUB-9_Female_Horizontal_P2.77x2.84mm_EdgePinOffset7.70mm_Housed_MountingHolesOffset9.12mm, F.Cu at (31.8, 115.6)
- added J14: Screw_Terminal_01x04, TerminalBlock:TerminalBlock_bornier-4_P5.08mm, F.Cu at (250.2, 149.9)
- added J7: Conn_02x03_Odd_Even, Connector_PinHeader_2.54mm:PinHeader_2x03_P2.54mm_Vertical, F.Cu at (-49.2, 165.2)
- added J8: Conn_02x03_Odd_Even, Connector_PinHeader_2.54mm:PinHeader_2x03_P2.54mm_Vertical, F.Cu at (-42.0, 165.2)
- added J9: Conn_02x03_Odd_Even, Connector_PinHeader_2.54mm:PinHeader_2x03_P2.54mm_Vertical, F.Cu at (-34.8, 165.2)
- added L1: 100uH, Inductor_THT:L_Radial_D10.0mm_P5.00mm_Fastron_07M, F.Cu at (36.5, -32.7)
- added R17: R, Resistor_THT:R_Axial_DIN0207_L6.3mm_D2.5mm_P7.62mm_Horizontal, F.Cu at (-71.1, 47.5)
- added R18: R, Resistor_THT:R_Axial_DIN0207_L6.3mm_D2.5mm_P7.62mm_Horizontal, F.Cu at (-169.9, 194.7)
- added R19: R, Resistor_THT:R_Axial_DIN0207_L6.3mm_D2.5mm_P7.62mm_Horizontal, F.Cu at (-169.9, 198.7)
- added R20: 1k, Resistor_THT:R_Axial_DIN0207_L6.3mm_D2.5mm_P7.62mm_Horizontal, F.Cu at (-34.2, 261.6)
- added R21: R, Resistor_THT:R_Axial_DIN0207_L6.3mm_D2.5mm_P7.62mm_Horizontal, F.Cu at (-117.6, 255.2)
- added R22: R, Resistor_THT:R_Axial_DIN0207_L6.3mm_D2.5mm_P7.62mm_Horizontal, F.Cu at (-117.6, 259.3)
- added R23: R, Resistor_THT:R_Axial_DIN0207_L6.3mm_D2.5mm_P7.62mm_Horizontal, F.Cu at (-21.3, 226.0)
- added U14: XR68C681, Package_LCC:PLCC-44_THT-Socket, F.Cu at (57.1, 105.4)
- added U15: LM2576T-5, Package_TO_SOT_THT:TO-220-5_Vertical, F.Cu at (50.2, -33.6)
- added U16: NE555P, Package_DIP:DIP-8_W7.62mm, F.Cu at (-99.9, 256.0)
- added U17: MAX3232, Package_DIP:DIP-16_W7.62mm_Socket, F.Cu at (-28.8, 68.8)
- added U18: MAX3232, Package_DIP:DIP-16_W7.62mm_Socket, F.Cu at (-17.1, 68.8)
- added X3: 3.6864MHz, Oscillator:Oscillator_DIP-8, F.Cu at (56.1, 91.2)
- C7: value C_Polarized -> 1000uF; footprint Capacitor_THT:CP_Radial_D5.0mm_P2.50mm -> Capacitor_THT:CP_Radial_D10.0mm_P5.00mm
- C8: value 0.1uF -> 1000uF; footprint Capacitor_THT:C_Disc_D4.7mm_W2.5mm_P5.00mm -> Capacitor_THT:CP_Radial_D10.0mm_P5.00mm
- D3: value LED -> 1N5822; footprint LED_THT:LED_D5.0mm -> Diode_THT:D_DO-27_P15.24mm_Horizontal
- J2: value Conn_01x06 -> Conn_02x05_Odd_Even; footprint Connector_PinHeader_2.54mm:PinHeader_1x06_P2.54mm_Vertical -> Connector_IDC:IDC-Header_2x05_P2.54mm_Vertical
- J3: value Conn_01x06 -> Conn_02x20_Odd_Even; footprint Connector_PinHeader_2.54mm:PinHeader_1x06_P2.54mm_Vertical -> Connector_IDC:IDC-Header_2x20_P2.54mm_Vertical
- J4: value Conn_01x10 -> Conn_01x06; footprint Connector_PinSocket_2.54mm:PinSocket_1x10_P2.54mm_Vertical -> Connector_PinHeader_2.54mm:PinHeader_1x06_P2.54mm_Vertical
- J5: value Conn_02x05_Odd_Even -> Conn_01x06; footprint Connector_IDC:IDC-Header_2x05_P2.54mm_Vertical -> Connector_PinHeader_2.54mm:PinHeader_1x06_P2.54mm_Vertical
- J6: value Conn_02x20_Odd_Even -> Barrel_Jack_MountingPin; footprint Connector_IDC:IDC-Header_2x20_P2.54mm_Vertical -> Connector_BarrelJack:BarrelJack_Horizontal
- R1, R10, R11, R12, R13, R2, R3, R4, R5, R6, R7, R8, R9: footprint Resistor_THT:R_Axial_DIN0204_L3.6mm_D1.6mm_P5.08mm_Horizontal -> Resistor_THT:R_Axial_DIN0207_L6.3mm_D2.5mm_P7.62mm_Horizontal
- R14, R15: value R -> 4k7; footprint Resistor_THT:R_Axial_DIN0204_L3.6mm_D1.6mm_P5.08mm_Horizontal -> Resistor_THT:R_Axial_DIN0207_L6.3mm_D2.5mm_P7.62mm_Horizontal
- R16: value R -> 470; footprint Resistor_THT:R_Axial_DIN0204_L3.6mm_D1.6mm_P5.08mm_Horizontal -> Resistor_THT:R_Axial_DIN0207_L6.3mm_D2.5mm_P7.62mm_Horizontal
- U7: value XR68C681 -> ~; footprint Package_LCC:PLCC-44_THT-Socket -> mackerel:SIMM-30
- U8: value NE555P -> ~; footprint Package_DIP:DIP-8_W7.62mm -> mackerel:SIMM-30
- X2: value 3.6864MHz -> 50MHz; footprint Oscillator:Oscillator_DIP-8 -> Oscillator:Oscillator_DIP-14
- moved H4 313.0 mm to (236.0, 156.0)
- moved H2 294.2 mm to (236.0, 24.0)
- moved J3 229.0 mm to (172.2, 162.3), turned to 90 degrees
- moved D3 225.4 mm to (41.9, -61.6)
- moved SW1 207.9 mm to (-92.2, 238.9)
- moved U8 196.4 mm to (143.7, 32.3), turned to 180 degrees
- moved J6 184.0 mm to (79.1, -26.8)
- moved D4 183.3 mm to (-17.3, 218.4)
- moved R10 180.5 mm to (-211.8, 58.9)
- moved R11 180.3 mm to (-211.8, 63.0)
- moved R12 180.0 mm to (-211.8, 67.0)
- moved R6 178.5 mm to (-215.9, 91.4)
- moved R9 178.5 mm to (-215.9, 103.5)
- moved R7 178.5 mm to (-215.9, 95.5)
- moved R8 178.5 mm to (-215.9, 99.5)
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Connections:
- C7 pad 1: +5V -> VCC
- C7 pad 2: Net-(U8-THR) -> GND
- D1 pad 1: GND -> Net-(D1-K)
- D1 pad 2: USR2 -> Net-(D1-A)
- D2 pad 2: USR1 -> Net-(D2-A)
- D3 pad 1: GND -> Net-(D3-K)
- D3 pad 2: USR0 -> GND
- J2 pad 1: GND -> TCK_DRAM
- J2 pad 2: unconnected-(J2-Pin_2-Pad2) -> GND
- J2 pad 3: unconnected-(J2-Pin_3-Pad3) -> TDO_DRAM
- J2 pad 4: RXA -> +5V
- J2 pad 5: TXA -> TMS_DRAM
- J3 pad 1: GND -> /RESET
- J3 pad 2: unconnected-(J3-Pin_2-Pad2) -> GND
- J3 pad 3: unconnected-(J3-Pin_3-Pad3) -> IDE_D7
- J3 pad 4: RXB -> IDE_D8
- J3 pad 5: TXB -> IDE_D6
- J3 pad 6: unconnected-(J3-Pin_6-Pad6) -> IDE_D9
- J4 pad 1: Net-(J4-Pin_1) -> GND
- J4 pad 2: Net-(J4-Pin_2) -> unconnected-(J4-Pin_2-Pad2)
- J4 pad 3: Net-(J4-Pin_3) -> unconnected-(J4-Pin_3-Pad3)
- J4 pad 4: Net-(J4-Pin_4) -> RXA
- J4 pad 5: Net-(J4-Pin_5) -> TXA
- J4 pad 6: Net-(J4-Pin_6) -> unconnected-(J4-Pin_6-Pad6)
- J5 pad 1: TCK -> GND
- J5 pad 2: GND -> unconnected-(J5-Pin_2-Pad2)
- J5 pad 3: TDO -> unconnected-(J5-Pin_3-Pad3)
- J5 pad 4: +5V -> RXB
- J5 pad 5: TMS -> TXB
- J6 pad 1: /RESET -> VCC
- J6 pad 3: IDE_D7 -> (no net)
- R10 pad 2: TMS -> TDO_DRAM
- R11 pad 2: TDI -> TMS_DRAM
- R12 pad 1: TCK -> +5V
- R12 pad 2: GND -> TDI_DRAM
- R13 pad 1: /IACK_DUART -> TCK_DRAM
- R13 pad 2: +5V -> GND
- R14 pad 1: +5V -> GND
- R14 pad 2: Net-(U8-R) -> IDE_RDY
- R15 pad 1: Net-(U8-THR) -> GND
- R15 pad 2: GND -> IDE_INT
- R16 pad 2: Net-(D4-A) -> Net-(D1-A)
- R6 pad 1: Net-(R6-Pad1) -> +5V
- R6 pad 2: USR0 -> TDO
- R7 pad 1: Net-(R7-Pad1) -> +5V
- R7 pad 2: USR1 -> TMS
- R8 pad 1: Net-(R8-Pad1) -> +5V
- R8 pad 2: USR2 -> TDI
- R9 pad 1: +5V -> TCK
- R9 pad 2: TDO -> GND
- SW1 pad 2: Net-(U8-R) -> Net-(U16-R)
- U10 pad 10: /DRAM/RAM_D10 -> D10
- U10 pad 13: /DRAM/RAM_D11 -> D11
- U10 pad 16: /DRAM/RAM_D12 -> D12
- U10 pad 20: /DRAM/RAM_D13 -> D13
- U10 pad 23: /DRAM/RAM_D14 -> D14
- U10 pad 25: /DRAM/RAM_D15 -> D15
- U10 pad 3: /DRAM/RAM_D8 -> D8
- U10 pad 6: /DRAM/RAM_D9 -> D9
- U11 pad 14: TDI -> TDI_DRAM
- U11 pad 2: GND -> unconnected-(U11-OE2/GCLK2-Pad2)
- U11 pad 22: Net-(J4-Pin_1) -> unconnected-(U11-IO-Pad22)
- U11 pad 23: TMS -> TMS_DRAM
- U11 pad 24: Net-(J4-Pin_2) -> unconnected-(U11-IO-Pad24)
- U11 pad 25: Net-(J4-Pin_3) -> unconnected-(U11-IO-Pad25)
- U11 pad 27: Net-(J4-Pin_4) -> unconnected-(U11-IO-Pad27)
- U11 pad 28: Net-(J4-Pin_5) -> unconnected-(U11-IO-Pad28)
- U11 pad 29: Net-(J4-Pin_6) -> unconnected-(U11-IO-Pad29)
- U11 pad 30: Net-(J4-Pin_7) -> unconnected-(U11-IO-Pad30)
- U11 pad 31: Net-(J4-Pin_8) -> unconnected-(U11-IO-Pad31)
- U11 pad 40: /DTACK_EXP -> unconnected-(U11-IO-Pad40)
- U11 pad 41: /EXP -> unconnected-(U11-IO-Pad41)
- U11 pad 62: TCK -> TCK_DRAM
- U11 pad 71: TDO -> TDO_DRAM
- U11 pad 83: CLK_SRC -> unconnected-(U11-GCLK1-Pad83)
- U2 pad 55: Net-(R6-Pad1) -> unconnected-(U2-IO-Pad55)
- U2 pad 56: Net-(R7-Pad1) -> unconnected-(U2-IO-Pad56)
- U2 pad 57: Net-(R8-Pad1) -> unconnected-(U2-IO-Pad57)
- U7 pad 10: /DTACK_DUART -> unconnected-(U7-DQ2-Pad10)
- U7 pad 11: RXB -> unconnected-(U7-A4-Pad11)
- U7 pad 13: TXB -> unconnected-(U7-DQ3-Pad13)
- U7 pad 18: D1 -> unconnected-(U7-A9-Pad18)
- U7 pad 19: D3 -> unconnected-(U7-A10-Pad19)
- U7 pad 2: A1 -> unconnected-(U7-/CAS-Pad2)
- U7 pad 20: D5 -> unconnected-(U7-DQ5-Pad20)
- U7 pad 21: D7 -> unconnected-(U7-/WE-Pad21)
- U7 pad 22: GND -> unconnected-(U7-GND-Pad22)
- U7 pad 24: /IRQ_DUART -> unconnected-(U7-A11-Pad24)
- U7 pad 25: D6 -> unconnected-(U7-DQ7-Pad25)
- U7 pad 26: D4 -> unconnected-(U7-QP-Pad26)
- U7 pad 27: D2 -> unconnected-(U7-/RAS-Pad27)
- U7 pad 28: D0 -> unconnected-(U7-/CASP-Pad28)
- U7 pad 3: GND -> unconnected-(U7-DQ0-Pad3)
- U7 pad 4: A2 -> unconnected-(U7-A0-Pad4)
- U7 pad 5: GND -> unconnected-(U7-A1-Pad5)
- U7 pad 6: A3 -> unconnected-(U7-DQ1-Pad6)
- U7 pad 7: A4 -> unconnected-(U7-A2-Pad7)
- U7 pad 8: GND -> unconnected-(U7-A3-Pad8)
- U7 pad 9: R/W -> unconnected-(U7-GND-Pad9)
- U8 pad 1: GND -> unconnected-(U8-VCC-Pad1)
- U8 pad 2: Net-(U8-THR) -> unconnected-(U8-/CAS-Pad2)
- U8 pad 3: /RESET -> unconnected-(U8-DQ0-Pad3)
- U8 pad 4: Net-(U8-R) -> unconnected-(U8-A0-Pad4)
- U8 pad 6: Net-(U8-THR) -> unconnected-(U8-DQ1-Pad6)
- U8 pad 8: +5V -> unconnected-(U8-A3-Pad8)
- U9 pad 10: /DRAM/RAM_D2 -> D2
- U9 pad 13: /DRAM/RAM_D3 -> D3
- U9 pad 16: /DRAM/RAM_D4 -> D4
- U9 pad 20: /DRAM/RAM_D5 -> D5
- U9 pad 23: /DRAM/RAM_D6 -> D6
- U9 pad 25: /DRAM/RAM_D7 -> D7
- U9 pad 3: /DRAM/RAM_D0 -> D0
- U9 pad 6: /DRAM/RAM_D1 -> D1
- X2 pad 8: +5V -> unconnected-(X2-OUT-Pad8)
Other:
- board size 170 x 170 mm -> 220 x 150 mm

Commit message: Settled on mini ITX form factor
Parts:
- removed C11, C12: 1000uF, Capacitor_THT:CP_Radial_D8.0mm_P3.50mm
- removed J11: Conn_02x20_Odd_Even, Connector_IDC:IDC-Header_2x20_P2.54mm_Vertical
- removed J12, J13: DE9_Receptacle_MountingHoles, Connector_Dsub:DSUB-9_Female_Horizontal_P2.77x2.84mm_EdgePinOffset7.70mm_Housed_MountingHolesOffset9.12mm
- removed U17, U18: MAX3232, Package_DIP:DIP-16_W7.62mm_Socket
- removed U7, U8: ~, mackerel:SIMM-30
- added G***: LOGO, LOGO, F.Cu at (15.7, 21.6)
- J4, J5: footprint Connector_PinHeader_2.54mm:PinHeader_1x06_P2.54mm_Vertical -> Connector_PinSocket_2.54mm:PinSocket_1x06_P2.54mm_Horizontal
- moved R20 216.1 mm to (-76.0, 49.6)
- moved J4 216.0 mm to (30.5, 63.7)
- moved R21 205.9 mm to (-76.0, 53.6)
- moved R22 205.9 mm to (-76.0, 57.7)
- moved D2 203.9 mm to (-64.3, 51.3)
- moved J5 202.2 mm to (30.5, 84.8)
- moved U16 201.8 mm to (-65.2, 57.2)
- moved C9 177.0 mm to (-56.6, 70.1)
- moved SW1 174.0 mm to (-75.6, 65.8)
- moved R23 173.2 mm to (-76.0, 61.7)
- moved D4 171.7 mm to (-56.9, 51.3)
- moved U10 166.3 mm to (175.5, 131.0), turned to 0 degrees
- moved R10 164.9 mm to (-48.2, 80.3)
- moved R11 164.9 mm to (-48.2, 84.4)
- moved R12 164.9 mm to (-48.2, 88.4)
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Connections:
- C7 pad 1: VCC -> +12V
- J10 pad 10: D13 -> D5
- J10 pad 11: D14 -> D6
- J10 pad 12: D15 -> D7
- J10 pad 23: A23 -> A9
- J10 pad 24: A22 -> A10
- J10 pad 25: A21 -> A11
- J10 pad 26: A20 -> A12
- J10 pad 27: A9 -> A13
- J10 pad 28: A10 -> A14
- J10 pad 29: A11 -> A15
- J10 pad 30: A12 -> unconnected-(J10-Pin_30-Pad30)
- J10 pad 31: A13 -> unconnected-(J10-Pin_31-Pad31)
- J10 pad 32: A14 -> unconnected-(J10-Pin_32-Pad32)
- J10 pad 33: A15 -> unconnected-(J10-Pin_33-Pad33)
- J10 pad 34: A16 -> unconnected-(J10-Pin_34-Pad34)
- J10 pad 35: A17 -> unconnected-(J10-Pin_35-Pad35)
- J10 pad 36: A18 -> unconnected-(J10-Pin_36-Pad36)
- J10 pad 37: A19 -> unconnected-(J10-Pin_37-Pad37)
- J10 pad 38: GND -> unconnected-(J10-Pin_38-Pad38)
- J10 pad 5: D8 -> D0
- J10 pad 6: D9 -> D1
- J10 pad 7: D10 -> D2
- J10 pad 8: D11 -> D3
- J10 pad 9: D12 -> D4
- J14 pad 1: unconnected-(J14-Pin_1-Pad1) -> +12V
- J14 pad 2: unconnected-(J14-Pin_2-Pad2) -> GND
- J14 pad 3: unconnected-(J14-Pin_3-Pad3) -> GND
- J14 pad 4: unconnected-(J14-Pin_4-Pad4) -> +5V
- J4 pad 2: unconnected-(J4-Pin_2-Pad2) -> /RTSA
- J5 pad 2: unconnected-(J5-Pin_2-Pad2) -> /RTSB
- J6 pad 1: VCC -> +12V
- J8 pad 1: VCC -> +12V
- J8 pad 3: VCC -> +12V
- J8 pad 5: VCC -> +12V
- U14 pad 14: unconnected-(U14-OP1-Pad14) -> /RTSB
- U14 pad 3: GND -> unconnected-(U14-IP3-Pad3)
- U14 pad 32: unconnected-(U14-OP0-Pad32) -> /RTSA
- U14 pad 40: GND -> unconnected-(U14-IP2-Pad40)
- U14 pad 42: GND -> unconnected-(U14-IP5-Pad42)
- U14 pad 43: GND -> unconnected-(U14-IP4-Pad43)
- U14 pad 5: GND -> unconnected-(U14-IP1-Pad5)
- U14 pad 8: GND -> unconnected-(U14-IP0-Pad8)
- U15 pad 1: VCC -> +12V
Other:
- board size 220 x 150 mm -> 170 x 170 mm
- copper layers 2 -> 4
- board text added: "12VDC"
- board text added: "GND"
- board text added: "LM2576"
- board text added: "MACKEREL-10 SBC v1.0"
- board text added: "RTSA"
- board text added: "RTSB"
- board text added: "RXA"
- board text added: "RXB"
- board text added: "TXA"
- board text added: "TXB"
- board text added: "github.com/crmaykish/mackerel-68k Colin Maykish - September 2024"

Commit message: Another layout plan
Parts:
- removed J10: Conn_02x20_Odd_Even, Connector_IDC:IDC-Header_2x20_P2.54mm_Vertical
- removed X2: 50MHz, Oscillator:Oscillator_DIP-14
- added C11: C, Capacitor_THT:C_Disc_D4.3mm_W1.9mm_P5.00mm, F.Cu at (156.1, 73.3)
- added C12: C, Capacitor_THT:C_Disc_D4.3mm_W1.9mm_P5.00mm, F.Cu at (82.3, 56.5)
- added C13: C, Capacitor_THT:C_Disc_D4.3mm_W1.9mm_P5.00mm, F.Cu at (150.4, 56.6)
- added C14: C, Capacitor_THT:C_Disc_D4.3mm_W1.9mm_P5.00mm, F.Cu at (82.3, 40.1)
- added C15: C, Capacitor_THT:C_Disc_D4.3mm_W1.9mm_P5.00mm, F.Cu at (150.9, 40.1)
- added J11: Conn_02x08_Odd_Even, Connector_PinHeader_2.54mm:PinHeader_2x08_P2.54mm_Vertical, F.Cu at (38.1, 213.4)
- added J12: Conn_02x04_Odd_Even, Connector_IDC:IDC-Header_2x04_P2.54mm_Vertical, F.Cu at (28.1, 152.4)
- added J13: Conn_02x04_Odd_Even, Connector_IDC:IDC-Header_2x04_P2.54mm_Vertical, F.Cu at (40.0, 152.4)
- added J15: Conn_02x04_Odd_Even, Connector_IDC:IDC-Header_2x04_P2.54mm_Vertical, F.Cu at (52.0, 152.4)
- added J16: Conn_02x04_Odd_Even, Connector_IDC:IDC-Header_2x04_P2.54mm_Vertical, F.Cu at (64.0, 152.4)
- added J17: Conn_02x30_Counter_Clockwise, Connector_IDC:IDC-Header_2x30_P2.54mm_Vertical, F.Cu at (86.9, 227.6)
- added U7: ~, mackerel:SIMM-30, F.Cu at (79.8, 68.4)
- added U8: ~, mackerel:SIMM-30, F.Cu at (79.8, 34.9)
- C1, C2, C3, C4: value 0.1uF -> 470uF; footprint Capacitor_THT:C_Disc_D4.7mm_W2.5mm_P5.00mm -> Capacitor_THT:CP_Radial_D8.0mm_P3.50mm
- C10, C5, C6: value 0.1uF -> C; footprint Capacitor_THT:C_Disc_D4.7mm_W2.5mm_P5.00mm -> Capacitor_THT:C_Disc_D4.3mm_W1.9mm_P5.00mm
- J4, J5: footprint Connector_PinSocket_2.54mm:PinSocket_1x06_P2.54mm_Horizontal -> Connector_PinSocket_2.54mm:PinSocket_1x06_P2.54mm_Vertical
- moved H4 266.8 mm to (22.9, -27.9)
- moved C6 230.3 mm to (155.7, 90.0), turned to 180 degrees
- moved H3 219.8 mm to (22.9, -35.9)
- moved C4 212.1 mm to (170.1, 40.2)
- moved C2 205.6 mm to (169.8, 73.4)
- moved J14 184.4 mm to (31.0, 55.9)
- moved J3 173.3 mm to (27.9, 83.3), turned to 0 degrees
- moved C5 157.3 mm to (82.5, 90.0), turned to 180 degrees
- moved U14 152.3 mm to (65.0, 180.8)
- moved X3 149.5 mm to (65.0, 212.9)
- moved C10 147.5 mm to (82.2, 73.3), turned to 180 degrees
- moved J2 146.3 mm to (173.2, 131.6)
- moved J1 145.7 mm to (173.2, 107.4)
- moved U12 126.3 mm to (48.3, 135.1), turned to 180 degrees
- moved U10 124.3 mm to (79.8, 51.6), turned to 180 degrees
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Connections:
- U10 pad 2: CAS1 -> CASA1
- U10 pad 21: RAMWR -> RAMWRA
- U10 pad 27: RAS -> RASA
- U11 pad 54: RAS -> unconnected-(U11-IO-Pad54)
- U11 pad 55: CAS0 -> unconnected-(U11-IO-Pad55)
- U11 pad 56: CAS1 -> unconnected-(U11-IO-Pad56)
- U11 pad 57: RAMWR -> unconnected-(U11-IO-Pad57)
- U11 pad 83: unconnected-(U11-GCLK1-Pad83) -> CLK_SRC
- U14 pad 15: unconnected-(U14-OP3-Pad15) -> OP3
- U14 pad 16: unconnected-(U14-OP5-Pad16) -> OP5
- U14 pad 17: unconnected-(U14-OP7-Pad17) -> OP7
- U14 pad 29: unconnected-(U14-OP6-Pad29) -> OP6
- U14 pad 3: unconnected-(U14-IP3-Pad3) -> IP3
- U14 pad 30: unconnected-(U14-OP4-Pad30) -> OP4
- U14 pad 31: unconnected-(U14-OP2-Pad31) -> OP2
- U14 pad 40: unconnected-(U14-IP2-Pad40) -> IP2
- U14 pad 42: unconnected-(U14-IP5-Pad42) -> IP5
- U14 pad 43: unconnected-(U14-IP4-Pad43) -> IP4
- U14 pad 5: unconnected-(U14-IP1-Pad5) -> IP1
- U14 pad 8: unconnected-(U14-IP0-Pad8) -> IP0
- U9 pad 2: CAS0 -> CASA0
- U9 pad 21: RAMWR -> RAMWRA
- U9 pad 27: RAS -> RASA
Routing:
- net RAM_A9: track 0.00 -> 50.1 mm
- net RAM_A8: track 0.00 -> 50.1 mm
- net RAM_A7: track 0.00 -> 50.1 mm
- net RAM_A6: track 0.00 -> 50.1 mm
- net RAM_A5: track 0.00 -> 50.1 mm
- net RAM_A4: track 0.00 -> 50.1 mm
- net RAM_A3: track 0.00 -> 50.1 mm
- net RAM_A2: track 0.00 -> 50.1 mm
- net RAM_A11: track 0.00 -> 50.1 mm
- net RAM_A10: track 0.00 -> 50.1 mm
- net RAM_A1: track 0.00 -> 50.1 mm
- net RAM_A0: track 0.00 -> 50.1 mm
- net RAMWRB: track 0.00 -> 35.2 mm
- net RASA: track 0.00 -> 34.5 mm
- net RASB: track 0.00 -> 34.5 mm
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Other:
- board size 170 x 170 mm -> 160 x 220 mm
- board text added: "SIMM_A0"
- board text added: "SIMM_A1"
- board text added: "SIMM_B0"
- board text added: "SIMM_B1"

Commit message: half routed
Parts:
- removed G***: LOGO, LOGO
- added C16: C, Capacitor_THT:C_Disc_D4.3mm_W1.9mm_P5.00mm, F.Cu at (178.2, 145.1)
- added C17: C, Capacitor_THT:C_Disc_D4.3mm_W1.9mm_P5.00mm, F.Cu at (183.1, 116.7)
- added C18: C, Capacitor_THT:C_Disc_D4.3mm_W1.9mm_P5.00mm, F.Cu at (160.2, 60.6)
- added C19: C, Capacitor_THT:C_Disc_D4.3mm_W1.9mm_P5.00mm, F.Cu at (181.5, 60.6)
- added C20: C, Capacitor_THT:C_Disc_D4.3mm_W1.9mm_P5.00mm, F.Cu at (202.9, 60.3)
- added C21: C, Capacitor_THT:C_Disc_D4.3mm_W1.9mm_P5.00mm, F.Cu at (224.1, 60.2)
- added C22: C, Capacitor_THT:C_Disc_D4.3mm_W1.9mm_P5.00mm, F.Cu at (203.9, 50.0)
- added C23: C, Capacitor_THT:C_Disc_D4.3mm_W1.9mm_P5.00mm, F.Cu at (157.6, 30.2)
- added C24: C, Capacitor_THT:C_Disc_D4.3mm_W1.9mm_P5.00mm, F.Cu at (172.4, 41.2)
- added C25: C, Capacitor_THT:C_Disc_D4.3mm_W1.9mm_P5.00mm, F.Cu at (46.2, 104.8)
- added C26: C, Capacitor_THT:C_Disc_D4.3mm_W1.9mm_P5.00mm, F.Cu at (58.9, 104.8)
- added C27: C, Capacitor_THT:C_Disc_D4.3mm_W1.9mm_P5.00mm, F.Cu at (36.1, 104.8)
- added C28: C, Capacitor_THT:C_Disc_D4.3mm_W1.9mm_P5.00mm, F.Cu at (28.5, 130.0)
- added C29: C, Capacitor_THT:C_Disc_D4.3mm_W1.9mm_P5.00mm, F.Cu at (46.1, 145.0)
- added C30: C, Capacitor_THT:C_Disc_D4.3mm_W1.9mm_P5.00mm, F.Cu at (56.4, 145.0)
- added C31: C, Capacitor_THT:C_Disc_D4.3mm_W1.9mm_P5.00mm, F.Cu at (68.8, 127.5)
- added C32: C, Capacitor_THT:C_Disc_D4.3mm_W1.9mm_P5.00mm, F.Cu at (112.3, 104.8)
- added C33: C, Capacitor_THT:C_Disc_D4.3mm_W1.9mm_P5.00mm, F.Cu at (48.7, 145.0)
- added C34: C, Capacitor_THT:C_Disc_D4.3mm_W1.9mm_P5.00mm, F.Cu at (120.2, 104.9)
- added C35: C, Capacitor_THT:C_Disc_D4.3mm_W1.9mm_P5.00mm, F.Cu at (97.1, 104.8)
- added C36: C, Capacitor_THT:C_Disc_D4.3mm_W1.9mm_P5.00mm, F.Cu at (89.7, 130.1)
- added C37: C, Capacitor_THT:C_Disc_D4.3mm_W1.9mm_P5.00mm, F.Cu at (107.2, 145.1)
- added C38: C, Capacitor_THT:C_Disc_D4.3mm_W1.9mm_P5.00mm, F.Cu at (117.6, 145.1)
- added C39: C, Capacitor_THT:C_Disc_D4.3mm_W1.9mm_P5.00mm, F.Cu at (114.9, 145.1)
- added C40: C, Capacitor_THT:C_Disc_D4.3mm_W1.9mm_P5.00mm, F.Cu at (129.9, 127.5)
- added C41: C, Capacitor_THT:C_Disc_D4.3mm_W1.9mm_P5.00mm, F.Cu at (76.6, 104.9)
- H1, H2, H3, H4: footprint MountingHole:MountingHole_3.2mm_M3_Pad -> MountingHole:MountingHole_3.2mm_M3_Pad_Via
- moved H4 280.9 mm to (226.0, 166.0)
- moved SW1 278.4 mm to (220.4, 50.0)
- moved R22 259.6 mm to (200.2, 56.1), turned to 180 degrees
- moved R20 259.5 mm to (200.2, 46.4), turned to 180 degrees
- moved R23 258.8 mm to (200.2, 49.6), turned to 180 degrees
- moved U16 255.8 mm to (207.2, 56.3), turned to 90 degrees
- moved J1 254.5 mm to (-54.6, -5.99), turned to 0 degrees
- moved C7 254.1 mm to (221.1, 41.0)
- moved R21 252.1 mm to (192.6, 52.8)
- moved C9 250.0 mm to (203.1, 44.9)
- moved HS1 247.5 mm to (201.1, 21.2), turned to 0 degrees
- moved U15 239.6 mm to (197.7, 24.5), turned to 0 degrees
- moved C8 239.2 mm to (209.3, 41.0)
- moved D3 238.2 mm to (190.2, 39.7), turned to 90 degrees
- moved L1 238.2 mm to (198.5, 33.8)
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Connections:
- J17 pad 20: GND -> unconnected-(J17-Pin_20-Pad20)
- J17 pad 41: GND -> unconnected-(J17-Pin_41-Pad41)
Routing:
- net D0: track 16.7 -> 259.7 mm, vias 0 -> 3
- net D8: track 16.7 -> 246.4 mm, vias 0 -> 4
- net D2: track 16.7 -> 239.7 mm, vias 0 -> 3
- net D1: track 16.7 -> 239.4 mm, vias 0 -> 3
- net D9: track 16.7 -> 236.8 mm, vias 0 -> 4
- net D3: track 16.7 -> 231.3 mm, vias 0 -> 2
- net D11: track 16.7 -> 229.2 mm, vias 0 -> 3
- net D10: track 16.7 -> 223.8 mm, vias 0 -> 4
- net D4: track 16.7 -> 222.6 mm, vias 0 -> 3
- net D12: track 16.7 -> 222.2 mm, vias 0 -> 3
- net D13: track 16.7 -> 216.7 mm, vias 0 -> 3
- net A1: track 0.00 -> 193.5 mm, vias 0 -> 2
- net D14: track 16.7 -> 210.2 mm, vias 0 -> 3
- net D15: track 16.7 -> 209.1 mm, vias 0 -> 3
- net A2: track 0.00 -> 190.8 mm, vias 0 -> 2
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Other:
- board size 160 x 220 mm -> 210 x 150 mm
- board text added: "3.6864 MHz"
- board text added: "555"
- board text added: "5V"
- board text added: "MC68010"
- board text added: "RESET"
- board text added: "ROM LOWER"
- board text added: "ROM UPPER"
- board text added: "RST"
- board text added: "SLOT A0"
- board text added: "SLOT A1"
- board text added: "SLOT B0"
- board text added: "SLOT B1"
- board text added: "SRAM LOWER"
- board text added: "SRAM UPPER"
- board text added: "XR68C681"
- board text removed: "12VDC"
- board text removed: "GND"
- board text removed: "LM2576"
- board text removed: "RTSA"
- board text removed: "RTSB"
- board text removed: "RXA"
- board text removed: "RXB"
- board text removed: "SIMM_A0"
- board text removed: "SIMM_A1"
- board text removed: "SIMM_B0"
- board text removed: "SIMM_B1"
- board text removed: "TXA"
- board text removed: "TXB"
