File: hardware/mackerel-10-v1/mackerel-10-v1.kicad_pcb (KiCad board)
At the start: 4 copper layers, 210 x 150 mm, 109 parts, among them J1 Conn_02x05_Odd_Even, J11 Conn_02x08_Odd_Even, J12 Conn_02x04_Odd_Even, J13 Conn_02x04_Odd_Even, J14 Screw_Terminal_01x04, J15 Conn_02x04_Odd_Even, J16 Conn_02x04_Odd_Even, J17 Conn_02x30_Counter_Clockwise, J2 Conn_02x05_Odd_Even, J3 Conn_02x20_Odd_Even, J4 Conn_01x06, J5 Conn_01x06, J6 Barrel_Jack_MountingPin, J7 Conn_02x03_Odd_Even, J8 Conn_02x03_Odd_Even, J9 Conn_02x03_Odd_Even, SW1 SW_Push, U1 68010D, U12 74HC245, U13 74HC245, U14 XR68C681, U15 LM2576T-5, U16 NE555P, U3 SST39SF040, U4 AS6C4008-55PCN, U5 SST39SF040, U6 AS6C4008-55PCN, X1 50MHz, X3 3.6864MHz

Commit message: DRAM controller mostly routed
Parts:
- removed D1: LED, LED_THT:LED_D5.0mm
- removed J1, J2: Conn_02x05_Odd_Even, Connector_IDC:IDC-Header_2x05_P2.54mm_Vertical
- removed J11: Conn_02x08_Odd_Even, Connector_PinHeader_2.54mm:PinHeader_2x08_P2.54mm_Vertical
- removed J12, J13, J15, J16: Conn_02x04_Odd_Even, Connector_IDC:IDC-Header_2x04_P2.54mm_Vertical
- removed J14: Screw_Terminal_01x04, TerminalBlock:TerminalBlock_bornier-4_P5.08mm
- removed J17: Conn_02x30_Counter_Clockwise, Connector_IDC:IDC-Header_2x30_P2.54mm_Vertical
- removed J3: Conn_02x20_Odd_Even, Connector_IDC:IDC-Header_2x20_P2.54mm_Vertical
- removed J7, J8, J9: Conn_02x03_Odd_Even, Connector_PinHeader_2.54mm:PinHeader_2x03_P2.54mm_Vertical
- removed R1, R10, R11, R12, R13, R17, R2, R3, R4, R5, R6, R7, R8, R9: R, Resistor_THT:R_Axial_DIN0207_L6.3mm_D2.5mm_P7.62mm_Horizontal
- removed R14, R15: 4k7, Resistor_THT:R_Axial_DIN0207_L6.3mm_D2.5mm_P7.62mm_Horizontal
- removed R16: 470, Resistor_THT:R_Axial_DIN0207_L6.3mm_D2.5mm_P7.62mm_Horizontal
- removed U12, U13: 74HC245, Package_DIP:DIP-20_W7.62mm_Socket
- added X2: 50MHz, Oscillator:Oscillator_DIP-14, F.Cu at (66.5, 132.9)
- moved R18 265.2 mm to (172.4, 31.3)
- moved R19 265.2 mm to (172.4, 35.4)
- moved U2 66.9 mm to (42.9, 109.6)
- moved U11 56.7 mm to (105.4, 109.8)
- moved J5 26.4 mm to (158.2, 22.1)
- moved C31 12.0 mm to (63.0, 138.0), turned to -90 degrees
- moved J4 11.3 mm to (181.9, 22.1)
- moved C36 9.04 mm to (85.3, 138.0)
- moved C25 5.81 mm to (40.4, 104.8)
- moved C26 5.81 mm to (53.1, 104.8)
- moved C27 5.81 mm to (30.3, 104.8)
- moved C28 5.81 mm to (22.7, 130.0)
- moved C29 5.81 mm to (40.3, 145.0)
- moved C30 5.81 mm to (50.6, 145.0)
- moved C33 5.81 mm to (42.9, 145.0)
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Connections:
- U11 pad 10: A13 -> RAM_A5
- U11 pad 11: A11 -> RAM_A4
- U11 pad 12: A9 -> RAM_A3
- U11 pad 15: A10 -> RAM_A2
- U11 pad 16: A21 -> RAM_A1
- U11 pad 17: A20 -> RAM_A0
- U11 pad 18: A22 -> CASB0
- U11 pad 2: unconnected-(U11-OE2/GCLK2-Pad2) -> CLK_ALT
- U11 pad 20: /RESET -> CASA0
- U11 pad 21: A23 -> CASA1
- U11 pad 22: unconnected-(U11-IO-Pad22) -> CASB1
- U11 pad 39: unconnected-(U11-IO-Pad39) -> R/W
- U11 pad 4: A17 -> RAM_A10
- U11 pad 40: unconnected-(U11-IO-Pad40) -> /LDS
- U11 pad 41: unconnected-(U11-IO-Pad41) -> /UDS
- U11 pad 44: A8 -> /AS
- U11 pad 45: A7 -> A1
- U11 pad 46: A6 -> A2
- U11 pad 48: A5 -> A3
- U11 pad 5: A15 -> RAM_A9
- U11 pad 50: A3 -> A5
- U11 pad 51: A2 -> A6
- U11 pad 52: A1 -> A7
- U11 pad 54: unconnected-(U11-IO-Pad54) -> A8
- U11 pad 55: unconnected-(U11-IO-Pad55) -> A9
- U11 pad 56: unconnected-(U11-IO-Pad56) -> A10
- U11 pad 57: unconnected-(U11-IO-Pad57) -> A11
- U11 pad 58: RAM_A0 -> A12
- U11 pad 6: A16 -> RAM_A8
- U11 pad 60: RAM_A1 -> A13
- U11 pad 61: RAM_A2 -> A14
- U11 pad 63: RAM_A3 -> A15
- U11 pad 64: RAM_A4 -> A16
- U11 pad 65: RAM_A5 -> A17
- U11 pad 67: RAM_A6 -> A18
- U11 pad 68: RAM_A7 -> A19
- U11 pad 69: RAM_A8 -> A20
- U11 pad 70: RAM_A9 -> A21
- U11 pad 73: RAM_A10 -> A22
- U11 pad 74: RAM_A11 -> A23
- U11 pad 75: /AS -> RASA
- U11 pad 76: R/W -> /RESET
- U11 pad 77: /LDS -> RASB
- U11 pad 79: A19 -> RAM_A11
- U11 pad 8: A14 -> RAM_A7
- U11 pad 80: /UDS -> RAMWRA
- U11 pad 81: A18 -> RAMWRB
- U11 pad 9: A12 -> RAM_A6
- U14 pad 15: OP3 -> unconnected-(U14-OP3-Pad15)
- U14 pad 16: OP5 -> unconnected-(U14-OP5-Pad16)
- U14 pad 17: OP7 -> unconnected-(U14-OP7-Pad17)
- U14 pad 29: OP6 -> unconnected-(U14-OP6-Pad29)
- U14 pad 3: IP3 -> GND
- U14 pad 30: OP4 -> unconnected-(U14-OP4-Pad30)
- U14 pad 31: OP2 -> unconnected-(U14-OP2-Pad31)
- U14 pad 40: IP2 -> GND
- U14 pad 42: IP5 -> GND
- U14 pad 43: IP4 -> GND
- U14 pad 5: IP1 -> GND
- U14 pad 8: IP0 -> GND
- U2 pad 10: A16 -> unconnected-(U2-IO-Pad10)
- U2 pad 11: A17 -> unconnected-(U2-IO-Pad11)
- U2 pad 12: A15 -> unconnected-(U2-IO-Pad12)
- U2 pad 15: A18 -> unconnected-(U2-IO-Pad15)
- U2 pad 16: A14 -> unconnected-(U2-IO-Pad16)
- U2 pad 17: R/W -> unconnected-(U2-IO-Pad17)
- U2 pad 18: A4 -> unconnected-(U2-IO-Pad18)
- U2 pad 2: unconnected-(U2-OE2/GCLK2-Pad2) -> CLK_ALT
- U2 pad 20: A3 -> unconnected-(U2-IO-Pad20)
- U2 pad 21: A2 -> unconnected-(U2-IO-Pad21)
- U2 pad 22: /SRAM_LOWER -> unconnected-(U2-IO-Pad22)
- U2 pad 24: A1 -> unconnected-(U2-IO-Pad24)
- U2 pad 25: D7 -> unconnected-(U2-IO-Pad25)
- U2 pad 27: D0 -> unconnected-(U2-IO-Pad27)
- U2 pad 28: D6 -> unconnected-(U2-IO-Pad28)
- U2 pad 29: D1 -> unconnected-(U2-IO-Pad29)
- U2 pad 30: D5 -> unconnected-(U2-IO-Pad30)
- U2 pad 31: D2 -> unconnected-(U2-IO-Pad31)
- U2 pad 33: D3 -> unconnected-(U2-IO-Pad33)
- U2 pad 34: D4 -> unconnected-(U2-IO-Pad34)
- U2 pad 35: /SRAM_UPPER -> unconnected-(U2-IO-Pad35)
- U2 pad 36: /ROM_LOWER -> unconnected-(U2-IO-Pad36)
- U2 pad 37: /ROM_UPPER -> unconnected-(U2-IO-Pad37)
- U2 pad 4: /IPL2 -> unconnected-(U2-IO-Pad4)
- U2 pad 5: /BERR -> unconnected-(U2-IO-Pad5)
- U2 pad 58: /IRQ_DUART -> unconnected-(U2-IO-Pad58)
- U2 pad 6: /VPA -> unconnected-(U2-IO-Pad6)
- U2 pad 60: /DTACK_DUART -> unconnected-(U2-IO-Pad60)
- U2 pad 61: /IACK_DUART -> unconnected-(U2-IO-Pad61)
- U2 pad 63: /DUART -> unconnected-(U2-IO-Pad63)
- U2 pad 64: A20 -> unconnected-(U2-IO-Pad64)
- U2 pad 65: A21 -> unconnected-(U2-IO-Pad65)
- U2 pad 67: A22 -> unconnected-(U2-IO-Pad67)
- U2 pad 68: A23 -> unconnected-(U2-IO-Pad68)
- U2 pad 69: /AS -> unconnected-(U2-IO-Pad69)
- U2 pad 70: /UDS -> unconnected-(U2-IO-Pad70)
- U2 pad 73: /LDS -> unconnected-(U2-IO-Pad73)
- U2 pad 74: /DTACK -> unconnected-(U2-IO-Pad74)
- U2 pad 76: FC0 -> unconnected-(U2-IO-Pad76)
- U2 pad 77: FC1 -> unconnected-(U2-IO-Pad77)
- U2 pad 79: FC2 -> unconnected-(U2-IO-Pad79)
- U2 pad 8: /RESET -> unconnected-(U2-IO-Pad8)
- U2 pad 80: /IPL0 -> unconnected-(U2-IO-Pad80)
- U2 pad 81: /IPL1 -> unconnected-(U2-IO-Pad81)
- U2 pad 9: A19 -> unconnected-(U2-IO-Pad9)
Routing:
- net /RESET: track 66.2 -> 224.4 mm, vias 1 -> 2
- net A15: track 69.7 -> 214.4 mm, vias 5 -> 7
- net CASB1: track 0.00 -> 123.8 mm
- net A5: track 118.6 -> 241.9 mm
- net A3: track 188.4 -> 308.7 mm
- net A2: track 190.8 -> 311.1 mm
- net A4: track 185.5 -> 304.1 mm
- net A1: track 193.5 -> 309.1 mm
- net A6: track 119.2 -> 234.5 mm
- net D7: track 183.6 -> 298.4 mm, vias 3 -> 4
- net D6: track 186.7 -> 300.6 mm, vias 3 -> 4
- net A7: track 119.7 -> 231.5 mm
- net D5: track 188.9 -> 300.1 mm, vias 3 -> 4
- net CLK_CPU: track 0.00 -> 110.9 mm
- net CASA1: track 0.00 -> 107.5 mm
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- added copper zone on In2.Cu, net +5V
- added copper zone on In1.Cu, net GND
Other:
- board size 210 x 150 mm -> 210 x 173.4 mm
- board text added: "CLK SRC"
- board text added: "DRAM"
- board text added: "SYSTEM"

Commit message: Glue logic CPLD almost fully routed
Parts:
- added C42: C, Capacitor_THT:C_Disc_D4.3mm_W1.9mm_P5.00mm, F.Cu at (71.4, 121.1)
- added D1: LED, LED_THT:LED_D5.0mm, F.Cu at (-250.5, 186.4)
- added J1: Conn_02x05_Odd_Even, Connector_IDC:IDC-Header_2x05_P2.54mm_Vertical, F.Cu at (-171.3, 165.3)
- added J14: Screw_Terminal_01x04, TerminalBlock:TerminalBlock_bornier-4_P5.08mm, F.Cu at (-264.9, 173.9)
- added J2: Conn_02x05_Odd_Even, Connector_IDC:IDC-Header_2x05_P2.54mm_Vertical, F.Cu at (-102.6, 172.8)
- added J3: Conn_02x20_Odd_Even, Connector_IDC:IDC-Header_2x20_P2.54mm_Vertical, F.Cu at (-274.9, 148.4)
- added J7: Conn_02x03_Odd_Even, Connector_PinHeader_2.54mm:PinHeader_2x03_P2.54mm_Vertical, F.Cu at (-220.2, 40.0)
- added J8: Conn_02x03_Odd_Even, Connector_PinHeader_2.54mm:PinHeader_2x03_P2.54mm_Vertical, F.Cu at (-213.0, 40.0)
- added J9: Conn_02x03_Odd_Even, Connector_PinHeader_2.54mm:PinHeader_2x03_P2.54mm_Vertical, F.Cu at (-205.8, 40.0)
- added R1: R, Resistor_THT:R_Axial_DIN0207_L6.3mm_D2.5mm_P7.62mm_Horizontal, F.Cu at (248.5, 146.3)
- added R10: R, Resistor_THT:R_Axial_DIN0207_L6.3mm_D2.5mm_P7.62mm_Horizontal, F.Cu at (-94.3, 168.7)
- added R11: R, Resistor_THT:R_Axial_DIN0207_L6.3mm_D2.5mm_P7.62mm_Horizontal, F.Cu at (-94.3, 172.7)
- added R12: R, Resistor_THT:R_Axial_DIN0207_L6.3mm_D2.5mm_P7.62mm_Horizontal, F.Cu at (-94.3, 176.8)
- added R13: R, Resistor_THT:R_Axial_DIN0207_L6.3mm_D2.5mm_P7.62mm_Horizontal, F.Cu at (-94.3, 180.8)
- added R14: 4k7, Resistor_THT:R_Axial_DIN0207_L6.3mm_D2.5mm_P7.62mm_Horizontal, F.Cu at (-265.8, 184.9)
- added R15: 4k7, Resistor_THT:R_Axial_DIN0207_L6.3mm_D2.5mm_P7.62mm_Horizontal, F.Cu at (-265.8, 189.0)
- added R16: 470, Resistor_THT:R_Axial_DIN0207_L6.3mm_D2.5mm_P7.62mm_Horizontal, F.Cu at (-253.6, 194.7)
- added R17: R, Resistor_THT:R_Axial_DIN0207_L6.3mm_D2.5mm_P7.62mm_Horizontal, F.Cu at (-265.9, 193.9)
- added R2: R, Resistor_THT:R_Axial_DIN0207_L6.3mm_D2.5mm_P7.62mm_Horizontal, F.Cu at (248.5, 150.4)
- added R3: R, Resistor_THT:R_Axial_DIN0207_L6.3mm_D2.5mm_P7.62mm_Horizontal, F.Cu at (248.5, 154.4)
- added R4: R, Resistor_THT:R_Axial_DIN0207_L6.3mm_D2.5mm_P7.62mm_Horizontal, F.Cu at (248.5, 158.5)
- added R5: R, Resistor_THT:R_Axial_DIN0207_L6.3mm_D2.5mm_P7.62mm_Horizontal, F.Cu at (248.5, 162.6)
- added R6: R, Resistor_THT:R_Axial_DIN0207_L6.3mm_D2.5mm_P7.62mm_Horizontal, F.Cu at (-163.0, 161.2)
- added R7: R, Resistor_THT:R_Axial_DIN0207_L6.3mm_D2.5mm_P7.62mm_Horizontal, F.Cu at (-163.0, 165.2)
- added R8: R, Resistor_THT:R_Axial_DIN0207_L6.3mm_D2.5mm_P7.62mm_Horizontal, F.Cu at (-163.0, 169.3)
- added R9: R, Resistor_THT:R_Axial_DIN0207_L6.3mm_D2.5mm_P7.62mm_Horizontal, F.Cu at (-163.0, 173.3)
- added U12: 74HC245, Package_DIP:DIP-20_W7.62mm_Socket, F.Cu at (-266.1, 144.4)
- added U13: 74HC245, Package_DIP:DIP-20_W7.62mm_Socket, F.Cu at (-254.4, 144.4)
- moved C32 0.33 mm to (107.9, 104.5)
- moved C34 0.33 mm to (115.8, 104.6)
- moved C20 0.30 mm to (202.9, 60.6)
- moved C35 0.27 mm to (92.7, 104.5)
- moved C25 0.27 mm to (40.4, 104.5)
- moved C27 0.27 mm to (30.3, 104.5)
- moved C26 0.27 mm to (53.1, 104.5)
Connections:
- U11 pad 24: unconnected-(U11-IO-Pad24) -> /CS_DRAM
- U11 pad 25: unconnected-(U11-IO-Pad25) -> /DTACK_DRAM
- U2 pad 10: unconnected-(U2-IO-Pad10) -> A19
- U2 pad 11: unconnected-(U2-IO-Pad11) -> A18
- U2 pad 12: unconnected-(U2-IO-Pad12) -> A17
- U2 pad 15: unconnected-(U2-IO-Pad15) -> A16
- U2 pad 16: unconnected-(U2-IO-Pad16) -> A15
- U2 pad 17: unconnected-(U2-IO-Pad17) -> A14
- U2 pad 18: unconnected-(U2-IO-Pad18) -> A1
- U2 pad 20: unconnected-(U2-IO-Pad20) -> A2
- U2 pad 21: unconnected-(U2-IO-Pad21) -> A3
- U2 pad 22: unconnected-(U2-IO-Pad22) -> A4
- U2 pad 4: unconnected-(U2-IO-Pad4) -> /RESET
- U2 pad 40: unconnected-(U2-IO-Pad40) -> FC0
- U2 pad 41: unconnected-(U2-IO-Pad41) -> FC1
- U2 pad 44: unconnected-(U2-IO-Pad44) -> FC2
- U2 pad 45: unconnected-(U2-IO-Pad45) -> /IPL1
- U2 pad 46: unconnected-(U2-IO-Pad46) -> /IPL0
- U2 pad 48: unconnected-(U2-IO-Pad48) -> /IPL2
- U2 pad 49: unconnected-(U2-IO-Pad49) -> /VPA
- U2 pad 5: unconnected-(U2-IO-Pad5) -> A23
- U2 pad 50: unconnected-(U2-IO-Pad50) -> /BERR
- U2 pad 51: unconnected-(U2-IO-Pad51) -> /DTACK
- U2 pad 52: unconnected-(U2-IO-Pad52) -> CLK_CPU
- U2 pad 54: unconnected-(U2-IO-Pad54) -> /CS_DRAM
- U2 pad 55: unconnected-(U2-IO-Pad55) -> /DTACK_DRAM
- U2 pad 56: unconnected-(U2-IO-Pad56) -> R/W
- U2 pad 57: unconnected-(U2-IO-Pad57) -> /LDS
- U2 pad 58: unconnected-(U2-IO-Pad58) -> D7
- U2 pad 6: unconnected-(U2-IO-Pad6) -> A22
- U2 pad 60: unconnected-(U2-IO-Pad60) -> /UDS
- U2 pad 61: unconnected-(U2-IO-Pad61) -> D6
- U2 pad 63: unconnected-(U2-IO-Pad63) -> /AS
- U2 pad 64: unconnected-(U2-IO-Pad64) -> D5
- U2 pad 65: unconnected-(U2-IO-Pad65) -> D0
- U2 pad 67: unconnected-(U2-IO-Pad67) -> D1
- U2 pad 68: unconnected-(U2-IO-Pad68) -> D2
- U2 pad 69: unconnected-(U2-IO-Pad69) -> D3
- U2 pad 70: unconnected-(U2-IO-Pad70) -> D4
- U2 pad 73: unconnected-(U2-IO-Pad73) -> /ROM_LOWER
- U2 pad 74: unconnected-(U2-IO-Pad74) -> /SRAM_UPPER
- U2 pad 75: unconnected-(U2-IO-Pad75) -> /ROM_UPPER
- U2 pad 76: unconnected-(U2-IO-Pad76) -> /SRAM_LOWER
- U2 pad 77: unconnected-(U2-IO-Pad77) -> /IRQ_DUART
- U2 pad 79: unconnected-(U2-IO-Pad79) -> /DTACK_DUART
- U2 pad 8: unconnected-(U2-IO-Pad8) -> A21
- U2 pad 80: unconnected-(U2-IO-Pad80) -> /IACK_DUART
- U2 pad 81: unconnected-(U2-IO-Pad81) -> /DUART
- U2 pad 9: unconnected-(U2-IO-Pad9) -> A20
Routing:
- net /SRAM_UPPER: track 0.00 -> 264.9 mm, vias 0 -> 2
- net /ROM_UPPER: track 0.00 -> 244.7 mm, vias 0 -> 3
- net /SRAM_LOWER: track 0.00 -> 223.4 mm, vias 0 -> 2
- net FC0: track 0.00 -> 201.9 mm
- net FC1: track 0.00 -> 194.3 mm
- net FC2: track 0.00 -> 190.8 mm
- net /IPL0: track 0.00 -> 185.9 mm
- net /IPL1: track 0.00 -> 178.9 mm
- net /IPL2: track 0.00 -> 178.2 mm
- net /BERR: track 0.00 -> 174.4 mm
- net A3: track 308.7 -> 482.8 mm, vias 2 -> 4
- net A4: track 304.1 -> 478.2 mm, vias 2 -> 4
- net /ROM_LOWER: track 0.00 -> 172.5 mm, vias 0 -> 1
- net A2: track 311.1 -> 478.7 mm, vias 2 -> 4
- net /VPA: track 0.00 -> 165.1 mm
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Other:
- board size 210 x 173.4 mm -> 210 x 150 mm
- board text added: "CLK ALT"

Commit message: Mostly routed except expansion
Parts:
- added C43: 1000uF, Capacitor_THT:CP_Radial_D10.0mm_P5.00mm, F.Cu at (202.6, 171.4)
- added C44: 470uF, Capacitor_THT:CP_Radial_D8.0mm_P3.50mm, F.Cu at (214.2, 172.7)
- J9: value Conn_02x03_Odd_Even -> Conn_02x20_Odd_Even; footprint Connector_PinHeader_2.54mm:PinHeader_2x03_P2.54mm_Vertical -> Connector_IDC:IDC-Header_2x20_P2.54mm_Vertical
- moved R16 471.8 mm to (216.5, 154.9)
- moved D1 468.3 mm to (217.2, 162.3)
- moved J14 467.6 mm to (202.6, 182.9)
- moved U12 462.8 mm to (196.2, 165.7), turned to -90 degrees
- moved R17 458.2 mm to (191.0, 159.5)
- moved R15 458.1 mm to (191.1, 156.0)
- moved R14 458.1 mm to (191.1, 152.4)
- moved J3 421.1 mm to (144.8, 182.9), turned to 90 degrees
- moved U13 420.0 mm to (165.1, 165.7), turned to -90 degrees
- moved J9 318.1 mm to (78.5, 182.7), turned to 90 degrees
- moved J7 309.9 mm to (56.7, 179.2)
- moved J8 309.9 mm to (63.9, 179.2)
- moved R9 220.6 mm to (56.4, 150.5), turned to -90 degrees
- moved R8 216.2 mm to (52.8, 158.1), turned to 90 degrees
- moved R7 212.4 mm to (49.3, 158.1), turned to 90 degrees
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Connections:
- J9 pad 1: +3.3V -> +5V
- J9 pad 2: GND -> +5V
- J9 pad 3: +3.3V -> GND
- J9 pad 5: +3.3V -> D0
- J9 pad 6: GND -> D1
- U2 pad 79: /DTACK_DUART -> /DUART
- U2 pad 81: /DUART -> /DTACK_DUART
Routing:
- net +12V: track 38.9 -> 203.8 mm
- net TDO_DRAM: track 0.00 -> 113.9 mm, vias 0 -> 1
- net TCK_DRAM: track 0.00 -> 113.5 mm
- net TDI_DRAM: track 0.00 -> 97.3 mm
- net TMS_DRAM: track 0.00 -> 90.6 mm
- net TDI: track 0.00 -> 64.1 mm
- net TCK: track 0.00 -> 58.2 mm
- net TDO: track 0.00 -> 57.0 mm, vias 0 -> 2
- net TMS: track 0.00 -> 55.6 mm
- net /DUART: track 147.0 -> 197.6 mm
- net /IACK_DUART: track 145.7 -> 195.7 mm, vias 1 -> 2
- net /DTACK_DUART: track 146.1 -> 182.2 mm
- net /IRQ_DUART: track 141.5 -> 177.2 mm
- net /RTSA: track 0.00 -> 31.8 mm
- net D14: track 210.2 -> 238.9 mm
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Other:
- board size 210 x 150 mm -> 210 x 170 mm
- board text added: "DRAM JTAG"
- board text added: "IDE"
- board text added: "SYSTEM JTAG"
