File: hardware/mackerel-10-v1/mackerel-10-v1.kicad_sch (KiCad schematic)
At the start: 0 parts

Commit message: Stubbed out mack-10 v1 design
Parts:
- added R1, R2, R3, R4, R5: R, Resistor_THT:R_Axial_DIN0204_L3.6mm_D1.6mm_P5.08mm_Horizontal, symbol Device:R
- added U1: 68010D, Package_DIP:DIP-64_W22.86mm, symbol CPU_NXP_68000:68010D
Connections:
- new net: R1.2, U1.13 (BR)
- new net: R2.2, U1.12 (BGACK)
- new net +5V: R1.1, R2.1, R3.1, R4.1, R5.1, U1.14 (VCC), U1.49 (VCC)
- new net A1: U1.29 (A1)
- new net A10: U1.38 (A10)
- new net A11: U1.39 (A11)
- new net A12: U1.40 (A12)
- new net A13: U1.41 (A13)
- new net A14: U1.42 (A14)
- new net A15: U1.43 (A15)
- new net A16: U1.44 (A16)
- new net A17: U1.45 (A17)
- new net A18: U1.46 (A18)
- new net A19: U1.47 (A19)
- new net A2: U1.30 (A2)
- new net A20: U1.48 (A20)
- new net A21: U1.50 (A21)
- new net A22: U1.51 (A22)
- new net A23: U1.52 (A23)
- new net A3: U1.31 (A3)
- new net A4: U1.32 (A4)
- new net A5: U1.33 (A5)
- new net A6: U1.34 (A6)
- new net A7: U1.35 (A7)
- new net A8: U1.36 (A8)
- new net A9: U1.37 (A9)
- new net CLK_CPU: U1.15 (CLK)
- new net D0: U1.5 (D0)
- new net D1: U1.4 (D1)
- new net D10: U1.59 (D10)
- new net D11: U1.58 (D11)
- new net D12: U1.57 (D12)
- new net D13: U1.56 (D13)
- new net D14: U1.55 (D14)
- new net D15: U1.54 (D15)
- new net D2: U1.3 (D2)
- new net D3: U1.2 (D3)
- new net D4: U1.1 (D4)
- new net D5: U1.64 (D5)
- new net D6: U1.63 (D6)
- new net D7: U1.62 (D7)
- new net D8: U1.61 (D8)
- new net D9: U1.60 (D9)
- new net FC0: U1.28 (FC0)
- new net FC1: U1.27 (FC1)
- new net FC2: U1.26 (FC2)
- new net GND: U1.16 (GND), U1.53 (GND)
- new net R/W: U1.9 (R/W)
- new net /AS: U1.6 (AS)
- new net /BERR: U1.22 (BERR)
- new net /DTACK: U1.10 (DTACK)
- new net /IPL0: R5.2, U1.25 (IPL0)
- new net /IPL1: R4.2, U1.24 (IPL1)
- new net /IPL2: R3.2, U1.23 (IPL2)
- new net /LDS: U1.8 (LDS)
- new net /RESET: U1.17 (HALT), U1.18 (RESET)
- new net /UDS: U1.7 (UDS)
- new net /VPA: U1.21 (VPA)
- no-connect marks 0 -> 3
Other:
- added sheet DRAM (dram.kicad_sch)
- added sheet DUART (duart.kicad_sch)
- added sheet Expansion (expansion.kicad_sch)
- added sheet Glue CPLD (glue_cpld.kicad_sch)
- added sheet IDE (ide.kicad_sch)
- added sheet Low Memory (low_mem.kicad_sch)
- added sheet Power and Reset (power_reset.kicad_sch)

Commit message: Rough layout of components on PCB
Parts:
- R1, R2, R3, R4, R5: footprint Resistor_THT:R_Axial_DIN0204_L3.6mm_D1.6mm_P5.08mm_Horizontal -> Resistor_THT:R_Axial_DIN0207_L6.3mm_D2.5mm_P7.62mm_Horizontal
Changed lines of the file:
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@@
 			)
 		)
-		(property "Footprint" "Resistor_THT:R_Axial_DIN0204_L3.6mm_D1.6mm_P5.08mm_Horizontal"
+		(property "Footprint" "Resistor_THT:R_Axial_DIN0207_L6.3mm_D2.5mm_P7.62mm_Horizontal"
 			(at 40.132 43.18 90)
 			(effects
@@
 			)
 		)
-		(property "Footprint" "Resistor_THT:R_Axial_DIN0204_L3.6mm_D1.6mm_P5.08mm_Horizontal"
+		(property "Footprint" "Resistor_THT:R_Axial_DIN0207_L6.3mm_D2.5mm_P7.62mm_Horizontal"
 			(at 42.672 43.18 90)
 			(effects
@@
 			)
 		)
-		(property "Footprint" "Resistor_THT:R_Axial_DIN0204_L3.6mm_D1.6mm_P5.08mm_Horizontal"
+		(property "Footprint" "Resistor_THT:R_Axial_DIN0207_L6.3mm_D2.5mm_P7.62mm_Horizontal"
 			(at 45.212 43.18 90)
 			(effects
@@
 			)
 		)
-		(property "Footprint" "Resistor_THT:R_Axial_DIN0204_L3.6mm_D1.6mm_P5.08mm_Horizontal"
+		(property "Footprint" "Resistor_THT:R_Axial_DIN0207_L6.3mm_D2.5mm_P7.62mm_Horizontal"
 			(at 50.292 43.18 90)
 			(effects
@@
 			)
 		)
-		(property "Footprint" "Resistor_THT:R_Axial_DIN0204_L3.6mm_D1.6mm_P5.08mm_Horizontal"
+		(property "Footprint" "Resistor_THT:R_Axial_DIN0207_L6.3mm_D2.5mm_P7.62mm_Horizontal"
 			(at 47.752 43.18 90)
 			(effects

Commit message: half routed
Parts:
- added C16, C17: C, Capacitor_THT:C_Disc_D4.3mm_W1.9mm_P5.00mm, symbol Device:C
Connections:
- net +5V: now also C16.1, C17.1
- net GND: now also C16.2, C17.2

Commit message: Remove BERR from CPLD
Parts:
- added R1: R, Resistor_THT:R_Axial_DIN0207_L6.3mm_D2.5mm_P7.62mm_Horizontal, symbol Device:R
- renumbered C16 to C1, C17 to C2, R1 to R2, R2 to R3, R3 to R4, R4 to R5, R5 to R6
Connections:
- net /IPL1 is gone; now on net /IPL0: R5.2, U1.24 (IPL1)
- net /IPL2 is gone; now on net /IPL0: R4.2, U1.23 (IPL2)
- net +5V: now also R1.1
- net /IPL0: now also R3.2, U1.12 (BGACK)
- net /BERR: no longer names the net of U1.22 (BERR)
- net /BERR: now also R1.2
Changed lines of the file:
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@@
+	)
+	(junction
+		(at 44.45 59.69)
+		(diameter 0)
+		(color 0 0 0 0)
+	)
+	(junction
+		(at 41.91 39.37)
+		(diameter 0)
+		(color 0 0 0 0)
 	)
 	(junction
@@
 	)
 	(junction
+		(at 46.99 57.15)
+		(diameter 0)
+		(color 0 0 0 0)
+	)
+	(junction
 		(at 149.86 43.18)
 		(diameter 0)
@@
 	)
 	(junction
+		(at 49.53 54.61)
+		(diameter 0)
+		(color 0 0 0 0)
+	)
+	(junction
 		(at 95.25 163.83)
 		(diameter 0)
@@
 	(wire
 		(pts
-			(xy 38.1 54.61) (xy 52.07 54.61)
+			(xy 35.56 54.61) (xy 49.53 54.61)
 		)
 		(stroke
@@
 	(wire
 		(pts
-			(xy 49.53 46.99) (xy 49.53 57.15)
+			(xy 49.53 46.99) (xy 49.53 54.61)
+		)
+		(stroke
+			(width 0)
+			(type default)
+		)
+	)
+	(wire
+		(pts
+			(xy 44.45 59.69) (xy 46.99 59.69)
+		)
+		(stroke
+			(width 0)
+			(type default)
+		)
+	)
+	(wire
+		(pts
+			(xy 39.37 39.37) (xy 41.91 39.37)
+		)
+		(stroke
+			(width 0)
+			(type default)
+		)
+	)
+	(wire
+		(pts
+			(xy 49.53 54.61) (xy 52.07 54.61)
 		)
 		(stroke
@@
 	(wire
 		(pts
-			(xy 38.1 59.69) (xy 46.99 59.69)
+			(xy 35.56 59.69) (xy 44.45 59.69)
 		)
 		(stroke
@@
 	(wire
 		(pts
-			(xy 44.45 46.99) (xy 44.45 64.77)
-		)
-		(stroke
-			(width 0)
-			(type default)
-		)
-	)
-	(wire
-		(pts
-			(xy 46.99 46.99) (xy 46.99 59.69)
+			(xy 44.45 46.99) (xy 44.45 59.69)
+		)
+		(stroke
+			(width 0)
+			(type default)
+		)
+	)
+	(wire
+		(pts
+			(xy 46.99 46.99) (xy 46.99 57.15)
 		)
 		(stroke
@@
 	(wire
 		(pts
+			(xy 46.99 57.15) (xy 46.99 59.69)
+		)
+		(stroke
+			(width 0)
+			(type default)
+		)
+	)
+	(wire
+		(pts
 			(xy 46.99 39.37) (xy 49.53 39.37)
 		)
@@
 	(wire
 		(pts
+			(xy 49.53 54.61) (xy 49.53 57.15)
+		)
+		(stroke
+			(width 0)
+			(type default)
+		)
+	)
+	(wire
+		(pts
 			(xy 44.45 39.37) (xy 46.99 39.37)
 		)
@@
 	(wire
 		(pts
-			(xy 38.1 57.15) (xy 49.53 57.15)
+			(xy 46.99 57.15) (xy 49.53 57.15)
+		)
+		(stroke
+			(width 0)
+			(type default)
+		)
+	)
+	(wire
+		(pts
+			(xy 44.45 59.69) (xy 44.45 64.77)
+		)
+		(stroke
+			(width 0)
+			(type default)
+		)
+	)
+	(wire
+		(pts
+			(xy 35.56 57.15) (xy 46.99 57.15)
 		)
 		(stroke
@@
 		(pts
 			(xy 92.71 41.91) (xy 95.25 41.91)
+		)
+		(stroke
+			(width 0)
+			(type default)
+		)
+	)
+	(wire
+		(pts
+			(xy 67.31 118.11) (xy 39.37 118.11)
+		)
+		(stroke
+			(width 0)
+			(type default)
+		)
+	)
+	(wire
+		(pts
+			(xy 39.37 118.11) (xy 39.37 46.99)
 		)
 		(stroke
@@
 	(global_label "{slash}IPL1"
 		(shape input)
-		(at 38.1 57.15 180)
+		(at 35.56 57.15 180)
 		(fields_autoplaced yes)
 		(effects
@@
 		)
 		(property "Intersheetrefs" "${INTERSHEET_REFS}"
-			(at 29.6719 57.15 0)
+			(at 27.1319 57.15 0)
 			(effects
 				(font
@@
 	(global_label "{slash}IPL2"
 		(shape input)
-		(at 38.1 59.69 180)
+		(at 35.56 59.69 180)
 		(fields_autoplaced yes)
 		(effects
@@
 		)
 		(property "Intersheetrefs" "${INTERSHEET_REFS}"
-			(at 29.6719 59.69 0)
+			(at 27.1319 59.69 0)
 			(effects
 				(font
@@
 				)
 				(justify left)
-				(hide yes)
-			)
-		)
-	)
-	(global_label "{slash}BERR"
-		(shape input)
-		(at 67.31 118.11 180)
-		(fields_autoplaced yes)
-		(effects
-			(font
-				(size 1.27 1.27)
-			)
-			(justify right)
-		)
-		(property "Intersheetrefs" "${INTERSHEET_REFS}"
-			(at 58.0353 118.11 0)
-			(effects
-				(font
-					(size 1.27 1.27)
-				)
-				(justify right)
 				(hide yes)
 			)
@@
 	(global_label "{slash}IPL0"
 		(shape input)
-		(at 38.1 54.61 180)
+		(at 35.56 54.61 180)
 		(fields_autoplaced yes)
 		(effects
@@
 		)
 		(property "Intersheetrefs" "${INTERSHEET_REFS}"
-			(at 29.6719 54.61 0)
+			(at 27.1319 54.61 0)
 			(effects
 				(font
@@
 		(dnp no)
 		(fields_autoplaced yes)
-		(property "Reference" "#PWR034"
+		(property "Reference" "#PWR03"
 			(at 142.24 34.29 0)
 			(effects
@@
 			(project ""
 				(path "/0a8f74be-008b-4256-a2d9-73a458311ea0"
-					(reference "#PWR034")
+					(reference "#PWR03")
 					(unit 1)
 				)
@@
 		(on_board yes)
 		(dnp no)
-		(property "Reference" "R1"
+		(property "Reference" "R2"
 			(at 41.91 44.45 90)
 			(effects
@@
 			(project "mackerel-10-v1"
 				(path "/0a8f74be-008b-4256-a2d9-73a458311ea0"
-					(reference "R1")
+					(reference "R2")
 					(unit 1)
 				)
@@
 		(dnp no)
 		(fields_autoplaced yes)
-		(property "Reference" "#PWR035"
+		(property "Reference" "#PWR04"
 			(at 149.86 49.53 0)
 			(effects
@@
 			(project ""
 				(path "/0a8f74be-008b-4256-a2d9-73a458311ea0"
-					(reference "#PWR035")
+					(reference "#PWR04")
 					(unit 1)
 				)
@@
 		(on_board yes)
 		(dnp no)
-		(property "Reference" "R2"
+		(property "Reference" "R3"
 			(at 44.45 44.45 90)
 			(effects
@@
 			(project "mackerel-10-v1"
 				(path "/0a8f74be-008b-4256-a2d9-73a458311ea0"
-					(reference "R2")
+					(reference "R3")
 					(unit 1)
 				)
@@
 		(on_board yes)
 		(dnp no)
-		(property "Reference" "R3"
+		(property "Reference" "R4"
 			(at 46.99 44.45 90)
 			(effects
@@
 			(project "mackerel-10-v1"
 				(path "/0a8f74be-008b-4256-a2d9-73a458311ea0"
-					(reference "R3")
+					(reference "R4")
 					(unit 1)
 				)
@@
 		(dnp no)
 		(fields_autoplaced yes)
-		(property "Reference" "C17"
+		(property "Reference" "C2"
 			(at 146.05 35.56 90)
 			(effects
@@
 			(project "mackerel-10-v1"
 				(path "/0a8f74be-008b-4256-a2d9-73a458311ea0"
-					(reference "C17")
+					(reference "C2")
 					(unit 1)
 				)
@@
 		(on_board yes)
 		(dnp no)
-		(property "Reference" "R5"
+		(property "Reference" "R6"
 			(at 52.07 44.45 90)
 			(effects
@@
 			(project "mackerel-10-v1"
 				(path "/0a8f74be-008b-4256-a2d9-73a458311ea0"
-					(reference "R5")
+					(reference "R6")
+					(unit 1)
+				)
+			)
+		)
+	)
+	(symbol
+		(lib_id "Device:R")
+		(at 39.37 43.18 0)
+		(unit 1)
+		(exclude_from_sim no)
+		(in_bom yes)
+		(on_board yes)
+		(dnp no)
+		(property "Reference" "R1"
+			(at 39.37 44.45 90)
+			(effects
+				(font
+					(size 1.27 1.27)
+				)
+				(justify left)
+			)
+		)
+		(property "Value" "R"
+			(at 41.91 44.4499 0)
+			(effects
+				(font
+					(size 1.27 1.27)
+				)
+				(justify left)
+				(hide yes)
+			)
+		)
+		(property "Footprint" "Resistor_THT:R_Axial_DIN0207_L6.3mm_D2.5mm_P7.62mm_Horizontal"
+			(at 37.592 43.18 90)
+			(effects
+				(font
+					(size 1.27 1.27)
+				)
+				(hide yes)
+			)
+		)
+		(property "Datasheet" "~"
+			(at 39.37 43.18 0)
+			(effects
+				(font
+					(size 1.27 1.27)
+				)
+				(hide yes)
+			)
+		)
+		(property "Description" "Resistor"
+			(at 39.37 43.18 0)
+			(effects
+				(font
+					(size 1.27 1.27)
+				)
+				(hide yes)
+			)
+		)
+		(pin "2"
+		)
+		(pin "1"
+		)
+		(instances
+			(project "mackerel-10-v1"
+				(path "/0a8f74be-008b-4256-a2d9-73a458311ea0"
+					(reference "R1")
 					(unit 1)
 				)
@@
 		(on_board yes)
 		(dnp no)
-		(property "Reference" "R4"
+		(property "Reference" "R5"
 			(at 49.53 44.45 90)
 			(effects
@@
 			(project "mackerel-10-v1"
 				(path "/0a8f74be-008b-4256-a2d9-73a458311ea0"
-					(reference "R4")
+					(reference "R5")
 					(unit 1)
 				)
@@
 		(dnp no)
 		(fields_autoplaced yes)
-		(property "Reference" "C16"
+		(property "Reference" "C1"
 			(at 146.05 22.86 90)
 			(effects
@@
 			(project "mackerel-10-v1"
 				(path "/0a8f74be-008b-4256-a2d9-73a458311ea0"
-					(reference "C16")
+					(reference "C1")
 					(unit 1)
 				)

Commit message: Rearranged power and reset on PCB
Connections:
- net /IPL0: no longer R3.2, R4.2, R5.2, U1.12 (BGACK), U1.23 (IPL2), U1.24 (IPL1)
- new net: R3.2, U1.12 (BGACK)
- new net /IPL1: R5.2, U1.24 (IPL1)
- new net /IPL2: R4.2, U1.23 (IPL2)
Changed lines of the file:
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@@
-	)
-	(junction
-		(at 44.45 59.69)
-		(diameter 0)
-		(color 0 0 0 0)
 	)
 	(junction
@@
 	)
 	(junction
-		(at 46.99 57.15)
-		(diameter 0)
-		(color 0 0 0 0)
-	)
-	(junction
 		(at 149.86 43.18)
 		(diameter 0)
@@
 	(junction
 		(at 142.24 30.48)
-		(diameter 0)
-		(color 0 0 0 0)
-	)
-	(junction
-		(at 49.53 54.61)
 		(diameter 0)
 		(color 0 0 0 0)
@@
 	(wire
 		(pts
-			(xy 35.56 54.61) (xy 49.53 54.61)
-		)
-		(stroke
-			(width 0)
-			(type default)
-		)
-	)
-	(wire
-		(pts
 			(xy 52.07 39.37) (xy 92.71 39.37)
 		)
@@
 	(wire
 		(pts
-			(xy 49.53 46.99) (xy 49.53 54.61)
-		)
-		(stroke
-			(width 0)
-			(type default)
-		)
-	)
-	(wire
-		(pts
-			(xy 44.45 59.69) (xy 46.99 59.69)
+			(xy 35.56 59.69) (xy 46.99 59.69)
 		)
 		(stroke
@@
 	(wire
 		(pts
-			(xy 49.53 54.61) (xy 52.07 54.61)
+			(xy 35.56 54.61) (xy 52.07 54.61)
 		)
 		(stroke
@@
 	(wire
 		(pts
-			(xy 35.56 59.69) (xy 44.45 59.69)
-		)
-		(stroke
-			(width 0)
-			(type default)
-		)
-	)
-	(wire
-		(pts
 			(xy 149.86 30.48) (xy 149.86 43.18)
 		)
@@
 	(wire
 		(pts
-			(xy 44.45 46.99) (xy 44.45 59.69)
-		)
-		(stroke
-			(width 0)
-			(type default)
-		)
-	)
-	(wire
-		(pts
-			(xy 46.99 46.99) (xy 46.99 57.15)
+			(xy 44.45 46.99) (xy 44.45 64.77)
+		)
+		(stroke
+			(width 0)
+			(type default)
+		)
+	)
+	(wire
+		(pts
+			(xy 46.99 46.99) (xy 46.99 59.69)
 		)
 		(stroke
@@
 	(wire
 		(pts
-			(xy 46.99 57.15) (xy 46.99 59.69)
-		)
-		(stroke
-			(width 0)
-			(type default)
-		)
-	)
-	(wire
-		(pts
 			(xy 46.99 39.37) (xy 49.53 39.37)
 		)
@@
 	(wire
 		(pts
-			(xy 49.53 54.61) (xy 49.53 57.15)
+			(xy 49.53 46.99) (xy 49.53 57.15)
 		)
 		(stroke
@@
 	(wire
 		(pts
-			(xy 46.99 57.15) (xy 49.53 57.15)
-		)
-		(stroke
-			(width 0)
-			(type default)
-		)
-	)
-	(wire
-		(pts
-			(xy 44.45 59.69) (xy 44.45 64.77)
-		)
-		(stroke
-			(width 0)
-			(type default)
-		)
-	)
-	(wire
-		(pts
-			(xy 35.56 57.15) (xy 46.99 57.15)
-		)
-		(stroke
+			(xy 35.56 57.15) (xy 49.53 57.15)
+		)
+		(stroke

Commit message: Mackerel-10 v1.1 release PCB
Other:
- title: Mackerel-10 SBC v1 -> Mackerel-10 SBC v1.1
Changed lines of the file:
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@@
 	(paper "A")
 	(title_block
-		(title "Mackerel-10 SBC v1")
-		(date "2024-09-23")
-		(rev "1.0a")
+		(title "Mackerel-10 SBC v1.1")
+		(date "2024-10-27")
+		(rev "1.1a")
 		(company "Colin Maykish")
 	)

Commit message: Add Mackerel-10 v1.1 BOM
Parts:
- C1, C2: value C -> 0.1uF
- R1, R2, R3, R4, R5, R6: value R -> 4k7
Changed lines of the file:
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@@
 			)
 		)
-		(property "Value" "R"
+		(property "Value" "4k7"
 			(at 44.45 44.4499 0)
 			(effects
@@
 			)
 		)
-		(property "Value" "R"
+		(property "Value" "4k7"
 			(at 46.99 44.4499 0)
 			(effects
@@
 			)
 		)
-		(property "Value" "R"
+		(property "Value" "4k7"
 			(at 49.53 44.4499 0)
 			(effects
@@
 			)
 		)
-		(property "Value" "C"
+		(property "Value" "0.1uF"
 			(at 146.05 38.1 90)
 			(effects
@@
 			)
 		)
-		(property "Value" "R"
+		(property "Value" "4k7"
 			(at 54.61 44.4499 0)
 			(effects
@@
 			)
 		)
-		(property "Value" "R"
+		(property "Value" "4k7"
 			(at 41.91 44.4499 0)
 			(effects
@@
 			)
 		)
-		(property "Value" "R"
+		(property "Value" "4k7"
 			(at 52.07 44.4499 0)
 			(effects
@@
 			)
 		)
-		(property "Value" "C"
+		(property "Value" "0.1uF"
 			(at 146.05 25.4 90)
 			(effects

Commit message: Mackerel-10 v1.2 Gerber release
Other:
- title: Mackerel-10 SBC v1.1 -> Mackerel-10
Changed lines of the file:
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@@
 	(paper "A")
 	(title_block
-		(title "Mackerel-10 SBC v1.1")
-		(date "2024-10-27")
-		(rev "1.1a")
+		(title "Mackerel-10")
+		(date "2024-11-09")
+		(rev "1.2")
 		(company "Colin Maykish")
 	)
