File: hardware/mackerel-10-dram/mackerel-10-dram.kicad_sch (KiCad schematic)
At the start: 28 parts, among them J1 Conn_02x20_Odd_Even, J2 Conn_02x20_Odd_Even, J3 Conn_02x05_Odd_Even, U4 74HC245, U5 74HC245

Commit message: Cleaned up the DRAM verilog and routed most of the PCB
Parts:
- removed U4, U5: 74HC245, Package_DIP:DIP-20_W7.62mm_Socket, symbol 74xx:74HC245
- added J4, J5: Conn_01x30, Connector_PinHeader_2.54mm:PinHeader_1x30_P2.54mm_Vertical, symbol Connector_Generic:Conn_01x30
- added R10, R11, R12, R13, R14, R15, R16, R17, R18, R19, R20, R21, R6, R7, R8, R9: 22, Resistor_THT:R_Axial_DIN0207_L6.3mm_D2.5mm_P2.54mm_Vertical, symbol Device:R
Connections:
- net +5V: now also J4.1 (Pin_1), J4.30 (Pin_30), J5.1 (Pin_1), J5.30 (Pin_30)
- net A1: no longer U3.4 (IO)
- net A10: now also U3.15 (IO); no longer U3.16 (IO)
- net A11: now also U3.11 (IO); no longer U3.17 (IO)
- net A12: now also U3.9 (IO); no longer U3.18 (IO)
- net A13: now also U3.10 (IO); no longer U3.20 (IO)
- net A14: now also U3.8 (IO); no longer U3.69 (IO)
- net A15: now also U3.5 (IO); no longer U3.70 (IO)
- net A16: now also U3.6 (IO); no longer U3.73 (IO)
- net A17: now also U3.4 (IO); no longer U3.74 (IO)
- net A18: now also U3.81 (IO); no longer U3.75 (IO)
- net A19: now also U3.79 (IO); no longer U3.76 (IO)
- net A2: no longer U3.5 (IO)
- net A20: now also U3.17 (IO); no longer U3.77 (IO)
- net A21: now also U3.16 (IO); no longer U3.79 (IO)
- net A22: now also U3.18 (IO); no longer U3.80 (IO)
- net A23: now also U3.21 (IO); no longer U3.81 (IO)
- net A3: no longer U3.6 (IO)
- net A4: no longer U3.8 (IO)
- net A5: no longer U3.9 (IO)
- net A6: no longer U3.10 (IO)
- net A7: no longer U3.11 (IO)
- net A8: no longer U3.12 (IO)
- net A9: now also U3.12 (IO); no longer U3.15 (IO)
- net CAS0: now also U3.55 (IO), J4.2 (Pin_2); no longer U3.24 (IO)
- net CAS1: now also U3.56 (IO), J5.2 (Pin_2); no longer U3.25 (IO)
- net CLK_CPU: no longer U3.2 (OE2/GCLK2)
- net D0: now also R13.2
- net D1: now also R12.2
- net D10: now also R16.2
- net D11: now also R17.2
- net D12: now also R18.2
- net D13: now also R19.2
- net D14: now also R20.2
- net D15: now also R21.2
- net D2: now also R11.2
- net D3: now also R10.2
- net D4: now also R9.2
- net D5: now also R8.2
- net D6: now also R7.2
- net D7: now also R6.2
- net D8: now also R14.2
- net D9: now also R15.2
- net GND: now also U3.2 (OE2/GCLK2), J4.22 (Pin_22), J4.9 (Pin_9), J5.22 (Pin_22), J5.9 (Pin_9)
- net RAMWR: now also U3.57 (IO), J4.21 (Pin_21), J5.21 (Pin_21); no longer U3.22 (IO)
- net RAM_A0: now also U3.58 (IO), J4.4 (Pin_4), J5.4 (Pin_4)
- net RAM_A1: now also U3.60 (IO), J4.5 (Pin_5), J5.5 (Pin_5)
- net RAM_A10: now also U3.73 (IO), J4.19 (Pin_19), J5.19 (Pin_19)
- net RAM_A11: now also U3.74 (IO), J4.24 (Pin_24), J5.24 (Pin_24)
- net RAM_A2: now also U3.61 (IO), J4.7 (Pin_7), J5.7 (Pin_7)
- net RAM_A3: now also U3.63 (IO), J4.8 (Pin_8), J5.8 (Pin_8)
- net RAM_A4: now also U3.64 (IO), J4.11 (Pin_11), J5.11 (Pin_11)
- net RAM_A5: now also U3.65 (IO), J4.12 (Pin_12), J5.12 (Pin_12)
- net RAM_A6: now also U3.67 (IO), J4.14 (Pin_14), J5.14 (Pin_14)
- net RAM_A7: now also U3.68 (IO), J4.15 (Pin_15), J5.15 (Pin_15)
- net RAM_A8: now also U3.69 (IO), J4.17 (Pin_17), J5.17 (Pin_17)
- net RAM_A9: now also U3.70 (IO), J4.18 (Pin_18), J5.18 (Pin_18)
- net RAS: now also U3.54 (IO), J4.27 (Pin_27), J5.27 (Pin_27); no longer U3.27 (IO)
- net R/W: now also U3.76 (IO)
- net /AS: now also U3.75 (IO)
- net /LDS: now also U3.77 (IO)
- net /UDS: now also U3.80 (IO)
- net RAM_OE0: no longer names the net of U3.28 (IO)
- net RAM_OE1: no longer names the net of U3.29 (IO)
- net RD0 renamed RAM_D7
- net RAM_D7: now also J4.25 (Pin_25), R13.1
- net RD1 renamed RAM_D6
- net RAM_D6: now also J4.23 (Pin_23), R12.1
- net RD10 renamed RAM_D10
- net RAM_D10: now also J5.10 (Pin_10), R16.1
- net RD11 renamed RAM_D11
- net RAM_D11: now also J5.13 (Pin_13), R17.1
- net RD12 renamed RAM_D12
- net RAM_D12: now also J5.16 (Pin_16), R18.1
- net RD13 renamed RAM_D13
- net RAM_D13: now also J5.20 (Pin_20), R19.1
- net RD14 renamed RAM_D14
- net RAM_D14: now also J5.23 (Pin_23), R20.1
- net RD15 renamed RAM_D15
- net RAM_D15: now also J5.25 (Pin_25), R21.1
- net RD2 renamed RAM_D5
- net RAM_D5: now also J4.20 (Pin_20), R11.1
- net RD3 renamed RAM_D4
- net RAM_D4: now also J4.16 (Pin_16), R10.1
- net RD4 renamed RAM_D3
- net RAM_D3: now also J4.13 (Pin_13), R9.1
- net RD5 renamed RAM_D2
- net RAM_D2: now also J4.10 (Pin_10), R8.1
- net RD6 renamed RAM_D1
- net RAM_D1: now also J4.6 (Pin_6), R7.1
- net RD7 renamed RAM_D0
- net RAM_D0: now also J4.3 (Pin_3), R6.1
- net RD8 renamed RAM_D8
- net RAM_D8: now also J5.3 (Pin_3), R14.1
- net RD9 renamed RAM_D9
- net RAM_D9: now also J5.6 (Pin_6), R15.1
Other:
- note added: "NOTE: data lines are reversed to facilitate routing"
- note removed: "Data lines intentional reversed to make routing easier"

Commit message: Update CPLD pin assignments for DRAM breakout PCB
Parts:
- added J6: Conn_01x10, Connector_PinSocket_2.54mm:PinSocket_1x10_P2.54mm_Vertical, symbol Connector_Generic:Conn_01x10
Connections:
- net +5V: now also J6.9 (Pin_9)
- net A1: now also U3.52 (IO)
- net A2: now also U3.51 (IO)
- net A3: now also U3.50 (IO)
- net A4: now also U3.49 (IO)
- net A5: now also U3.48 (IO)
- net A6: now also U3.46 (IO)
- net A7: now also U3.45 (IO)
- net A8: now also U3.44 (IO)
- net GND: now also J6.10 (Pin_10)
- net /DTACK_EXP: now also U3.40 (IO)
- net /EXP: now also U3.41 (IO)
- net /RESET: now also U3.20 (IO)
- net at U3.22 (IO): now also J6.1 (Pin_1)
- net at U3.24 (IO): now also J6.2 (Pin_2)
- net at U3.25 (IO): now also J6.3 (Pin_3)
- net at U3.27 (IO): now also J6.4 (Pin_4)
- net at U3.28 (IO): now also J6.5 (Pin_5)
- net at U3.29 (IO): now also J6.6 (Pin_6)
- net at U3.30 (IO): now also J6.7 (Pin_7)
- net at U3.31 (IO): now also J6.8 (Pin_8)
- no-connect marks 9 -> 34
Other:
- company: (none) -> Colin Maykish
- title: (none) -> Mackerel-10 DRAM Proto
- moved on the sheet: C1, C10, C2, C3, C4, C5, C6, C7, C8, C9, D1, H1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
