File: hardware/mackerel-08-v1/mackerel-08-duart.kicad_sch (KiCad schematic)
At the start: 15 parts, among them J1 Conn_01x08, J2 Conn_02x09_Odd_Even, J3 Conn_01x06, J4 Conn_01x06, U14 XR68C681, X2 CXO_DIP14

Commit message: Add Mackerel-08 BOM list
Parts:
- R12, R13, R14, R16, R17, R18, R19: value R -> 4k7
- R15: value R -> 1k
Other:
- title: Mackerel-08 SBC v1 -> Mackerel-08 SBC v1.1
- moved on the sheet: R16, R17
Changed lines of the file:
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@@
 	(paper "A")
 	(title_block
-		(title "Mackerel-08 SBC v1")
+		(title "Mackerel-08 SBC v1.1")
 		(date "2024-08-22")
 		(rev "1.1")
@@
 	)
 	(junction
-		(at 187.96 58.42)
-		(diameter 0)
-		(color 0 0 0 0)
-	)
-	(junction
 		(at 195.58 66.04)
 		(diameter 0)
@@
 	)
 	(junction
-		(at 190.5 40.64)
+		(at 182.88 58.42)
 		(diameter 0)
 		(color 0 0 0 0)
 	)
 	(junction
-		(at 190.5 60.96)
+		(at 195.58 40.64)
 		(diameter 0)
 		(color 0 0 0 0)
 	)
 	(junction
-		(at 195.58 40.64)
+		(at 187.96 40.64)
 		(diameter 0)
 		(color 0 0 0 0)
@@
 	)
 	(junction
+		(at 187.96 60.96)
+		(diameter 0)
+		(color 0 0 0 0)
+	)
+	(junction
 		(at 193.04 63.5)
 		(diameter 0)
@@
 	(wire
 		(pts
-			(xy 196.85 58.42) (xy 187.96 58.42)
+			(xy 195.58 66.04) (xy 196.85 66.04)
 		)
 		(stroke
@@
 	(wire
 		(pts
-			(xy 195.58 66.04) (xy 196.85 66.04)
+			(xy 187.96 40.64) (xy 193.04 40.64)
 		)
 		(stroke
@@
 	(wire
 		(pts
-			(xy 187.96 40.64) (xy 190.5 40.64)
+			(xy 182.88 40.64) (xy 187.96 40.64)
 		)
 		(stroke
@@
 	(wire
 		(pts
-			(xy 190.5 60.96) (xy 162.56 60.96)
+			(xy 181.61 88.9) (xy 181.61 92.71)
 		)
 		(stroke
@@
 	(wire
 		(pts
-			(xy 190.5 40.64) (xy 193.04 40.64)
+			(xy 187.96 60.96) (xy 162.56 60.96)
 		)
 		(stroke
@@
 	(wire
 		(pts
-			(xy 181.61 88.9) (xy 181.61 92.71)
+			(xy 177.8 53.34) (xy 162.56 53.34)
 		)
 		(stroke
@@
 	(wire
 		(pts
-			(xy 177.8 53.34) (xy 162.56 53.34)
+			(xy 24.13 146.05) (xy 36.83 146.05)
 		)
 		(stroke
@@
 	(wire
 		(pts
-			(xy 24.13 146.05) (xy 36.83 146.05)
+			(xy 57.15 101.6) (xy 43.18 101.6)
 		)
 		(stroke
@@
 	(wire
 		(pts
-			(xy 57.15 101.6) (xy 43.18 101.6)
+			(xy 187.96 48.26) (xy 187.96 60.96)
 		)
 		(stroke
@@
 	(wire
 		(pts
-			(xy 190.5 48.26) (xy 190.5 60.96)
+			(xy 40.64 22.86) (xy 53.34 22.86)
 		)
 		(stroke
@@
 	(wire
 		(pts
-			(xy 187.96 58.42) (xy 162.56 58.42)
+			(xy 182.88 58.42) (xy 196.85 58.42)
 		)
 		(stroke
@@
 	(wire
 		(pts
-			(xy 40.64 22.86) (xy 53.34 22.86)
+			(xy 182.88 58.42) (xy 162.56 58.42)
 		)
 		(stroke
@@
 	(wire
 		(pts
-			(xy 177.8 76.2) (xy 180.34 76.2)
+			(xy 187.96 60.96) (xy 196.85 60.96)
 		)
 		(stroke
@@
 	(wire
 		(pts
-			(xy 196.85 53.34) (xy 177.8 53.34)
+			(xy 177.8 76.2) (xy 180.34 76.2)
 		)
 		(stroke
@@
 	(wire
 		(pts
-			(xy 162.56 66.04) (xy 195.58 66.04)
+			(xy 196.85 53.34) (xy 177.8 53.34)
 		)
 		(stroke
@@
 	(wire
 		(pts
-			(xy 196.85 60.96) (xy 190.5 60.96)
+			(xy 162.56 66.04) (xy 195.58 66.04)
 		)
 		(stroke
@@
 	(wire
 		(pts
-			(xy 187.96 48.26) (xy 187.96 58.42)
+			(xy 182.88 48.26) (xy 182.88 58.42)
 		)
 		(stroke
@@
 		(dnp no)
 		(property "Reference" "R12"
-			(at 118.11 81.28 90)
+			(at 116.078 81.788 90)
 			(effects
 				(font
@@
 			)
 		)
-		(property "Value" "R"
-			(at 115.57 81.28 0)
+		(property "Value" "4k7"
+			(at 118.11 81.788 90)
 			(effects
 				(font
@@
 				)
 				(justify right)
-				(hide yes)
 			)
 		)
@@
 	(symbol
 		(lib_id "Device:R")
-		(at 190.5 44.45 180)
+		(at 187.96 44.45 180)
 		(unit 1)
 		(exclude_from_sim no)
@@
 		(dnp no)
 		(property "Reference" "R17"
-			(at 190.5 45.72 90)
+			(at 185.928 46.482 90)
 			(effects
 				(font
@@
 			)
 		)
-		(property "Value" "R"
-			(at 189.992 44.704 0)
+		(property "Value" "4k7"
+			(at 187.96 46.228 90)
 			(effects
 				(font
@@
 				)
 				(justify right)
-				(hide yes)
 			)
 		)
 		(property "Footprint" "Resistor_SMD:R_1206_3216Metric_Pad1.30x1.75mm_HandSolder"
-			(at 192.278 44.45 90)
+			(at 189.738 44.45 90)
 			(effects
 				(font
@@
 		)
 		(property "Datasheet" "~"
-			(at 190.5 44.45 0)
+			(at 187.96 44.45 0)
 			(effects
 				(font
@@
 		)
 		(property "Description" "Resistor"
-			(at 190.5 44.45 0)
+			(at 187.96 44.45 0)
 			(effects
 				(font
@@
 		(dnp no)
 		(property "Reference" "R18"
-			(at 193.04 45.72 90)
+			(at 191.008 46.482 90)
 			(effects
 				(font
@@
 			)
 		)
-		(property "Value" "R"
-			(at 192.532 44.704 0)
+		(property "Value" "4k7"
+			(at 193.04 46.228 90)
 			(effects
 				(font
@@
 				)
 				(justify right)
-				(hide yes)
 			)
 		)
@@
 		(dnp no)
 		(property "Reference" "R13"
-			(at 177.8 73.66 90)
+			(at 175.768 74.168 90)
 			(effects
 				(font
@@
 			)
 		)
-		(property "Value" "R"
-			(at 177.292 72.644 0)
+		(property "Value" "4k7"
+			(at 177.8 74.168 90)
 			(effects
 				(font
@@
 				)
 				(justify right)
-				(hide yes)
 			)
 		)
@@
 		(dnp no)
 		(property "Reference" "R14"
-			(at 180.34 73.66 90)
+			(at 182.626 74.168 90)
 			(effects
 				(font
@@
 			)
 		)
-		(property "Value" "R"
-			(at 179.832 72.644 0)
+		(property "Value" "4k7"
+			(at 180.34 74.168 90)
 			(effects
 				(font
@@
 				)
 				(justify right)
-				(hide yes)
 			)
 		)
@@
 		(dnp no)
 		(property "Reference" "R19"
-			(at 195.58 45.72 90)
+			(at 197.612 46.482 90)
 			(effects
 				(font
@@
 			)
 		)
-		(property "Value" "R"
-			(at 195.072 44.704 0)
+		(property "Value" "4k7"
+			(at 195.58 46.228 90)
 			(effects
 				(font
@@
 				)
 				(justify right)
-				(hide yes)
 			)
 		)
@@
 	(symbol
 		(lib_id "Device:R")
-		(at 187.96 44.45 180)
+		(at 182.88 44.45 180)
 		(unit 1)
 		(exclude_from_sim no)
@@
 		(dnp no)
 		(property "Reference" "R16"
-			(at 187.96 45.72 90)
+			(at 180.848 46.482 90)
 			(effects
 				(font
@@
 			)
 		)
-		(property "Value" "R"
-			(at 187.452 44.704 0)
+		(property "Value" "4k7"
+			(at 182.88 46.228 90)
 			(effects
 				(font
@@
 				)
 				(justify right)
-				(hide yes)
 			)
 		)
 		(property "Footprint" "Resistor_SMD:R_1206_3216Metric_Pad1.30x1.75mm_HandSolder"
-			(at 189.738 44.45 90)
+			(at 184.658 44.45 90)
 			(effects
 				(font
@@
 		)
 		(property "Datasheet" "~"
-			(at 187.96 44.45 0)
+			(at 182.88 44.45 0)
 			(effects
 				(font
@@
 		)
 		(property "Description" "Resistor"
-			(at 187.96 44.45 0)
+			(at 182.88 44.45 0)
 			(effects
 				(font
@@
 		(on_board yes)
 		(dnp no)
-		(fields_autoplaced yes)
 		(property "Reference" "R15"
-			(at 184.15 95.2499 0)
+			(at 179.578 98.552 90)
 			(effects
 				(font
@@
 			)
 		)
-		(property "Value" "R"
-			(at 184.15 97.7899 0)
+		(property "Value" "1k"
+			(at 181.61 97.79 90)
 			(effects
 				(font
