File: hardware/mackerel-08-v1/mackerel-08-duart.kicad_sch (KiCad schematic)
At the start: 15 parts, among them J1 Conn_01x08, J2 Conn_02x09_Odd_Even, J3 Conn_01x06, J4 Conn_01x06, U14 XR68C681, X2 CXO_DIP14

Commit message: Mackerel-8: Remove 555 reset, 3.3v regulator, user LED
Parts:
- removed D1: LED, LED_THT:LED_D5.0mm, symbol Device:LED
- removed R15: 1k, Resistor_SMD:R_1206_3216Metric_Pad1.30x1.75mm_HandSolder, symbol Device:R
Connections:
- net +3.3V: no longer names the net of J2.3 (Pin_3)
- net +3.3V: no longer J2.4 (Pin_4)
- net USR_LED: no longer names the net of U14.17 (OP7)
