File: hardware/mackerel-08-v1/mackerel-08-v1.kicad_pcb (KiCad board)
At the start: 4 copper layers, 180 x 120 mm, 83 parts, among them J1 Conn_01x08, J2 Conn_02x08_Odd_Even, J3 Conn_01x06, J4 Conn_01x06, J5 Barrel_Jack_MountingPin, J6 Conn_02x03_Odd_Even, J7 Conn_02x03_Odd_Even, J8 Conn_02x20_Odd_Even, J9 Conn_02x10_Odd_Even, SW1 SW_Push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

Commit message: Mackerel-08 v1.1 release
Parts:
- removed REF**: OSHW-Logo2_7.3x6mm_SilkScreen, Symbol:OSHW-Logo2_7.3x6mm_SilkScreen

Commit message: Mackerel-08 rev 1.1 release
Parts:
- added C21: C_Polarized, Capacitor_THT:CP_Radial_D5.0mm_P2.50mm, F.Cu at (61.7, 155.7)
- added C22: C_Polarized, Capacitor_THT:CP_Radial_D5.0mm_P2.50mm, F.Cu at (66.3, 143.8)
- added J10: Conn_02x03_Odd_Even, Connector_PinHeader_2.54mm:PinHeader_2x03_P2.54mm_Vertical, F.Cu at (72.3, 148.2)
- added U17: ~, Package_TO_SOT_SMD:TO-252-2, F.Cu at (60.7, 145.9)
- J2: value Conn_02x08_Odd_Even -> Conn_02x09_Odd_Even; footprint Connector_PinHeader_2.54mm:PinHeader_2x08_P2.54mm_Vertical -> Connector_PinHeader_2.54mm:PinHeader_2x09_P2.54mm_Vertical
- moved SW1 80.5 mm to (27.4, 83.9), turned to -90 degrees
- moved J7 3.95 mm to (79.7, 148.2)
- moved J2 2.52 mm to (88.3, 47.5)
- moved J6 2.24 mm to (87.0, 148.2)
- moved G*** 2.22 mm to (43.2, 47.3)
Connections:
- J2 pad 10: SPI_CLK -> SPI_DO
- J2 pad 11: SPI_CS0 -> SPI_CLK
- J2 pad 12: SPI_CS1 -> SPI_CLK
- J2 pad 13: SPI_INT0 -> SPI_CS0
- J2 pad 14: SPI_INT1 -> SPI_CS1
- J2 pad 15: /RESET -> SPI_INT0
- J2 pad 16: /RESET -> SPI_INT1
- J2 pad 3: GND -> +3.3V
- J2 pad 4: GND -> +3.3V
- J2 pad 5: SPI_DI -> GND
- J2 pad 6: SPI_DI -> GND
- J2 pad 7: SPI_DO -> SPI_DI
- J2 pad 8: SPI_DO -> SPI_DI
- J2 pad 9: SPI_CLK -> SPI_DO
Routing:
- net +3.3V: track 0.00 -> 137.0 mm
- net Net-(U16-R): track 83.5 -> 58.4 mm
- net +5V: track 43.5 -> 48.8 mm
- net GND: track 22.6 -> 27.6 mm
- net D4: track 311.4 -> 308.5 mm, vias 5 -> 4
- net VCC: track 161.6 -> 164.2 mm
- net D5: track 310.4 -> 307.9 mm, vias 5 -> 4
- net D6: track 304.5 -> 302.5 mm, vias 5 -> 4
- net D7: track 304.9 -> 303.3 mm
- net D1: track 313.2 -> 312.1 mm
- net D3: track 317.0 -> 316.1 mm
- net D2: track 327.9 -> 327.1 mm
- net D0: track 308.5 -> 307.7 mm
Other:
- board text added: "3.3V"
- board text added: "AP1084"
- board text added: "LM2576"
