File: hardware/mackerel-30-proto/mackerel-30-proto.kicad_sch (KiCad schematic)
At the start: 20 parts, among them U1 MC68030RC, U2 EPM7128

Commit message: Add power and DUART
Parts:
- added J5: Conn_02x05_Odd_Even, Connector_IDC:IDC-Header_2x05_P2.54mm_Vertical, symbol Connector_Generic:Conn_02x05_Odd_Even
- added R4, R5, R6, R7: R, Resistor_THT:R_Axial_DIN0207_L6.3mm_D2.5mm_P7.62mm_Horizontal, symbol Device:R
Connections:
- net +5V: now also J5.4 (Pin_4), R4.1, R5.1, R6.1
- net GND: now also J5.10 (Pin_10), J5.2 (Pin_2), R7.2
- net TDI: now reaches U2.14 (TDI)
- net TDI: now also J5.9 (Pin_9), R6.2
- net TMS: now reaches U2.23 (TMS)
- net TMS: now also J5.5 (Pin_5), R5.2
- net TCK: now reaches U2.62 (TCK)
- net TCK: now also J5.1 (Pin_1), R7.1
- net TDO: now reaches U2.71 (TDO)
- net TDO: now also J5.3 (Pin_3), R4.2
- no-connect marks 0 -> 3
Other:
- added sheet Power (power.kicad_sch)
- moved on the sheet: U2

Commit message: Add 68882 FPU symbol
Parts:
- renumbered J5 to J1, R4 to R1, R5 to R2, R6 to R3, R7 to R4
Other:
- added sheet DRAM (dram.kicad_sch)
- added sheet FPU (fpu.kicad_sch)
- note added: "TODO: A1-A3 (at least) for FC and interrupt decode"
Changed lines of the file:
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@@
 		)
 	)
+	(text "TODO: A1-A3 (at least) for FC and interrupt decode"
+		(exclude_from_sim no)
+		(at 182.626 22.352 0)
+		(effects
+			(font
+				(size 1.27 1.27)
+			)
+		)
+	)
 	(global_label "{slash}IPL1"
 		(shape input)
@@
 		)
 	)
+	(global_label "{slash}CS_SRAM"
+		(shape output)
+		(at 217.17 71.12 0)
+		(fields_autoplaced yes)
+		(effects
+			(font
+				(size 1.27 1.27)
+			)
+			(justify left)
+		)
+		(property "Intersheetrefs" "${INTERSHEET_REFS}"
+			(at 229.9523 71.12 0)
+			(effects
+				(font
+					(size 1.27 1.27)
+				)
+				(justify left)
+				(hide yes)
+			)
+		)
+	)
 	(global_label "D23"
 		(shape bidirectional)
@@
 		)
 	)
+	(global_label "{slash}CS_DRAM"
+		(shape output)
+		(at 217.17 73.66 0)
+		(fields_autoplaced yes)
+		(effects
+			(font
+				(size 1.27 1.27)
+			)
+			(justify left)
+		)
+		(property "Intersheetrefs" "${INTERSHEET_REFS}"
+			(at 230.0128 73.66 0)
+			(effects
+				(font
+					(size 1.27 1.27)
+				)
+				(justify left)
+				(hide yes)
+			)
+		)
+	)
 	(global_label "D9"
 		(shape bidirectional)
@@
 		)
 	)
+	(global_label "{slash}CS_ROM"
+		(shape output)
+		(at 217.17 68.58 0)
+		(fields_autoplaced yes)
+		(effects
+			(font
+				(size 1.27 1.27)
+			)
+			(justify left)
+		)
+		(property "Intersheetrefs" "${INTERSHEET_REFS}"
+			(at 228.9847 68.58 0)
+			(effects
+				(font
+					(size 1.27 1.27)
+				)
+				(justify left)
+				(hide yes)
+			)
+		)
+	)
 	(global_label "A23"
 		(shape output)
@@
 		)
 	)
+	(global_label "{slash}DRAM_DTACK"
+		(shape input)
+		(at 217.17 77.47 0)
+		(fields_autoplaced yes)
+		(effects
+			(font
+				(size 1.27 1.27)
+			)
+			(justify left)
+		)
+		(property "Intersheetrefs" "${INTERSHEET_REFS}"
+			(at 233.3995 77.47 0)
+			(effects
+				(font
+					(size 1.27 1.27)
+				)
+				(justify left)
+				(hide yes)
+			)
+		)
+	)
 	(global_label "TMS"
 		(shape output)
@@
 		(on_board yes)
 		(dnp no)
-		(property "Reference" "R4"
+		(property "Reference" "R1"
 			(at 238.76 140.97 90)
 			(effects
@@
 			(project "mackerel-30-proto"
 				(path "/9307474f-ec99-494d-b4c9-fbd0b10ce86a"
-					(reference "R4")
+					(reference "R1")
 					(unit 1)
 				)
@@
 		(dnp no)
 		(fields_autoplaced yes)
-		(property "Reference" "#PWR039"
+		(property "Reference" "#PWR09"
 			(at 261.62 170.18 0)
 			(effects
@@
 			(project "mackerel-30-proto"
 				(path "/9307474f-ec99-494d-b4c9-fbd0b10ce86a"
-					(reference "#PWR039")
+					(reference "#PWR09")
 					(unit 1)
 				)
@@
 		(dnp no)
 		(fields_autoplaced yes)
-		(property "Reference" "J5"
+		(property "Reference" "J1"
 			(at 254 138.43 0)
 			(effects
@@
 			(project "mackerel-30-proto"
 				(path "/9307474f-ec99-494d-b4c9-fbd0b10ce86a"
-					(reference "J5")
+					(reference "J1")
 					(unit 1)
 				)
@@
 		(on_board yes)
 		(dnp no)
-		(property "Reference" "R6"
+		(property "Reference" "R3"
 			(at 243.84 140.97 90)
 			(effects
@@
 			(project "mackerel-30-proto"
 				(path "/9307474f-ec99-494d-b4c9-fbd0b10ce86a"
-					(reference "R6")
+					(reference "R3")
 					(unit 1)
 				)
@@
 		(dnp no)
 		(fields_autoplaced yes)
-		(property "Reference" "#PWR038"
+		(property "Reference" "#PWR010"
 			(at 262.89 132.08 0)
 			(effects
@@
 			(project "mackerel-30-proto"
 				(path "/9307474f-ec99-494d-b4c9-fbd0b10ce86a"
-					(reference "#PWR038")
+					(reference "#PWR010")
 					(unit 1)
 				)
@@
 		(on_board yes)
 		(dnp no)
-		(property "Reference" "R5"
+		(property "Reference" "R2"
 			(at 241.3 140.97 90)
 			(effects
@@
 			(project "mackerel-30-proto"
 				(path "/9307474f-ec99-494d-b4c9-fbd0b10ce86a"
-					(reference "R5")
+					(reference "R2")
 					(unit 1)
 				)
@@
 		(on_board yes)
 		(dnp no)
-		(property "Reference" "R7"
+		(property "Reference" "R4"
 			(at 246.38 161.036 90)
 			(effects
@@
 			(project "mackerel-30-proto"
 				(path "/9307474f-ec99-494d-b4c9-fbd0b10ce86a"
-					(reference "R7")
+					(reference "R4")
 					(unit 1)
 				)
@@
 	)
 	(sheet
+		(at 33.655 165.735)
+		(size 12.7 3.81)
+		(fields_autoplaced yes)
+		(stroke
+			(width 0.1524)
+			(type solid)
+		)
+		(fill
+			(color 0 0 0 0.0000)
+		)
+		(property "Sheetname" "DRAM"
+			(at 33.655 165.0234 0)
+			(effects
+				(font
+					(size 1.27 1.27)
+				)
+				(justify left bottom)
+			)
+		)
+		(property "Sheetfile" "dram.kicad_sch"
+			(at 33.655 170.1296 0)
+			(effects
+				(font
+					(size 1.27 1.27)
+				)
+				(justify left top)
+			)
+		)
+		(instances
+			(project "mackerel-30-proto"
+				(path "/9307474f-ec99-494d-b4c9-fbd0b10ce86a"
+					(page "5")
+				)
+			)
+		)
+	)
+	(sheet
 		(at 57.15 196.85)
 		(size 12.7 3.81)
@@
 				)
 			)
+		)
+	)
+	(sheet
+		(at 29.21 152.4)
+		(size 12.7 3.81)
+		(fields_autoplaced yes)
+		(stroke
+			(width 0.1524)
+			(type solid)
+		)
+		(fill
+			(color 0 0 0 0.0000)
+		)
+		(property "Sheetname" "FPU"
+			(at 29.21 151.6884 0)
+			(effects
+				(font
+					(size 1.27 1.27)
+				)
+				(justify left bottom)
+			)
+		)
+		(property "Sheetfile" "fpu.kicad_sch"
+			(at 29.21 156.7946 0)
+			(effects
+				(font
+					(size 1.27 1.27)
+				)
+				(justify left top)
+			)
+		)
+		(instances
+			(project "mackerel-30-proto"
+				(path "/9307474f-ec99-494d-b4c9-fbd0b10ce86a"
+					(page "6")
+				)
+			)

Commit message: Working on control and glue
Parts:
- added J7, J8: Conn_01x03, Connector_PinHeader_2.54mm:PinHeader_1x03_P2.54mm_Vertical, symbol Connector_Generic:Conn_01x03
- added R13, R14, R15, R16, R17: 4k7, symbol Device:R
Connections:
- net +5V: now also J7.1 (Pin_1), J8.1 (Pin_1), R13.1, R14.1, R15.1, R16.1, R17.1
- net GND: now also J7.3 (Pin_3), J8.3 (Pin_3)
- net /IPL0: now also R13.2
- net /IPL1: now also R14.2
- net /IPL2: now also R15.2
- net at U1.A1 (/BR): now also R16.2
- net at U1.C3 (/BGACK): now also R17.2
- net /MMUDIS: now reaches U1.F13 (/MMUDIS)
- net /MMUDIS: now also J7.2 (Pin_2)
- net /CDIS: now reaches U1.H12 (/CDIS)
- net /CDIS: now also J8.2 (Pin_2)
- no-connect marks 3 -> 4

Commit message: Wired most of the control signals for the CPU and DRAM
Parts:
- removed J7, J8: Conn_01x03, Connector_PinHeader_2.54mm:PinHeader_1x03_P2.54mm_Vertical, symbol Connector_Generic:Conn_01x03
- added J1, J2: Conn_01x02, Connector_PinHeader_2.54mm:PinHeader_1x02_P2.54mm_Vertical, symbol Connector_Generic:Conn_01x02
- added R1, R2, R3, R4: 4k7, Resistor_THT:R_Axial_DIN0207_L6.3mm_D2.5mm_P7.62mm_Horizontal, symbol Device:R
- added X1: CXO_DIP14, Oscillator:Oscillator_DIP-14, symbol Oscillator:CXO_DIP14
- R5: renamed from R13; footprint (none) -> Resistor_THT:R_Axial_DIN0207_L6.3mm_D2.5mm_P7.62mm_Horizontal
- R6: renamed from R14; footprint (none) -> Resistor_THT:R_Axial_DIN0207_L6.3mm_D2.5mm_P7.62mm_Horizontal
- R7: renamed from R15; footprint (none) -> Resistor_THT:R_Axial_DIN0207_L6.3mm_D2.5mm_P7.62mm_Horizontal
- R8: renamed from R16; footprint (none) -> Resistor_THT:R_Axial_DIN0207_L6.3mm_D2.5mm_P7.62mm_Horizontal
- R9: renamed from R17; footprint (none) -> Resistor_THT:R_Axial_DIN0207_L6.3mm_D2.5mm_P7.62mm_Horizontal
- renumbered J1 to J3, R1 to R10, R2 to R11, R3 to R12, R4 to R13
Connections:
- net +5V: now also R1.1, R2.1, R3.1, R4.1, X1.14 (Vcc)
- net A0: now also U2.44 (IO)
- net A1: now also U2.45 (IO)
- net A16: now also U2.49 (IO)
- net A17: now also U2.50 (IO)
- net A18: now also U2.51 (IO)
- net A19: now also U2.52 (IO)
- net A2: now also U2.46 (IO)
- net A20: now also U2.54 (IO)
- net A21: now also U2.55 (IO)
- net A22: now also U2.56 (IO)
- net A23: now also U2.57 (IO)
- net A24: now also U2.58 (IO)
- net A25: now also U2.60 (IO)
- net A26: now also U2.61 (IO)
- net A27: now also U2.63 (IO)
- net A3: now also U2.48 (IO)
- net D24: now also U2.33 (IO)
- net D25: now also U2.34 (IO)
- net D26: now also U2.35 (IO)
- net D27: now also U2.36 (IO)
- net D28: now also U2.37 (IO)
- net D29: now also U2.39 (IO)
- net D30: now also U2.40 (IO)
- net D31: now also U2.41 (IO)
- net FC0: now also U2.77 (IO)
- net FC1: now also U2.79 (IO)
- net FC2: now also U2.80 (IO)
- net GND: now also J1.2 (Pin_2), J2.2 (Pin_2), X1.7 (GND)
- net R/W: now also U2.67 (IO)
- net SIZ0: now also U2.70 (IO)
- net SIZ1: now also U2.73 (IO)
- net /AS: now also U2.64 (IO)
- net /AVEC: now also U2.81 (IO)
- net /CS_DRAM: now also U2.10 (IO)
- net /CS_ROM: now also U2.8 (IO)
- net /CS_SRAM: now also U2.9 (IO)
- net /DS: now also U2.65 (IO)
- net /DSACK0: now also U2.68 (IO)
- net /DSACK1: now also U2.69 (IO)
- net /IPL0: now also U2.74 (IO)
- net /IPL1: now also U2.75 (IO)
- net /IPL2: now also U2.76 (IO)
- net CLK_CPU: now reaches U1.E1 (CLK)
- net CLK_CPU: now also U2.83 (GCLK1), X1.8 (OUT)
- net /RESET: now reaches U1.F12 (/RESET)
- net /STERM: now reaches U1.G1 (/STERM)
- net /STERM: now also U2.5 (IO)
- net /BERR: now reaches U1.H1 (/BERR)
- net /BERR: now also U2.6 (IO)
- net at U1.H2 (/HALT): now also R4.2
- net at U1.J1 (/CBACK): now also R2.2
- net /CIIN: now reaches U1.L1 (/CIIN)
- net /CIIN: now also U2.4 (IO)
- net /DTACK_DRAM: now reaches U2.11 (IO)
- net /CS_DUART: now reaches U2.12 (IO)
- net /DTACK_DUART: now reaches U2.15 (IO)
- net /IRQ_DUART: now reaches U2.16 (IO)
- net /IACK_DUART: now reaches U2.17 (IO)
- net IDE_INT: now reaches U2.18 (IO)
- net /IDE_CS0: now reaches U2.20 (IO)
- net IDE_RDY: now reaches U2.21 (IO)
- net /IDE_RD: now reaches U2.22 (IO)
- net /IDE_WR: now reaches U2.24 (IO)
- net /IDE_BUF: now reaches U2.25 (IO)
- net /CS_FPU: now reaches U2.27 (IO)
- net /DSACK0_FPU: now reaches U2.28 (IO)
- net /DSACK1_FPU: now reaches U2.29 (IO)
- net A28: no longer names the net of U1.A4 (A28)
- net A29: no longer names the net of U1.B4 (A29)
- net A30: no longer names the net of U1.A3 (A30)
- net A31: no longer names the net of U1.B3 (A31)
- net /CDIS: no longer names the net of U1.H12 (/CDIS)
- net /CDIS: now also J2.1 (Pin_1), R1.2
- net /MMUDIS: no longer names the net of U1.F13 (/MMUDIS)
- net /MMUDIS: now also J1.1 (Pin_1), R3.2
- no-connect marks 4 -> 18
Other:
- added sheet IDE (ide.kicad_sch)
- note added: "TODO: Run CPU clock through CPLD?"
- note added: "TODO: make some room for SPI pins Or bitbang it with DUART?"
- note removed: "TODO: A1-A3 (at least) for FC and interrupt decode"
- moved on the sheet: U2

Commit message: More glue wiring
Connections:
- net A20: no longer U2.54 (IO)
- net A21: no longer U2.55 (IO)
- net A22: no longer U2.56 (IO)
- net A23: no longer U2.57 (IO)
Other:
- note added: "TODO: SPI clock source?"

Commit message: A bit of cleanup
Parts:
- added R4: 4k7, Resistor_THT:R_Axial_DIN0207_L6.3mm_D2.5mm_P7.62mm_Horizontal, symbol Device:R
- renumbered R9 to R10, R10 to R11, R11 to R12, R12 to R13, R13 to R14, R4 to R5, R5 to R6, R6 to R7, R7 to R8, R8 to R9
Connections:
- net +5V: now also R4.1
- net A20: now also U2.54 (IO)
- net A21: now also U2.55 (IO)
- net A22: now also U2.56 (IO)
- net A23: now also U2.57 (IO)
- net D24: no longer U2.33 (IO)
- net D25: no longer U2.34 (IO)
- net D26: no longer U2.35 (IO)
- net D27: no longer U2.36 (IO)
- net D28: no longer U2.37 (IO)
- net D29: no longer U2.39 (IO)
- net D30: no longer U2.40 (IO)
- net D31: no longer U2.41 (IO)
- net /BERR: no longer names the net of U1.H1 (/BERR)
- net /BERR: now also R4.2; no longer U2.6 (IO)
Other:
- added sheet Expansion (expansion.kicad_sch)
- note removed: "TODO: SPI clock source?"
- note removed: "TODO: make some room for SPI pins Or bitbang it with DUART?"
- moved on the sheet: J1, R1, R2, R3

Commit message: positioning
Parts:
- C1, C10, C11, C12, C13, C14, C15, C16, C17, C18, C2, C3, C4, C5, C6, C7, C8, C9: footprint Capacitor_SMD:C_1210_3225Metric_Pad1.33x2.70mm_HandSolder -> Capacitor_SMD:C_1206_3216Metric_Pad1.33x1.80mm_HandSolder
- R1, R10, R11, R12, R13, R14, R2, R3, R4, R5, R6, R7, R8, R9: footprint Resistor_THT:R_Axial_DIN0207_L6.3mm_D2.5mm_P7.62mm_Horizontal -> Resistor_SMD:R_0805_2012Metric_Pad1.20x1.40mm_HandSolder
Connections:
- net A0: no longer U2.44 (IO)
- net A1: no longer U2.45 (IO)
- net A16: no longer U2.49 (IO)
- net A17: no longer U2.50 (IO)
- net A18: no longer U2.51 (IO)
- net A19: no longer U2.52 (IO)
- net A2: no longer U2.46 (IO)
- net A20: no longer U2.54 (IO)
- net A21: no longer U2.55 (IO)
- net A22: no longer U2.56 (IO)
- net A23: no longer U2.57 (IO)
- net A24: no longer U2.58 (IO)
- net A25: no longer U2.60 (IO)
- net A26: no longer U2.61 (IO)
- net A27: no longer U2.63 (IO)
- net A3: no longer U2.48 (IO)
- net FC0: no longer U2.77 (IO)
- net FC1: no longer U2.79 (IO)
- net FC2: no longer U2.80 (IO)
- net IDE_INT: no longer U2.18 (IO)
- net IDE_RDY: no longer U2.21 (IO)
- net R/W: no longer U2.67 (IO)
- net SIZ0: no longer U2.70 (IO)
- net SIZ1: no longer U2.73 (IO)
- net /AS: no longer U2.64 (IO)
- net /AVEC: no longer U2.81 (IO)
- net /CIIN: no longer U2.4 (IO)
- net /CS_DRAM: no longer U2.10 (IO)
- net /CS_DUART: no longer U2.12 (IO)
- net /CS_FPU: no longer U2.27 (IO)
- net /CS_ROM: no longer U2.8 (IO)
- net /CS_SRAM: no longer U2.9 (IO)
- net /DS: no longer U2.65 (IO)
- net /DSACK0: no longer U2.68 (IO)
- net /DSACK0_FPU: no longer U2.28 (IO)
- net /DSACK1: no longer U2.69 (IO)
- net /DSACK1_FPU: no longer U2.29 (IO)
- net /DTACK_DRAM: no longer U2.11 (IO)
- net /DTACK_DUART: no longer U2.15 (IO)
- net /IACK_DUART: no longer U2.17 (IO)
- net /IDE_BUF: no longer U2.25 (IO)
- net /IDE_CS0: no longer U2.20 (IO)
- net /IDE_RD: no longer U2.22 (IO)
- net /IDE_WR: no longer U2.24 (IO)
- net /IPL0: no longer U2.74 (IO)
- net /IPL1: no longer U2.75 (IO)
- net /IPL2: no longer U2.76 (IO)
- net /IRQ_DUART: no longer U2.16 (IO)
- net /STERM: no longer U2.5 (IO)

Commit message: rough layout of the PCB components
Parts:
- removed R4: 4k7, Resistor_SMD:R_0805_2012Metric_Pad1.20x1.40mm_HandSolder, symbol Device:R
- C1, C10, C11, C12, C13, C14, C15, C16, C17, C18, C2, C3, C4, C5, C6, C7, C8, C9: footprint Capacitor_SMD:C_1206_3216Metric_Pad1.33x1.80mm_HandSolder -> Capacitor_THT:C_Disc_D4.3mm_W1.9mm_P5.00mm
- R1, R2, R3: footprint Resistor_SMD:R_0805_2012Metric_Pad1.20x1.40mm_HandSolder -> Resistor_THT:R_Axial_DIN0207_L6.3mm_D2.5mm_P7.62mm_Horizontal
- R10: renamed from R11; footprint Resistor_SMD:R_0805_2012Metric_Pad1.20x1.40mm_HandSolder -> Resistor_THT:R_Axial_DIN0207_L6.3mm_D2.5mm_P7.62mm_Horizontal
- R11: renamed from R12; footprint Resistor_SMD:R_0805_2012Metric_Pad1.20x1.40mm_HandSolder -> Resistor_THT:R_Axial_DIN0207_L6.3mm_D2.5mm_P7.62mm_Horizontal
- R12: renamed from R13; footprint Resistor_SMD:R_0805_2012Metric_Pad1.20x1.40mm_HandSolder -> Resistor_THT:R_Axial_DIN0207_L6.3mm_D2.5mm_P7.62mm_Horizontal
- R13: renamed from R14; footprint Resistor_SMD:R_0805_2012Metric_Pad1.20x1.40mm_HandSolder -> Resistor_THT:R_Axial_DIN0207_L6.3mm_D2.5mm_P7.62mm_Horizontal
- R4: renamed from R5; footprint Resistor_SMD:R_0805_2012Metric_Pad1.20x1.40mm_HandSolder -> Resistor_THT:R_Axial_DIN0207_L6.3mm_D2.5mm_P7.62mm_Horizontal
- R5: renamed from R6; footprint Resistor_SMD:R_0805_2012Metric_Pad1.20x1.40mm_HandSolder -> Resistor_THT:R_Axial_DIN0207_L6.3mm_D2.5mm_P7.62mm_Horizontal
- R6: renamed from R7; footprint Resistor_SMD:R_0805_2012Metric_Pad1.20x1.40mm_HandSolder -> Resistor_THT:R_Axial_DIN0207_L6.3mm_D2.5mm_P7.62mm_Horizontal
- R7: renamed from R8; footprint Resistor_SMD:R_0805_2012Metric_Pad1.20x1.40mm_HandSolder -> Resistor_THT:R_Axial_DIN0207_L6.3mm_D2.5mm_P7.62mm_Horizontal
- R8: renamed from R9; footprint Resistor_SMD:R_0805_2012Metric_Pad1.20x1.40mm_HandSolder -> Resistor_THT:R_Axial_DIN0207_L6.3mm_D2.5mm_P7.62mm_Horizontal
- R9: renamed from R10; footprint Resistor_SMD:R_0805_2012Metric_Pad1.20x1.40mm_HandSolder -> Resistor_THT:R_Axial_DIN0207_L6.3mm_D2.5mm_P7.62mm_Horizontal
Connections:
- net A0: now also U2.49 (IO)
- net A1: now also U2.50 (IO)
- net A16: now also U2.54 (IO)
- net A17: now also U2.55 (IO)
- net A18: now also U2.56 (IO)
- net A19: now also U2.57 (IO)
- net A2: now also U2.51 (IO)
- net A3: now also U2.52 (IO)
- net FC0: now also U2.77 (IO)
- net FC1: now also U2.79 (IO)
- net FC2: now also U2.80 (IO)
- net IDE_INT: now also U2.18 (IO)
- net IDE_RDY: now also U2.22 (IO)
- net R/W: now also U2.67 (IO)
- net SIZ0: now also U2.70 (IO)
- net SIZ1: now also U2.73 (IO)
- net /AS: now also U2.64 (IO)
- net /AVEC: now also U2.81 (IO)
- net /CIIN: now also U2.5 (IO)
- net /CS_DUART: now also U2.12 (IO)
- net /CS_FPU: now also U2.28 (IO)
- net /CS_ROM: now also U2.8 (IO)
- net /CS_SRAM: now also U2.9 (IO)
- net /DS: now also U2.65 (IO)
- net /DSACK0: now also U2.68 (IO)
- net /DSACK0_FPU: now also U2.29 (IO)
- net /DSACK1: now also U2.69 (IO)
- net /DSACK1_FPU: now also U2.30 (IO)
- net /DTACK_DRAM: now also U2.11 (IO)
- net /DTACK_DUART: now also U2.15 (IO)
- net /IACK_DUART: now also U2.17 (IO)
- net /IDE_BUF: now also U2.27 (IO)
- net /IDE_CS0: now also U2.20 (IO)
- net /IDE_CS1: now also U2.21 (IO)
- net /IDE_RD: now also U2.24 (IO)
- net /IDE_WR: now also U2.25 (IO)
- net /IPL0: now also U2.74 (IO)
- net /IPL1: now also U2.75 (IO)
- net /IPL2: now also U2.76 (IO)
- net /IRQ_DUART: now also U2.16 (IO)
- net /RESET: now also U2.4 (IO)
- net /STERM: now also U2.6 (IO)
- net /BERR: now reaches U1.H1 (/BERR)
- net A30: now reaches U1.A3 (A30)
- net A30: now also U2.61 (IO)
- net A28: now reaches U1.A4 (A28)
- net A28: now also U2.58 (IO)
- net A31: now reaches U1.B3 (A31)
- net A31: now also U2.63 (IO)
- net A29: now reaches U1.B4 (A29)
- net A29: now also U2.60 (IO)
- no-connect marks 18 -> 14
Other:
- note added: "TODO: could get away with a lot fewer address pins here Just make sure the DRAM controller has all the signals it needs to decode its own address range (AS, DS, IACK, SIZ? etc.)"
- note added: "TODO: maybe better to put the GPIO and other peripherals on a daughter card"
- note added: "TODO: no expansion CS"
- note removed: "TODO: Run CPU clock through CPLD?"
