File: hardware/mackerel-30-proto/mackerel-30-proto.kicad_pcb (KiCad board)
At the start: 4 copper layers, 200 x 140 mm, 111 parts, among them J1 Conn_01x02, J10 Conn_02x03_Odd_Even, J11 Conn_02x05_Odd_Even, J12 Screw_Terminal_01x04, J13 Conn_02x20_Odd_Even, J14 DIN41612_03x32_ABC, J2 Conn_01x02, J3 Conn_02x05_Odd_Even, J4 Conn_01x06, J5 Conn_01x06, J6 Conn_02x10_Odd_Even, J7 Barrel_Jack_MountingPin, J8 Conn_02x03_Odd_Even, J9 Conn_02x03_Odd_Even, SW1 SW_Push, U1 MC68030RC, U10 SIMM72, U11 MC68882, U12 74HC245, U13 74HC245, U14 74HC245, U15 74HC245, U16 74HC245, U17 74HC245, U18 74HC245, U19 74HC245, U2 EPM7128, U20 74HC245, U3 SST39SF040, U4 AS6C4008-55PCN, U5 XR68C681, U6 LM2576T-5, U7 AMS1117-3.3, U8 DS1233, U9 EPM7128, X1 CXO_DIP14, X2 3.6864MHz, X3 CXO_DIP14

Commit message: Routed power supply section
Parts:
- removed the C37 at (-37.2, 39.7)
- U4: footprint Package_DIP:DIP-32_W15.24mm -> Package_DIP:DIP-32_W15.24mm_Socket
- moved C25 241.5 mm to (57.5, 44.9)
- moved C23 232.4 mm to (46.4, 44.9)
- moved C24 224.5 mm to (40.3, 45.1), turned to 90 degrees
- moved J9 223.3 mm to (52.3, 53.1)
- moved HS1 219.9 mm to (53.6, 21.3)
- moved C26 218.0 mm to (34.3, 45.1), turned to 90 degrees
- moved D2 215.4 mm to (43.1, 37.7), turned to 90 degrees
- moved J10 209.5 mm to (45.2, 53.1)
- moved L1 206.5 mm to (50.9, 33.6)
- moved J8 203.4 mm to (30.3, 25.3), turned to 90 degrees
- moved U6 202.2 mm to (50.1, 24.5)
- moved U7 194.1 mm to (38.0, 50.9)
- moved C37 64.7 mm to (34.8, 61.6), turned to 90 degrees
- moved J4 38.0 mm to (67.4, -5.44)
- moved J5 38.0 mm to (67.4, -10.8)
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- renumbered C38 to C37, U19 to U14, U16 to U15, U18 to U16, U14 to U17, U15 to U18, U17 to U19
Routing:
- net +12V: track 0.00 -> 71.9 mm
- net +3.3V: track 0.00 -> 25.4 mm
- net GND: track 0.00 -> 9.52 mm
- net Net-(D2-K): track 0.00 -> 9.47 mm
Other:
- board size 200 x 140 mm -> 210 x 140 mm
- board text added: "12V"
- board text added: "12VDC"
- board text added: "3V3"
- board text added: "5V"
- board text added: "GND"

Commit message: Routed IDE connector
Parts:
- moved R19 259.6 mm to (149.4, 174.3)
- moved R20 259.6 mm to (149.4, 178.3)
- moved R21 259.6 mm to (149.4, 182.4)
- moved R22 259.6 mm to (149.4, 186.4)
- moved R23 140.0 mm to (42.7, 97.8), turned to 180 degrees
- moved R24 139.6 mm to (42.7, 94.3), turned to 180 degrees
- moved C36 133.6 mm to (45.7, 68.0), turned to -90 degrees
- moved C35 132.6 mm to (45.7, 101.2), turned to -90 degrees
- moved R25 123.0 mm to (21.4, 129.0)
- moved D4 115.7 mm to (23.9, 134.1)
- moved D1 55.4 mm to (-197.0, 2.72)
- moved J14 54.7 mm to (43.7, 210.6)
- moved U14 54.7 mm to (102.7, 176.6)
- moved U15 54.7 mm to (67.4, 176.6)
- moved U16 54.7 mm to (90.9, 176.6)
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Routing:
- net IDE_D15: track 0.00 -> 36.6 mm
- net IDE_D13: track 0.00 -> 36.6 mm
- net IDE_D8: track 0.00 -> 36.5 mm
- net IDE_D10: track 0.00 -> 36.5 mm
- net IDE_D9: track 0.00 -> 36.5 mm
- net IDE_D12: track 0.00 -> 36.5 mm
- net IDE_D14: track 0.00 -> 36.5 mm
- net IDE_D11: track 0.00 -> 36.4 mm
- net /IDE_BUF: track 0.00 -> 34.3 mm
- net R/W: track 0.00 -> 34.3 mm
- net IDE_RDY: track 0.00 -> 16.5 mm
- net IDE_INT: track 0.00 -> 15.8 mm
- net IDE_D7: track 0.00 -> 10.2 mm
- net IDE_D6: track 0.00 -> 10.2 mm
- net IDE_D4: track 0.00 -> 10.2 mm
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Other:
- board text added: "IDE ACT"

Commit message: Routed ROM and SRAM
Parts:
- removed the U14 at (102.7, 176.6)
- removed the U15 at (67.4, 176.6)
- removed U19, U20: 74HC245, Package_DIP:DIP-20_W7.62mm_Socket
- moved R17 441.7 mm to (204.9, 171.0)
- moved R18 441.7 mm to (230.3, 181.7)
- moved SW1 441.7 mm to (242.8, 171.2)
- moved C27 441.7 mm to (255.3, 177.9)
- moved D1 441.7 mm to (208.8, 177.2)
- moved D3 441.7 mm to (232.2, 173.6)
- moved U8 441.7 mm to (255.7, 173.6)
- moved R1 433.9 mm to (236.0, 120.6)
- moved R10 381.0 mm to (179.2, 171.1)
- moved R11 381.0 mm to (179.2, 175.1)
- moved R12 381.0 mm to (179.2, 179.2)
- moved R13 381.0 mm to (179.2, 183.2)
- moved R15 215.5 mm to (96.2, 48.2)
- moved R16 215.5 mm to (96.2, 52.3)
- moved C20 204.1 mm to (94.2, 86.0), turned to -90 degrees
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- renumbered U16 to U14, U17 to U15, U18 to U16
Routing:
- net D28: track 0.00 -> 69.5 mm, vias 0 -> 2
- net Net-(D4-K): track 0.00 -> 68.7 mm
- net D29: track 0.00 -> 67.7 mm, vias 0 -> 2
- net D30: track 0.00 -> 66.0 mm, vias 0 -> 2
- net D31: track 0.00 -> 62.0 mm, vias 0 -> 1
- net D27: track 0.00 -> 55.6 mm
- net Net-(U3-PGM): track 0.00 -> 44.6 mm, vias 0 -> 1
- net GND: track 9.52 -> 53.5 mm
- net D26: track 0.00 -> 38.6 mm
- net D25: track 0.00 -> 38.6 mm
- net D24: track 0.00 -> 38.6 mm
- net A15: track 0.00 -> 38.2 mm
- net A6: track 0.00 -> 22.9 mm
- net A4: track 0.00 -> 22.9 mm
- net A2: track 0.00 -> 22.9 mm
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- added copper zone on In2.Cu, net +5V
- added copper zone on In1.Cu, net GND
Other:
- board text added: "DUART"
- board text added: "IP0"
- board text added: "IP1"
- board text added: "IP2"
- board text added: "IP3"
- board text added: "IP4"
- board text added: "IP5"
- board text added: "OP2"
- board text added: "OP3"
- board text added: "OP4"
- board text added: "OP5"
- board text added: "OP6"
- board text added: "OP7"
- board text added: "ROM"
- board text added: "RTSA"
- board text added: "RTSB"
- board text added: "RXA"
- board text added: "RXB"
- board text added: "SRAM"
- board text added: "TXA"
- board text added: "TXB"

Commit message: Routed DUART serial and GPIO
Parts:
- added R26: 4k7, Resistor_THT:R_Axial_DIN0207_L6.3mm_D2.5mm_P7.62mm_Horizontal, F.Cu at (132.8, 87.5)
- added R27: 4k7, Resistor_THT:R_Axial_DIN0207_L6.3mm_D2.5mm_P7.62mm_Horizontal, F.Cu at (132.8, 91.5)
- moved R2 299.6 mm to (253.5, 88.8)
- moved R3 299.6 mm to (253.5, 92.9)
- moved R4 299.6 mm to (253.5, 96.9)
- moved R5 299.6 mm to (253.5, 101.0)
- moved R6 299.6 mm to (253.5, 105.0)
- moved R7 299.6 mm to (253.5, 109.1)
- moved R8 299.6 mm to (253.5, 113.1)
- moved R9 299.6 mm to (253.5, 117.2)
- moved J1 266.7 mm to (244.1, 136.3)
- moved J2 266.7 mm to (248.7, 136.3)
- moved C22 134.8 mm to (97.3, 55.9)
- moved C21 120.1 mm to (82.4, 44.9)
- moved C1 71.4 mm to (-59.6, 24.6)
- moved C10 71.4 mm to (-51.4, 35.0)
- moved C11 71.4 mm to (-51.4, 38.4)
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Connections:
- U11 pad 18: +5V -> Net-(U11-/SIZE)
- U11 pad 26: +5V -> Net-(U11-A0)
Routing:
- net OP7: track 0.00 -> 97.0 mm, vias 0 -> 1
- net OP5: track 0.00 -> 86.2 mm, vias 0 -> 1
- net OP3: track 0.00 -> 83.0 mm, vias 0 -> 2
- net A1: track 22.9 -> 98.6 mm, vias 0 -> 1
- net A2: track 22.9 -> 91.8 mm, vias 0 -> 1
- net D26: track 38.6 -> 107.0 mm, vias 0 -> 1
- net D27: track 55.6 -> 121.3 mm, vias 0 -> 1
- net A3: track 22.9 -> 84.7 mm, vias 0 -> 1
- net D24: track 38.6 -> 99.4 mm, vias 0 -> 1
- net +3.3V: track 24.4 -> 81.0 mm
- net D25: track 38.6 -> 93.3 mm, vias 0 -> 1
- net D28: track 69.5 -> 124.2 mm, vias 2 -> 3
- net A4: track 22.9 -> 76.9 mm, vias 0 -> 1
- net D30: track 66.0 -> 118.9 mm, vias 2 -> 3
- net D29: track 67.7 -> 119.6 mm, vias 2 -> 3
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Other:
- board text added: "3.6864 MHz"

Commit message: Rough routing of data bus to FPU and RAM
Parts:
- added C28: 0.1uF, Capacitor_THT:C_Disc_D4.3mm_W1.9mm_P5.00mm, F.Cu at (172.3, 38.2)
- added C29: 0.1uF, Capacitor_THT:C_Disc_D4.3mm_W1.9mm_P5.00mm, F.Cu at (182.5, 38.2)
- added C30: 0.1uF, Capacitor_THT:C_Disc_D4.3mm_W1.9mm_P5.00mm, F.Cu at (195.2, 38.2)
- added C31: 0.1uF, Capacitor_THT:C_Disc_D4.3mm_W1.9mm_P5.00mm, F.Cu at (164.9, 63.3)
- added C32: 0.1uF, Capacitor_THT:C_Disc_D4.3mm_W1.9mm_P5.00mm, F.Cu at (177.4, 78.3)
- added C33: 0.1uF, Capacitor_THT:C_Disc_D4.3mm_W1.9mm_P5.00mm, F.Cu at (185.0, 78.3)
- added C34: 0.1uF, Capacitor_THT:C_Disc_D4.3mm_W1.9mm_P5.00mm, F.Cu at (197.4, 78.4)
- added C35: 0.1uF, Capacitor_THT:C_Disc_D4.3mm_W1.9mm_P5.00mm, F.Cu at (205.0, 53.1)
- added C46: 0.1uF, Capacitor_THT:C_Disc_D4.3mm_W1.9mm_P5.00mm, F.Cu at (149.5, 116.5)
- C1, C10, C2, C3, C4, C5, C6, C7, C8, C9: footprint Capacitor_THT:C_Disc_D4.3mm_W1.9mm_P5.00mm -> Capacitor_SMD:C_1206_3216Metric_Pad1.33x1.80mm_HandSolder; moved to B.Cu
- moved C6 259.8 mm to (190.0, 114.0), turned to 90 degrees
- moved C7 256.9 mm to (191.1, 109.3), turned to 180 degrees
- moved C5 255.5 mm to (184.0, 115.7)
- moved C9 252.7 mm to (191.0, 102.9), turned to 180 degrees
- moved C8 252.3 mm to (188.7, 105.5), turned to 180 degrees
- moved C2 251.4 mm to (178.8, 108.0), turned to 180 degrees
- moved C3 251.1 mm to (178.8, 110.5)
- moved C1 251.0 mm to (179.0, 102.9)
- moved C4 250.9 mm to (178.8, 113.1)
- moved C10 244.2 mm to (183.9, 100.2)
- moved C16 198.4 mm to (154.1, 55.7), turned to 90 degrees
- moved C17 193.9 mm to (146.5, 78.2)
- moved C15 187.6 mm to (144.2, 38.2)
- moved C40 183.7 mm to (149.6, 93.6), turned to -90 degrees
- moved C39 183.5 mm to (134.8, 124.1)
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- renumbered C28 to C36, C29 to C37, C30 to C38, C31 to C39, C32 to C40, C33 to C41, C34 to C42, C35 to C43, C36 to C44, C37 to C45, R26 to R23, R27 to R24, R23 to R25, R24 to R26, R25 to R27
Connections:
- U9 pad 33: A0 -> A1
- U9 pad 34: A1 -> A0
Routing:
- net D17: track 0.00 -> 197.7 mm, vias 0 -> 2
- net D19: track 0.00 -> 197.1 mm, vias 0 -> 2
- net D18: track 0.00 -> 191.6 mm, vias 0 -> 2
- net D23: track 0.00 -> 190.5 mm, vias 0 -> 3
- net D16: track 0.00 -> 189.7 mm, vias 0 -> 2
- net D22: track 0.00 -> 187.1 mm, vias 0 -> 2
- net D21: track 0.00 -> 186.0 mm, vias 0 -> 2
- net D20: track 0.00 -> 185.4 mm, vias 0 -> 2
- net D30: track 118.9 -> 297.4 mm, vias 3 -> 6
- net D31: track 111.6 -> 284.6 mm, vias 2 -> 5
- net D1: track 0.00 -> 173.0 mm, vias 0 -> 3
- net D29: track 119.6 -> 291.4 mm, vias 3 -> 6
- net D28: track 124.2 -> 292.5 mm, vias 3 -> 6
- net D27: track 121.3 -> 287.3 mm, vias 1 -> 4
- net D26: track 107.0 -> 272.0 mm, vias 1 -> 4
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Other:
- board size 210 x 140 mm -> 215 x 140 mm
- board text added: "DRAM CLOCK"
- board text added: "DRAM Controller"
- board text added: "MC68030"
- board text added: "MC68882 FPU"
- board text added: "SYS CLOCK"
- board text added: "System Controller"
