File: hardware/mackerel-30-proto/low_mem.kicad_sch (KiCad schematic)
At the start: 4 parts, among them U1 SST39SF040, U2 AS6C4008-55PCN

Commit message: Add power and DUART
Parts:
- renumbered U1 to U3, U2 to U4
Changed lines of the file:
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@@
 		(dnp no)
 		(fields_autoplaced yes)
-		(property "Reference" "U2"
+		(property "Reference" "U4"
 			(at 185.0741 39.37 0)
 			(effects
@@
 		(dnp no)
 		(fields_autoplaced yes)
-		(property "Reference" "#PWR01"
+		(property "Reference" "#PWR011"
 			(at 82.55 43.18 0)
 			(effects
@@
 		(dnp no)
 		(fields_autoplaced yes)
-		(property "Reference" "U1"
+		(property "Reference" "U3"
 			(at 84.7441 39.37 0)
 			(effects
@@
 		(dnp no)
 		(fields_autoplaced yes)
-		(property "Reference" "#PWR03"
+		(property "Reference" "#PWR012"
 			(at 82.55 116.84 0)
 			(effects

Commit message: Add 68882 FPU symbol
Parts:
- added R5: 4k7, symbol Device:R
- U4: footprint Package_DIP:DIP-32_W15.24mm_Socket -> Package_DIP:DIP-32_W15.24mm
Connections:
- net +5V: now also R5.1
- net GND: now also U3.24 (OE), U4.24 (OE#)
- net /CS_SRAM: now reaches U4.22 (CE#)
- net /CS_ROM: now reaches U3.22 (CE)
- net at U3.31 (PGM): now also R5.2

Commit message: Wired most of the control signals for the CPU and DRAM
Parts:
- R14: renamed from R5; footprint (none) -> Resistor_THT:R_Axial_DIN0207_L6.3mm_D2.5mm_P7.62mm_Horizontal
Changed lines of the file:
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@@
 		(dnp no)
 		(fields_autoplaced yes)
-		(property "Reference" "#PWR011"
+		(property "Reference" "#PWR017"
 			(at 29.21 38.1 0)
 			(effects
@@
 			(project ""
 				(path "/9307474f-ec99-494d-b4c9-fbd0b10ce86a/2233f134-711f-41c0-bcb6-ed6edb8cdb44"
-					(reference "#PWR011")
+					(reference "#PWR017")
 					(unit 1)
 				)
@@
 		(on_board yes)
 		(dnp no)
-		(property "Reference" "R5"
+		(property "Reference" "R14"
 			(at 48.768 89.408 90)
 			(effects
@@
 			)
 		)
-		(property "Footprint" ""
+		(property "Footprint" "Resistor_THT:R_Axial_DIN0207_L6.3mm_D2.5mm_P7.62mm_Horizontal"
 			(at 49.022 87.63 90)
 			(effects
@@
 			(project ""
 				(path "/9307474f-ec99-494d-b4c9-fbd0b10ce86a/2233f134-711f-41c0-bcb6-ed6edb8cdb44"
-					(reference "R5")
+					(reference "R14")
 					(unit 1)
 				)
@@
 		(dnp no)
 		(fields_autoplaced yes)
-		(property "Reference" "#PWR014"
+		(property "Reference" "#PWR020"
 			(at 82.55 43.18 0)
 			(effects
@@
 			(project ""
 				(path "/9307474f-ec99-494d-b4c9-fbd0b10ce86a/2233f134-711f-41c0-bcb6-ed6edb8cdb44"
-					(reference "#PWR014")
+					(reference "#PWR020")
 					(unit 1)
 				)
@@
 		(dnp no)
 		(fields_autoplaced yes)
-		(property "Reference" "#PWR016"
+		(property "Reference" "#PWR022"
 			(at 182.88 45.72 0)
 			(effects
@@
 			(project "mackerel-30-proto"
 				(path "/9307474f-ec99-494d-b4c9-fbd0b10ce86a/2233f134-711f-41c0-bcb6-ed6edb8cdb44"
-					(reference "#PWR016")
+					(reference "#PWR022")
 					(unit 1)
 				)
@@
 		(dnp no)
 		(fields_autoplaced yes)
-		(property "Reference" "#PWR012"
+		(property "Reference" "#PWR018"
 			(at 36.83 50.8 0)
 			(effects
@@
 			(project "mackerel-30-proto"
 				(path "/9307474f-ec99-494d-b4c9-fbd0b10ce86a/2233f134-711f-41c0-bcb6-ed6edb8cdb44"
-					(reference "#PWR012")
+					(reference "#PWR018")
 					(unit 1)
 				)
@@
 		(dnp no)
 		(fields_autoplaced yes)
-		(property "Reference" "#PWR017"
+		(property "Reference" "#PWR023"
 			(at 182.88 106.68 0)
 			(effects
@@
 			(project "mackerel-30-proto"
 				(path "/9307474f-ec99-494d-b4c9-fbd0b10ce86a/2233f134-711f-41c0-bcb6-ed6edb8cdb44"
-					(reference "#PWR017")
+					(reference "#PWR023")
 					(unit 1)
 				)
@@
 		(dnp no)
 		(fields_autoplaced yes)
-		(property "Reference" "#PWR015"
+		(property "Reference" "#PWR021"
 			(at 82.55 121.92 0)
 			(effects
@@
 			(project ""
 				(path "/9307474f-ec99-494d-b4c9-fbd0b10ce86a/2233f134-711f-41c0-bcb6-ed6edb8cdb44"
-					(reference "#PWR015")
+					(reference "#PWR021")
 					(unit 1)
 				)
@@
 		(dnp no)
 		(fields_autoplaced yes)
-		(property "Reference" "#PWR013"
+		(property "Reference" "#PWR019"
 			(at 50.8 87.63 0)
 			(effects
@@
 			(project ""
 				(path "/9307474f-ec99-494d-b4c9-fbd0b10ce86a/2233f134-711f-41c0-bcb6-ed6edb8cdb44"
-					(reference "#PWR013")
-					(unit 1)
-				)
+					(reference "#PWR019")
+					(unit 1)
+				)

Commit message: A bit of cleanup
Parts:
- renumbered R14 to R15
Changed lines of the file:
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@@
 		(on_board yes)
 		(dnp no)
-		(property "Reference" "R14"
+		(property "Reference" "R15"
 			(at 48.768 89.408 90)
 			(effects
@@
 			(project ""
 				(path "/9307474f-ec99-494d-b4c9-fbd0b10ce86a/2233f134-711f-41c0-bcb6-ed6edb8cdb44"
-					(reference "R14")
+					(reference "R15")
 					(unit 1)
 				)

Commit message: positioning
Parts:
- C19, C20: footprint Capacitor_SMD:C_1210_3225Metric_Pad1.33x2.70mm_HandSolder -> Capacitor_SMD:C_1206_3216Metric_Pad1.33x1.80mm_HandSolder
- R15: footprint Resistor_THT:R_Axial_DIN0207_L6.3mm_D2.5mm_P7.62mm_Horizontal -> Resistor_SMD:R_0805_2012Metric_Pad1.20x1.40mm_HandSolder
Changed lines of the file:
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@@
 			)
 		)
-		(property "Footprint" "Resistor_THT:R_Axial_DIN0207_L6.3mm_D2.5mm_P7.62mm_Horizontal"
+		(property "Footprint" "Resistor_SMD:R_0805_2012Metric_Pad1.20x1.40mm_HandSolder"
 			(at 49.022 87.63 90)
 			(effects
@@
 			)
 		)
-		(property "Footprint" "Capacitor_SMD:C_1210_3225Metric_Pad1.33x2.70mm_HandSolder"
+		(property "Footprint" "Capacitor_SMD:C_1206_3216Metric_Pad1.33x1.80mm_HandSolder"
 			(at 36.83 43.4848 0)
 			(effects
@@
 			)
 		)
-		(property "Footprint" "Capacitor_SMD:C_1210_3225Metric_Pad1.33x2.70mm_HandSolder"
+		(property "Footprint" "Capacitor_SMD:C_1206_3216Metric_Pad1.33x1.80mm_HandSolder"
 			(at 36.83 38.4048 0)
 			(effects

Commit message: rough layout of the PCB components
Parts:
- C19, C20: footprint Capacitor_SMD:C_1206_3216Metric_Pad1.33x1.80mm_HandSolder -> Capacitor_THT:C_Disc_D4.3mm_W1.9mm_P5.00mm
- R14: renamed from R15; footprint Resistor_SMD:R_0805_2012Metric_Pad1.20x1.40mm_HandSolder -> Resistor_THT:R_Axial_DIN0207_L6.3mm_D2.5mm_P7.62mm_Horizontal
Changed lines of the file:
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@@
 		(on_board yes)
 		(dnp no)
-		(property "Reference" "R15"
+		(property "Reference" "R14"
 			(at 48.768 89.408 90)
 			(effects
@@
 			)
 		)
-		(property "Footprint" "Resistor_SMD:R_0805_2012Metric_Pad1.20x1.40mm_HandSolder"
+		(property "Footprint" "Resistor_THT:R_Axial_DIN0207_L6.3mm_D2.5mm_P7.62mm_Horizontal"
 			(at 49.022 87.63 90)
 			(effects
@@
 			(project ""
 				(path "/9307474f-ec99-494d-b4c9-fbd0b10ce86a/2233f134-711f-41c0-bcb6-ed6edb8cdb44"
-					(reference "R15")
+					(reference "R14")
 					(unit 1)
 				)
@@
 			)
 		)
-		(property "Footprint" "Capacitor_SMD:C_1206_3216Metric_Pad1.33x1.80mm_HandSolder"
+		(property "Footprint" "Capacitor_THT:C_Disc_D4.3mm_W1.9mm_P5.00mm"
 			(at 36.83 43.4848 0)
 			(effects
@@
 			)
 		)
-		(property "Footprint" "Capacitor_SMD:C_1206_3216Metric_Pad1.33x1.80mm_HandSolder"
+		(property "Footprint" "Capacitor_THT:C_Disc_D4.3mm_W1.9mm_P5.00mm"
 			(at 36.83 38.4048 0)
 			(effects

Commit message: Routed power supply section
Parts:
- U4: footprint Package_DIP:DIP-32_W15.24mm -> Package_DIP:DIP-32_W15.24mm_Socket
Changed lines of the file:
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@@
 			)
 		)
-		(property "Footprint" "Package_DIP:DIP-32_W15.24mm"
+		(property "Footprint" "Package_DIP:DIP-32_W15.24mm_Socket"
 			(at 182.88 67.31 0)
 			(effects

Commit message: Mack-30 routed except for expansion header
Parts:
- renumbered C19 to C20, C20 to C21
Changed lines of the file:
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@@
 		(dnp no)
 		(fields_autoplaced yes)
-		(property "Reference" "#PWR017"
+		(property "Reference" "#PWR019"
 			(at 29.21 38.1 0)
 			(effects
@@
 			(project ""
 				(path "/9307474f-ec99-494d-b4c9-fbd0b10ce86a/2233f134-711f-41c0-bcb6-ed6edb8cdb44"
-					(reference "#PWR017")
+					(reference "#PWR019")
 					(unit 1)
 				)
@@
 		(dnp no)
 		(fields_autoplaced yes)
-		(property "Reference" "#PWR020"
+		(property "Reference" "#PWR022"
 			(at 82.55 43.18 0)
 			(effects
@@
 			(project ""
 				(path "/9307474f-ec99-494d-b4c9-fbd0b10ce86a/2233f134-711f-41c0-bcb6-ed6edb8cdb44"
-					(reference "#PWR020")
+					(reference "#PWR022")
 					(unit 1)
 				)
@@
 		(dnp no)
 		(fields_autoplaced yes)
-		(property "Reference" "#PWR022"
+		(property "Reference" "#PWR024"
 			(at 182.88 45.72 0)
 			(effects
@@
 			(project "mackerel-30-proto"
 				(path "/9307474f-ec99-494d-b4c9-fbd0b10ce86a/2233f134-711f-41c0-bcb6-ed6edb8cdb44"
-					(reference "#PWR022")
+					(reference "#PWR024")
 					(unit 1)
 				)
@@
 		(dnp no)
 		(fields_autoplaced yes)
-		(property "Reference" "#PWR018"
+		(property "Reference" "#PWR020"
 			(at 36.83 50.8 0)
 			(effects
@@
 			(project "mackerel-30-proto"
 				(path "/9307474f-ec99-494d-b4c9-fbd0b10ce86a/2233f134-711f-41c0-bcb6-ed6edb8cdb44"
-					(reference "#PWR018")
+					(reference "#PWR020")
 					(unit 1)
 				)
@@
 		(on_board yes)
 		(dnp no)
-		(property "Reference" "C20"
+		(property "Reference" "C21"
 			(at 35.306 43.18 90)
 			(effects
@@
 			(project "mackerel-30-proto"
 				(path "/9307474f-ec99-494d-b4c9-fbd0b10ce86a/2233f134-711f-41c0-bcb6-ed6edb8cdb44"
-					(reference "C20")
+					(reference "C21")
 					(unit 1)
 				)
@@
 		(dnp no)
 		(fields_autoplaced yes)
-		(property "Reference" "#PWR023"
+		(property "Reference" "#PWR025"
 			(at 182.88 106.68 0)
 			(effects
@@
 			(project "mackerel-30-proto"
 				(path "/9307474f-ec99-494d-b4c9-fbd0b10ce86a/2233f134-711f-41c0-bcb6-ed6edb8cdb44"
-					(reference "#PWR023")
+					(reference "#PWR025")
 					(unit 1)
 				)
@@
 		(on_board yes)
 		(dnp no)
-		(property "Reference" "C19"
+		(property "Reference" "C20"
 			(at 35.306 38.1 90)
 			(effects
@@
 			(project "mackerel-30-proto"
 				(path "/9307474f-ec99-494d-b4c9-fbd0b10ce86a/2233f134-711f-41c0-bcb6-ed6edb8cdb44"
-					(reference "C19")
+					(reference "C20")
 					(unit 1)
 				)
@@
 		(dnp no)
 		(fields_autoplaced yes)
-		(property "Reference" "#PWR021"
+		(property "Reference" "#PWR023"
 			(at 82.55 121.92 0)
 			(effects
@@
 			(project ""
 				(path "/9307474f-ec99-494d-b4c9-fbd0b10ce86a/2233f134-711f-41c0-bcb6-ed6edb8cdb44"
-					(reference "#PWR021")
+					(reference "#PWR023")
 					(unit 1)
 				)
@@
 		(dnp no)
 		(fields_autoplaced yes)
-		(property "Reference" "#PWR019"
+		(property "Reference" "#PWR021"
 			(at 50.8 87.63 0)
 			(effects
@@
 			(project ""
 				(path "/9307474f-ec99-494d-b4c9-fbd0b10ce86a/2233f134-711f-41c0-bcb6-ed6edb8cdb44"
-					(reference "#PWR019")
-					(unit 1)
-				)
+					(reference "#PWR021")
+					(unit 1)
+				)
