File: hardware/mackerel-30-proto/low_mem.kicad_sch (KiCad schematic)
At the start: 5 parts, among them U3 SST39SF040, U4 AS6C4008-55PCN

Commit message: PCB cleanup
Other:
- company: (none) -> Colin Maykish
- title: (none) -> Mackerel-30
Changed lines of the file:
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@@
 	(generator_version "8.0")
 	(paper "A")
+	(title_block
+		(title "Mackerel-30")
+		(date "2024-11-09")
+		(rev "0.1")
+		(company "Colin Maykish")
+	)
 	(junction
 		(at 82.55 113.03)
