File: hardware/mackerel-30-proto/power.kicad_sch (KiCad schematic)
At the start: 18 parts, among them J1 Barrel_Jack_MountingPin, J2 Conn_02x03_Odd_Even, J3 Conn_02x03_Odd_Even, J4 Conn_02x03_Odd_Even, U6 LM2576T-5, U7 AMS1117-3.3

Commit message: Add 68882 FPU symbol
Parts:
- renumbered C25 to C24, C24 to C25, D2 to D1, D1 to D2, J1 to J2, J2 to J3, J3 to J4, J4 to J5, R3 to R8
Changed lines of the file:
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@@
 		(dnp no)
 		(fields_autoplaced yes)
-		(property "Reference" "J2"
+		(property "Reference" "J3"
 			(at 172.72 107.95 0)
 			(effects
@@
 			(project "mackerel-30-proto"
 				(path "/9307474f-ec99-494d-b4c9-fbd0b10ce86a/89853077-d9a7-463a-b48b-4d81b0ac6897"
-					(reference "J2")
+					(reference "J3")
 					(unit 1)
 				)
@@
 		(dnp no)
 		(fields_autoplaced yes)
-		(property "Reference" "#PWR025"
+		(property "Reference" "#PWR032"
 			(at 97.79 49.53 0)
 			(effects
@@
 			(project "mackerel-30-proto"
 				(path "/9307474f-ec99-494d-b4c9-fbd0b10ce86a/89853077-d9a7-463a-b48b-4d81b0ac6897"
-					(reference "#PWR025")
+					(reference "#PWR032")
 					(unit 1)
 				)
@@
 		(on_board yes)
 		(dnp no)
-		(property "Reference" "D1"
+		(property "Reference" "D2"
 			(at 85.598 55.118 90)
 			(effects
@@
 			(project "mackerel-30-proto"
 				(path "/9307474f-ec99-494d-b4c9-fbd0b10ce86a/89853077-d9a7-463a-b48b-4d81b0ac6897"
-					(reference "D1")
+					(reference "D2")
 					(unit 1)
 				)
@@
 		(dnp no)
 		(fields_autoplaced yes)
-		(property "Reference" "#PWR031"
+		(property "Reference" "#PWR029"
 			(at 57.15 124.46 0)
 			(effects
@@
 			(project "mackerel-30-proto"
 				(path "/9307474f-ec99-494d-b4c9-fbd0b10ce86a/89853077-d9a7-463a-b48b-4d81b0ac6897"
-					(reference "#PWR031")
+					(reference "#PWR029")
 					(unit 1)
 				)
@@
 		(dnp no)
 		(fields_autoplaced yes)
-		(property "Reference" "#PWR034"
+		(property "Reference" "#PWR037"
 			(at 186.69 118.11 0)
 			(effects
@@
 			(project "mackerel-30-proto"
 				(path "/9307474f-ec99-494d-b4c9-fbd0b10ce86a/89853077-d9a7-463a-b48b-4d81b0ac6897"
-					(reference "#PWR034")
+					(reference "#PWR037")
 					(unit 1)
 				)
@@
 		(on_board yes)
 		(dnp no)
-		(property "Reference" "#PWR029"
+		(property "Reference" "#PWR034"
 			(at 105.41 152.4 0)
 			(effects
@@
 			(project "mackerel-30-proto"
 				(path "/9307474f-ec99-494d-b4c9-fbd0b10ce86a/89853077-d9a7-463a-b48b-4d81b0ac6897"
-					(reference "#PWR029")
+					(reference "#PWR034")
 					(unit 1)
 				)
@@
 		(dnp no)
 		(fields_autoplaced yes)
-		(property "Reference" "#PWR033"
+		(property "Reference" "#PWR036"
 			(at 179.07 125.73 0)
 			(effects
@@
 			(project "mackerel-30-proto"
 				(path "/9307474f-ec99-494d-b4c9-fbd0b10ce86a/89853077-d9a7-463a-b48b-4d81b0ac6897"
-					(reference "#PWR033")
+					(reference "#PWR036")
 					(unit 1)
 				)
@@
 		(on_board yes)
 		(dnp no)
-		(property "Reference" "C24"
+		(property "Reference" "C25"
 			(at 98.552 52.07 0)
 			(effects
@@
 			(project "mackerel-30-proto"
 				(path "/9307474f-ec99-494d-b4c9-fbd0b10ce86a/89853077-d9a7-463a-b48b-4d81b0ac6897"
-					(reference "C24")
+					(reference "C25")
 					(unit 1)
 				)
@@
 		(dnp no)
 		(fields_autoplaced yes)
-		(property "Reference" "#PWR037"
+		(property "Reference" "#PWR040"
 			(at 219.71 125.73 0)
 			(effects
@@
 			(project "mackerel-30-proto"
 				(path "/9307474f-ec99-494d-b4c9-fbd0b10ce86a/89853077-d9a7-463a-b48b-4d81b0ac6897"
-					(reference "#PWR037")
+					(reference "#PWR040")
 					(unit 1)
 				)
@@
 		(dnp no)
 		(fields_autoplaced yes)
-		(property "Reference" "D2"
+		(property "Reference" "D1"
 			(at 60.706 114.6174 90)
 			(effects
@@
 			(project "mackerel-30-proto"
 				(path "/9307474f-ec99-494d-b4c9-fbd0b10ce86a/89853077-d9a7-463a-b48b-4d81b0ac6897"
-					(reference "D2")
+					(reference "D1")
 					(unit 1)
 				)
@@
 		(dnp no)
 		(fields_autoplaced yes)
-		(property "Reference" "J1"
+		(property "Reference" "J2"
 			(at 38.1 39.37 0)
 			(effects
@@
 			(project "mackerel-30-proto"
 				(path "/9307474f-ec99-494d-b4c9-fbd0b10ce86a/89853077-d9a7-463a-b48b-4d81b0ac6897"
-					(reference "J1")
+					(reference "J2")
 					(unit 1)
 				)
@@
 		(dnp no)
 		(fields_autoplaced yes)
-		(property "Reference" "#PWR028"
+		(property "Reference" "#PWR033"
 			(at 97.79 166.37 0)
 			(effects
@@
 			(project "mackerel-30-proto"
 				(path "/9307474f-ec99-494d-b4c9-fbd0b10ce86a/89853077-d9a7-463a-b48b-4d81b0ac6897"
-					(reference "#PWR028")
+					(reference "#PWR033")
 					(unit 1)
 				)
@@
 		(dnp no)
 		(fields_autoplaced yes)
-		(property "Reference" "R3"
+		(property "Reference" "R8"
 			(at 59.69 105.4099 0)
 			(effects
@@
 			(project "mackerel-30-proto"
 				(path "/9307474f-ec99-494d-b4c9-fbd0b10ce86a/89853077-d9a7-463a-b48b-4d81b0ac6897"
-					(reference "R3")
+					(reference "R8")
 					(unit 1)
 				)
@@
 		(dnp no)
 		(fields_autoplaced yes)
-		(property "Reference" "#PWR024"
+		(property "Reference" "#PWR030"
 			(at 77.47 64.77 0)
 			(effects
@@
 			(project "mackerel-30-proto"
 				(path "/9307474f-ec99-494d-b4c9-fbd0b10ce86a/89853077-d9a7-463a-b48b-4d81b0ac6897"
-					(reference "#PWR024")
+					(reference "#PWR030")
 					(unit 1)
 				)
@@
 		(dnp no)
 		(fields_autoplaced yes)
-		(property "Reference" "#PWR035"
+		(property "Reference" "#PWR038"
 			(at 199.39 125.73 0)
 			(effects
@@
 			(project "mackerel-30-proto"
 				(path "/9307474f-ec99-494d-b4c9-fbd0b10ce86a/89853077-d9a7-463a-b48b-4d81b0ac6897"
-					(reference "#PWR035")
+					(reference "#PWR038")
 					(unit 1)
 				)
@@
 		(on_board yes)
 		(dnp no)
-		(property "Reference" "#PWR027"
+		(property "Reference" "#PWR031"
 			(at 90.17 152.4 0)
 			(effects
@@
 			(project "mackerel-30-proto"
 				(path "/9307474f-ec99-494d-b4c9-fbd0b10ce86a/89853077-d9a7-463a-b48b-4d81b0ac6897"
-					(reference "#PWR027")
+					(reference "#PWR031")
 					(unit 1)
 				)
@@
 		(dnp no)
 		(fields_autoplaced yes)
-		(property "Reference" "#PWR032"
+		(property "Reference" "#PWR035"
 			(at 166.37 118.11 0)
 			(effects
@@
 			(project "mackerel-30-proto"
 				(path "/9307474f-ec99-494d-b4c9-fbd0b10ce86a/89853077-d9a7-463a-b48b-4d81b0ac6897"
-					(reference "#PWR032")
+					(reference "#PWR035")
 					(unit 1)
 				)
@@
 		(dnp no)
 		(fields_autoplaced yes)
-		(property "Reference" "#PWR030"
+		(property "Reference" "#PWR028"
 			(at 57.15 106.68 0)
 			(effects
@@
 			(project "mackerel-30-proto"
 				(path "/9307474f-ec99-494d-b4c9-fbd0b10ce86a/89853077-d9a7-463a-b48b-4d81b0ac6897"
-					(reference "#PWR030")
+					(reference "#PWR028")
 					(unit 1)
 				)
@@
 		(dnp no)
 		(fields_autoplaced yes)
-		(property "Reference" "J4"
+		(property "Reference" "J5"
 			(at 213.36 107.95 0)
 			(effects
@@
 			(project "mackerel-30-proto"
 				(path "/9307474f-ec99-494d-b4c9-fbd0b10ce86a/89853077-d9a7-463a-b48b-4d81b0ac6897"
-					(reference "J4")
+					(reference "J5")
 					(unit 1)
 				)
@@
 		(dnp no)
 		(fields_autoplaced yes)
-		(property "Reference" "J3"
+		(property "Reference" "J4"
 			(at 193.04 107.95 0)
 			(effects
@@
 			(project "mackerel-30-proto"
 				(path "/9307474f-ec99-494d-b4c9-fbd0b10ce86a/89853077-d9a7-463a-b48b-4d81b0ac6897"
-					(reference "J3")
+					(reference "J4")
 					(unit 1)
 				)
@@
 		(on_board yes)
 		(dnp no)
-		(property "Reference" "C25"
+		(property "Reference" "C24"
 			(at 86.36 150.4949 0)
 			(effects
@@
 			(project "mackerel-30-proto"
 				(path "/9307474f-ec99-494d-b4c9-fbd0b10ce86a/89853077-d9a7-463a-b48b-4d81b0ac6897"
-					(reference "C25")
+					(reference "C24")
 					(unit 1)
 				)
@@
 		(dnp no)
 		(fields_autoplaced yes)
-		(property "Reference" "#PWR036"
+		(property "Reference" "#PWR039"
 			(at 207.01 118.11 0)
 			(effects
@@
 			(project "mackerel-30-proto"
 				(path "/9307474f-ec99-494d-b4c9-fbd0b10ce86a/89853077-d9a7-463a-b48b-4d81b0ac6897"
-					(reference "#PWR036")
+					(reference "#PWR039")
 					(unit 1)
 				)
@@
 		(dnp no)
 		(fields_autoplaced yes)
-		(property "Reference" "#PWR023"
+		(property "Reference" "#PWR027"
 			(at 50.8 49.53 0)
 			(effects
@@
 			(project "mackerel-30-proto"
 				(path "/9307474f-ec99-494d-b4c9-fbd0b10ce86a/89853077-d9a7-463a-b48b-4d81b0ac6897"
-					(reference "#PWR023")
-					(unit 1)
-				)
+					(reference "#PWR027")
+					(unit 1)
+				)

Commit message: Wired most of the control signals for the CPU and DRAM
Parts:
- removed J3, J4, J5: Conn_02x03_Odd_Even, Connector_PinHeader_2.54mm:PinHeader_2x03_P2.54mm_Vertical, symbol Connector_Generic:Conn_02x03_Odd_Even
- renumbered J2 to J4, R8 to R17

Commit message: A bit of cleanup
Parts:
- renumbered R17 to R18
Changed lines of the file:
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@@
 		(dnp no)
 		(fields_autoplaced yes)
-		(property "Reference" "R17"
+		(property "Reference" "R18"
 			(at 59.69 105.4099 0)
 			(effects
@@
 			(project "mackerel-30-proto"
 				(path "/9307474f-ec99-494d-b4c9-fbd0b10ce86a/89853077-d9a7-463a-b48b-4d81b0ac6897"
-					(reference "R17")
+					(reference "R18")
 					(unit 1)
 				)

Commit message: positioning
Parts:
- added C27: C_Polarized, Capacitor_THT:CP_Radial_D5.0mm_P2.50mm, symbol Device:C_Polarized
- added C28: C, Capacitor_THT:C_Disc_D4.3mm_W1.9mm_P5.00mm, symbol Device:C
- added D3: LED, LED_THT:LED_D5.0mm, symbol Device:LED
- added HS1: Heatsink, Heatsink:Heatsink_Stonecold_HS-S02_13.21x9.53mm, symbol Mechanical:Heatsink
- added J10, J8, J9: Conn_02x03_Odd_Even, Connector_PinHeader_2.54mm:PinHeader_2x03_P2.54mm_Vertical, symbol Connector_Generic:Conn_02x03_Odd_Even
- added R19, R20, R21: R, Resistor_SMD:R_0805_2012Metric_Pad1.20x1.40mm_HandSolder, symbol Device:R
- added SW1: SW_Push, Button_Switch_THT:SW_PUSH_6mm_H5mm, symbol Switch:SW_Push
- added U8: NE555P, Package_DIP:DIP-8_W7.62mm, symbol Timer:NE555P
- R18: footprint Resistor_THT:R_Axial_DIN0207_L6.3mm_D2.5mm_P7.62mm_Horizontal -> Resistor_SMD:R_0805_2012Metric_Pad1.20x1.40mm_HandSolder
- renumbered J4 to J7
Connections:
- net +12V: now also J8.1 (Pin_1), J8.3 (Pin_3), J8.5 (Pin_5)
- net +3.3V: now also J10.1 (Pin_1), J10.3 (Pin_3), J10.5 (Pin_5)
- net +5V: now also C27.1, C28.1, J9.1 (Pin_1), J9.3 (Pin_3), J9.5 (Pin_5), R19.1, R21.1, U8.8 (VCC)
- net GND: now also C28.2, J10.2 (Pin_2), J10.4 (Pin_4), J10.6 (Pin_6), J8.2 (Pin_2), J8.4 (Pin_4), J8.6 (Pin_6), J9.2 (Pin_2), J9.4 (Pin_4), J9.6 (Pin_6), R20.2, SW1.1, U8.1 (GND)
- new net: D3.2 (A), R21.2
- new net: C27.2, R20.1, U8.2 (TR), U8.6 (THR)
- new net: R19.2, SW1.2, U8.4 (R)
- new net /RESET: D3.1 (K), U8.3 (Q)
- no-connect marks 1 -> 3
Other:
- note removed: "TODO: better heatsink"
- note removed: "TODO: reset circuit"

Commit message: Add DS1233 for reset
Parts:
- removed C27: C_Polarized, Capacitor_THT:CP_Radial_D5.0mm_P2.50mm, symbol Device:C_Polarized
- removed C28: C, Capacitor_THT:C_Disc_D4.3mm_W1.9mm_P5.00mm, symbol Device:C
- removed R20, R21: R, Resistor_SMD:R_0805_2012Metric_Pad1.20x1.40mm_HandSolder, symbol Device:R
- removed U8: NE555P, Package_DIP:DIP-8_W7.62mm, symbol Timer:NE555P
- added C27: 0.01uF, Capacitor_SMD:C_1206_3216Metric_Pad1.33x1.80mm_HandSolder, symbol Device:C
- added U8: DS1233, Package_TO_SOT_THT:TO-92, symbol mackerel-68k-symbols:DS1233
- R19: value R -> 1k
Connections:
- net +5V: now also U8.3 (VCC)
- net GND: now also SW1.2, C27.2, U8.1 (GND); no longer SW1.1
- net /RESET: now also SW1.1, C27.1, U8.2 (/RESET)
- net at D3.2 (A): now also R19.2
- no-connect marks 3 -> 1
Other:
- moved on the sheet: SW1

Commit message: rough layout of the PCB components
Parts:
- C27: footprint Capacitor_SMD:C_1206_3216Metric_Pad1.33x1.80mm_HandSolder -> Capacitor_THT:C_Disc_D4.3mm_W1.9mm_P5.00mm
- R17: renamed from R18; footprint Resistor_SMD:R_0805_2012Metric_Pad1.20x1.40mm_HandSolder -> Resistor_THT:R_Axial_DIN0207_L6.3mm_D2.5mm_P7.62mm_Horizontal
- R18: renamed from R19; footprint Resistor_SMD:R_0805_2012Metric_Pad1.20x1.40mm_HandSolder -> Resistor_THT:R_Axial_DIN0207_L6.3mm_D2.5mm_P7.62mm_Horizontal
Changed lines of the file:
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@@
 			)
 		)
-		(property "Footprint" "Capacitor_SMD:C_1206_3216Metric_Pad1.33x1.80mm_HandSolder"
+		(property "Footprint" "Capacitor_THT:C_Disc_D4.3mm_W1.9mm_P5.00mm"
 			(at 215.5952 46.99 0)
 			(effects
@@
 		(dnp no)
 		(fields_autoplaced yes)
-		(property "Reference" "R18"
+		(property "Reference" "R17"
 			(at 59.69 105.4099 0)
 			(effects
@@
 			)
 		)
-		(property "Footprint" "Resistor_SMD:R_0805_2012Metric_Pad1.20x1.40mm_HandSolder"
+		(property "Footprint" "Resistor_THT:R_Axial_DIN0207_L6.3mm_D2.5mm_P7.62mm_Horizontal"
 			(at 55.372 106.68 90)
 			(effects
@@
 			(project "mackerel-30-proto"
 				(path "/9307474f-ec99-494d-b4c9-fbd0b10ce86a/89853077-d9a7-463a-b48b-4d81b0ac6897"
-					(reference "R18")
+					(reference "R17")
 					(unit 1)
 				)
@@
 		(dnp no)
 		(fields_autoplaced yes)
-		(property "Reference" "R19"
+		(property "Reference" "R18"
 			(at 228.6 24.1299 0)
 			(effects
@@
 			)
 		)
-		(property "Footprint" "Resistor_SMD:R_0805_2012Metric_Pad1.20x1.40mm_HandSolder"
+		(property "Footprint" "Resistor_THT:R_Axial_DIN0207_L6.3mm_D2.5mm_P7.62mm_Horizontal"
 			(at 224.282 25.4 90)
 			(effects
@@
 			(project "mackerel-30-proto"
 				(path "/9307474f-ec99-494d-b4c9-fbd0b10ce86a/89853077-d9a7-463a-b48b-4d81b0ac6897"
-					(reference "R19")
-					(unit 1)
-				)
+					(reference "R18")
+					(unit 1)
+				)

Commit message: Mack-30 routed except for expansion header
Parts:
- U8: footprint Package_TO_SOT_THT:TO-92 -> Package_TO_SOT_THT:TO-92L_Inline
- renumbered C23 to C24, C24 to C25, C25 to C26, C26 to C27, C27 to C28
Changed lines of the file:
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@@
 		(dnp no)
 		(fields_autoplaced yes)
-		(property "Reference" "#PWR048"
+		(property "Reference" "#PWR050"
 			(at 97.79 49.53 0)
 			(effects
@@
 			(project "mackerel-30-proto"
 				(path "/9307474f-ec99-494d-b4c9-fbd0b10ce86a/89853077-d9a7-463a-b48b-4d81b0ac6897"
-					(reference "#PWR048")
+					(reference "#PWR050")
 					(unit 1)
 				)
@@
 		(on_board yes)
 		(dnp no)
-		(property "Reference" "C26"
+		(property "Reference" "C27"
 			(at 109.22 150.4949 0)
 			(effects
@@
 			(project "mackerel-30-proto"
 				(path "/9307474f-ec99-494d-b4c9-fbd0b10ce86a/89853077-d9a7-463a-b48b-4d81b0ac6897"
-					(reference "C26")
+					(reference "C27")
 					(unit 1)
 				)
@@
 		(dnp no)
 		(fields_autoplaced yes)
-		(property "Reference" "#PWR045"
+		(property "Reference" "#PWR047"
 			(at 57.15 124.46 0)
 			(effects
@@
 			(project "mackerel-30-proto"
 				(path "/9307474f-ec99-494d-b4c9-fbd0b10ce86a/89853077-d9a7-463a-b48b-4d81b0ac6897"
-					(reference "#PWR045")
+					(reference "#PWR047")
 					(unit 1)
 				)
@@
 		(dnp no)
 		(fields_autoplaced yes)
-		(property "Reference" "#PWR042"
+		(property "Reference" "#PWR044"
 			(at 38.1 199.39 0)
 			(effects
@@
 			(project "mackerel-30-proto"
 				(path "/9307474f-ec99-494d-b4c9-fbd0b10ce86a/89853077-d9a7-463a-b48b-4d81b0ac6897"
-					(reference "#PWR042")
+					(reference "#PWR044")
 					(unit 1)
 				)
@@
 		(on_board yes)
 		(dnp no)
-		(property "Reference" "#PWR050"
+		(property "Reference" "#PWR052"
 			(at 105.41 152.4 0)
 			(effects
@@
 			(project "mackerel-30-proto"
 				(path "/9307474f-ec99-494d-b4c9-fbd0b10ce86a/89853077-d9a7-463a-b48b-4d81b0ac6897"
-					(reference "#PWR050")
+					(reference "#PWR052")
 					(unit 1)
 				)
@@
 		(dnp no)
 		(fields_autoplaced yes)
-		(property "Reference" "#PWR051"
+		(property "Reference" "#PWR053"
 			(at 168.91 127 0)
 			(effects
@@
 			(project "mackerel-30-proto"
 				(path "/9307474f-ec99-494d-b4c9-fbd0b10ce86a/89853077-d9a7-463a-b48b-4d81b0ac6897"
-					(reference "#PWR051")
+					(reference "#PWR053")
 					(unit 1)
 				)
@@
 		(dnp no)
 		(fields_autoplaced yes)
-		(property "Reference" "#PWR056"
+		(property "Reference" "#PWR058"
 			(at 201.93 134.62 0)
 			(effects
@@
 			(project "mackerel-30-proto"
 				(path "/9307474f-ec99-494d-b4c9-fbd0b10ce86a/89853077-d9a7-463a-b48b-4d81b0ac6897"
-					(reference "#PWR056")
+					(reference "#PWR058")
 					(unit 1)
 				)
@@
 		(on_board yes)
 		(dnp no)
-		(property "Reference" "C27"
+		(property "Reference" "C28"
 			(at 212.09 40.894 0)
 			(effects
@@
 			(project "mackerel-30-proto"
 				(path "/9307474f-ec99-494d-b4c9-fbd0b10ce86a/89853077-d9a7-463a-b48b-4d81b0ac6897"
-					(reference "C27")
+					(reference "C28")
 					(unit 1)
 				)
@@
 			)
 		)
-		(property "Footprint" "Package_TO_SOT_THT:TO-92"
+		(property "Footprint" "Package_TO_SOT_THT:TO-92L_Inline"
 			(at 201.93 39.37 0)
 			(effects
@@
 		(on_board yes)
 		(dnp no)
-		(property "Reference" "C25"
+		(property "Reference" "C26"
 			(at 98.552 52.07 0)
 			(effects
@@
 			(project "mackerel-30-proto"
 				(path "/9307474f-ec99-494d-b4c9-fbd0b10ce86a/89853077-d9a7-463a-b48b-4d81b0ac6897"
-					(reference "C25")
+					(reference "C26")
 					(unit 1)
 				)
@@
 		(dnp no)
 		(fields_autoplaced yes)
-		(property "Reference" "#PWR059"
+		(property "Reference" "#PWR061"
 			(at 226.06 25.4 0)
 			(effects
@@
 			(project "mackerel-30-proto"
 				(path "/9307474f-ec99-494d-b4c9-fbd0b10ce86a/89853077-d9a7-463a-b48b-4d81b0ac6897"
-					(reference "#PWR059")
+					(reference "#PWR061")
 					(unit 1)
 				)
@@
 		(dnp no)
 		(fields_autoplaced yes)
-		(property "Reference" "#PWR049"
+		(property "Reference" "#PWR051"
 			(at 97.79 166.37 0)
 			(effects
@@
 			(project "mackerel-30-proto"
 				(path "/9307474f-ec99-494d-b4c9-fbd0b10ce86a/89853077-d9a7-463a-b48b-4d81b0ac6897"
-					(reference "#PWR049")
+					(reference "#PWR051")
 					(unit 1)
 				)
@@
 		(dnp no)
 		(fields_autoplaced yes)
-		(property "Reference" "#PWR053"
+		(property "Reference" "#PWR055"
 			(at 189.23 127 0)
 			(effects
@@
 			(project "mackerel-30-proto"
 				(path "/9307474f-ec99-494d-b4c9-fbd0b10ce86a/89853077-d9a7-463a-b48b-4d81b0ac6897"
-					(reference "#PWR053")
+					(reference "#PWR055")
 					(unit 1)
 				)
@@
 		(dnp no)
 		(fields_autoplaced yes)
-		(property "Reference" "#PWR046"
+		(property "Reference" "#PWR048"
 			(at 77.47 64.77 0)
 			(effects
@@
 			(project "mackerel-30-proto"
 				(path "/9307474f-ec99-494d-b4c9-fbd0b10ce86a/89853077-d9a7-463a-b48b-4d81b0ac6897"
-					(reference "#PWR046")
+					(reference "#PWR048")
 					(unit 1)
 				)
@@
 		(on_board yes)
 		(dnp no)
-		(property "Reference" "#PWR047"
+		(property "Reference" "#PWR049"
 			(at 90.17 152.4 0)
 			(effects
@@
 			(project "mackerel-30-proto"
 				(path "/9307474f-ec99-494d-b4c9-fbd0b10ce86a/89853077-d9a7-463a-b48b-4d81b0ac6897"
-					(reference "#PWR047")
+					(reference "#PWR049")
 					(unit 1)
 				)
@@
 		(dnp no)
 		(fields_autoplaced yes)
-		(property "Reference" "#PWR052"
+		(property "Reference" "#PWR054"
 			(at 181.61 134.62 0)
 			(effects
@@
 			(project "mackerel-30-proto"
 				(path "/9307474f-ec99-494d-b4c9-fbd0b10ce86a/89853077-d9a7-463a-b48b-4d81b0ac6897"
-					(reference "#PWR052")
+					(reference "#PWR054")
 					(unit 1)
 				)
@@
 		(dnp no)
 		(fields_autoplaced yes)
-		(property "Reference" "#PWR058"
+		(property "Reference" "#PWR060"
 			(at 222.25 134.62 0)
 			(effects
@@
 			(project "mackerel-30-proto"
 				(path "/9307474f-ec99-494d-b4c9-fbd0b10ce86a/89853077-d9a7-463a-b48b-4d81b0ac6897"
-					(reference "#PWR058")
+					(reference "#PWR060")
 					(unit 1)
 				)
@@
 		(dnp no)
 		(fields_autoplaced yes)
-		(property "Reference" "#PWR044"
+		(property "Reference" "#PWR046"
 			(at 57.15 106.68 0)
 			(effects
@@
 			(project "mackerel-30-proto"
 				(path "/9307474f-ec99-494d-b4c9-fbd0b10ce86a/89853077-d9a7-463a-b48b-4d81b0ac6897"
-					(reference "#PWR044")
+					(reference "#PWR046")
 					(unit 1)
 				)
@@
 		(dnp no)
 		(fields_autoplaced yes)
-		(property "Reference" "#PWR054"
+		(property "Reference" "#PWR056"
 			(at 201.93 34.29 0)
 			(effects
@@
 			(project ""
 				(path "/9307474f-ec99-494d-b4c9-fbd0b10ce86a/89853077-d9a7-463a-b48b-4d81b0ac6897"
-					(reference "#PWR054")
+					(reference "#PWR056")
 					(unit 1)
 				)
@@
 		(on_board yes)
 		(dnp no)
-		(property "Reference" "C24"
+		(property "Reference" "C25"
 			(at 86.36 150.4949 0)
 			(effects
@@
 			(project "mackerel-30-proto"
 				(path "/9307474f-ec99-494d-b4c9-fbd0b10ce86a/89853077-d9a7-463a-b48b-4d81b0ac6897"
-					(reference "C24")
+					(reference "C25")
 					(unit 1)
 				)
@@
 		(on_board yes)
 		(dnp no)
-		(property "Reference" "C23"
+		(property "Reference" "C24"
 			(at 51.562 46.99 0)
 			(effects
@@
 			(project "mackerel-30-proto"
 				(path "/9307474f-ec99-494d-b4c9-fbd0b10ce86a/89853077-d9a7-463a-b48b-4d81b0ac6897"
-					(reference "C23")
+					(reference "C24")
 					(unit 1)
 				)
@@
 		(dnp no)
 		(fields_autoplaced yes)
-		(property "Reference" "#PWR057"
+		(property "Reference" "#PWR059"
 			(at 209.55 127 0)
 			(effects
@@
 			(project "mackerel-30-proto"
 				(path "/9307474f-ec99-494d-b4c9-fbd0b10ce86a/89853077-d9a7-463a-b48b-4d81b0ac6897"
-					(reference "#PWR057")
+					(reference "#PWR059")
 					(unit 1)
 				)
@@
 		(dnp no)
 		(fields_autoplaced yes)
-		(property "Reference" "#PWR043"
+		(property "Reference" "#PWR045"
 			(at 50.8 49.53 0)
 			(effects
@@
 			(project "mackerel-30-proto"
 				(path "/9307474f-ec99-494d-b4c9-fbd0b10ce86a/89853077-d9a7-463a-b48b-4d81b0ac6897"
-					(reference "#PWR043")
+					(reference "#PWR045")
 					(unit 1)
 				)
@@
 		(dnp no)
 		(fields_autoplaced yes)
-		(property "Reference" "#PWR055"
+		(property "Reference" "#PWR057"
 			(at 201.93 60.96 0)
 			(effects
@@
 			(project ""
 				(path "/9307474f-ec99-494d-b4c9-fbd0b10ce86a/89853077-d9a7-463a-b48b-4d81b0ac6897"
-					(reference "#PWR055")
-					(unit 1)
-				)
+					(reference "#PWR057")
+					(unit 1)
+				)

Commit message: PCB cleanup
Other:
- title: Mackerel-30 Proto -> Mackerel-30
Changed lines of the file:
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@@
 	(paper "A")
 	(title_block
-		(title "Mackerel-30 Proto")
-		(date "2024-10-05")
-		(rev "1.0")
+		(title "Mackerel-30")
+		(date "2024-11-09")
+		(rev "0.1")
 		(company "Colin Maykish")
 	)
