File: hardware/mackerel-30-proto/uart.kicad_sch (KiCad schematic)
At the start: 9 parts, among them J4 Conn_01x06, J5 Conn_01x06, J6 Conn_02x10_Odd_Even, U5 XR68C681, X2 3.6864MHz

Commit message: Mackerel-30 v0.1 PCB release
Parts:
- R15, R16: value R -> 4k7
Changed lines of the file:
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@@
 			)
 		)
-		(property "Value" "R"
+		(property "Value" "4k7"
 			(at 104.14 107.95 0)
 			(effects
@@
 			)
 		)
-		(property "Value" "R"
+		(property "Value" "4k7"
 			(at 165.1 118.11 0)
 			(effects
