File: hardware/mackerel-30-v1/duart.kicad_sch (KiCad schematic)
At the start: 6 parts, among them J4 Conn_01x06, J5 Conn_01x06, J6 Conn_02x10_Odd_Even, U12 XR68C681

Commit message: SIMM and data buffers mostly routed
Parts:
- removed C41: 1u, Capacitor_SMD:C_0805_2012Metric_Pad1.18x1.45mm_HandSolder, symbol Device:C_US
- removed J4, J5: Conn_01x06, Connector_PinHeader_2.54mm:PinHeader_1x06_P2.54mm_Vertical, symbol Connector_Generic:Conn_01x06
- removed J6: Conn_02x10_Odd_Even, Connector_PinHeader_2.54mm:PinHeader_2x10_P2.54mm_Vertical, symbol Connector_Generic:Conn_02x10_Odd_Even
- removed R25: 4k7, Resistor_THT:R_Axial_DIN0207_L6.3mm_D2.5mm_P7.62mm_Horizontal, symbol Device:R
- removed U12: XR68C681, Package_LCC:PLCC-44_THT-Socket, symbol mackerel-68k-symbols:XR68C681
Connections:
- no-connect marks 5 -> 0
