File: hardware/mackerel-30-v1/ide.kicad_sch (KiCad schematic)
At the start: 0 parts

Commit message: SIMM and data buffers mostly routed
Parts:
- added C64, C65: 0.1uF, Capacitor_SMD:C_1206_3216Metric_Pad1.33x1.80mm_HandSolder, symbol Device:C_US
- added C66: 470uF, Capacitor_THT:CP_Radial_D8.0mm_P3.50mm, symbol Device:C_Polarized_US
- added D4: LED, LED_THT:LED_D5.0mm, symbol Device:LED
- added J11: Conn_02x20_Odd_Even, Connector_IDC:IDC-Header_2x20_P2.54mm_Vertical, symbol Connector_Generic:Conn_02x20_Odd_Even
- added R20, R21: 4k7, Resistor_SMD:R_1206_3216Metric_Pad1.30x1.75mm_HandSolder, symbol Device:R
- added R22: 1k, Resistor_SMD:R_1206_3216Metric_Pad1.30x1.75mm_HandSolder, symbol Device:R
- added U18, U19: 74HC245, Package_DIP:DIP-20_W7.62mm_Socket, symbol 74xx:74HC245
Connections:
- new net: D4.2 (A), R22.2
- new net +5V: C64.1, C65.1, C66.1, R22.1, U18.20 (VCC), U19.20 (VCC)
- new net A1: J11.35 (Pin_35)
- new net A2: J11.33 (Pin_33)
- new net A3: J11.36 (Pin_36)
- new net D16: U19.11 (B7)
- new net D17: U19.12 (B6)
- new net D18: U19.13 (B5)
- new net D19: U19.14 (B4)
- new net D20: U19.15 (B3)
- new net D21: U19.16 (B2)
- new net D22: U19.17 (B1)
- new net D23: U19.18 (B0)
- new net D24: U18.11 (B7)
- new net D25: U18.12 (B6)
- new net D26: U18.13 (B5)
- new net D27: U18.14 (B4)
- new net D28: U18.15 (B3)
- new net D29: U18.16 (B2)
- new net D30: U18.17 (B1)
- new net D31: U18.18 (B0)
- new net GND: C64.2, C65.2, C66.2, J11.19 (Pin_19), J11.2 (Pin_2), J11.22 (Pin_22), J11.24 (Pin_24), J11.26 (Pin_26), J11.30 (Pin_30), J11.40 (Pin_40), R20.1, R21.1, U18.10 (GND), U19.10 (GND)
- new net IDE_D0: J11.17 (Pin_17), U18.9 (A7)
- new net IDE_D1: J11.15 (Pin_15), U18.8 (A6)
- new net IDE_D10: J11.8 (Pin_8), U19.7 (A5)
- new net IDE_D11: J11.10 (Pin_10), U19.6 (A4)
- new net IDE_D12: J11.12 (Pin_12), U19.5 (A3)
- new net IDE_D13: J11.14 (Pin_14), U19.4 (A2)
- new net IDE_D14: J11.16 (Pin_16), U19.3 (A1)
- new net IDE_D15: J11.18 (Pin_18), U19.2 (A0)
- new net IDE_D2: J11.13 (Pin_13), U18.7 (A5)
- new net IDE_D3: J11.11 (Pin_11), U18.6 (A4)
- new net IDE_D4: J11.9 (Pin_9), U18.5 (A3)
- new net IDE_D5: J11.7 (Pin_7), U18.4 (A2)
- new net IDE_D6: J11.5 (Pin_5), U18.3 (A1)
- new net IDE_D7: J11.3 (Pin_3), U18.2 (A0)
- new net IDE_D8: J11.4 (Pin_4), U19.9 (A7)
- new net IDE_D9: J11.6 (Pin_6), U19.8 (A6)
- new net IDE_INT: J11.31 (Pin_31), R21.2
- new net IDE_RDY: J11.27 (Pin_27), R20.2
- new net R/W: U18.1 (A->B), U19.1 (A->B)
- new net /IDE_BUF: U18.19 (CE), U19.19 (CE)
- new net /IDE_CS0: J11.37 (Pin_37)
- new net /IDE_CS1: J11.38 (Pin_38)
- new net /IDE_RD: J11.25 (Pin_25)
- new net /IDE_WR: J11.23 (Pin_23)
- new net /RESET: J11.1 (Pin_1)
- no-connect marks 0 -> 6
Other:
- note added: "Activity LED"
- note added: "Basically DTACK, active HIGH"
- note added: "IDE Header"
- note added: "IRQ, active HIGH"
- note added: "NOTE: High and low bytes swapped between the CPU and the IDE header"
- note added: "TODO: Molex connector"
- note added: "TODO: review this activity LED"
