File: hardware/mackerel-30-v1/rom_sram.kicad_sch (KiCad schematic)
At the start: 6 parts, among them U10 AS6C4008-55PCN, U9 SST39SF040

Commit message: SIMM and data buffers mostly routed
Parts:
- removed U10: AS6C4008-55PCN, Package_DIP:DIP-32_W15.24mm_Socket, symbol Memory_RAM:AS6C4008-55PCN
- added C43, C44, C45, C46, C47, C48, C49, C50, C51, C52, C53, C67: 0.1uF, Capacitor_SMD:C_1206_3216Metric_Pad1.33x1.80mm_HandSolder, symbol Device:C_US
- added J10, J9: Conn_01x06, Connector_PinHeader_2.54mm:PinHeader_1x06_P2.54mm_Vertical, symbol Connector_Generic:Conn_01x06
- added J6: DE9_Socket_MountingHoles, Connector_Dsub:DSUB-9_Socket_Horizontal_P2.77x2.84mm_EdgePinOffset7.70mm_Housed_MountingHolesOffset9.12mm, symbol Connector:DE9_Socket_MountingHoles
- added J7: DE9_Pins_MountingHoles, Connector_Dsub:DSUB-9_Pins_Horizontal_P2.77x2.84mm_EdgePinOffset7.70mm_Housed_MountingHolesOffset9.12mm, symbol Connector:DE9_Pins_MountingHoles
- added J8: Conn_02x10_Odd_Even, Connector_PinHeader_2.54mm:PinHeader_2x10_P2.54mm_Vertical, symbol Connector_Generic:Conn_02x10_Odd_Even
- added R15: 4k7, Resistor_SMD:R_1206_3216Metric_Pad1.30x1.75mm_HandSolder, symbol Device:R
- added U11, U12: MAX232, Package_DIP:DIP-16_W7.62mm_Socket, symbol Interface_UART:MAX232
- added U13: XR68C681, Package_LCC:PLCC-44_THT-Socket, symbol mackerel-68k-symbols:XR68C681
- added U15: 74ABT245, Package_DIP:DIP-20_W7.62mm_Socket_LongPads, symbol 74xx:74HC245
- added U16: AS6C4008-55PCN, Package_DIP:DIP-32_W15.24mm_Socket, symbol Memory_RAM:AS6C4008-55PCN
- added X3: 3.6864MHz, Oscillator:Oscillator_DIP-8, symbol Oscillator:CXO_DIP8
- C54: renamed from C31; value 1u -> 0.1uF; footprint Capacitor_SMD:C_0805_2012Metric_Pad1.18x1.45mm_HandSolder -> Capacitor_SMD:C_1206_3216Metric_Pad1.33x1.80mm_HandSolder
- C55: renamed from C32; value 1u -> 0.1uF; footprint Capacitor_SMD:C_0805_2012Metric_Pad1.18x1.45mm_HandSolder -> Capacitor_SMD:C_1206_3216Metric_Pad1.33x1.80mm_HandSolder
- R16: renamed from R20; footprint Resistor_THT:R_Axial_DIN0207_L6.3mm_D2.5mm_P7.62mm_Horizontal -> Resistor_SMD:R_1206_3216Metric_Pad1.30x1.75mm_HandSolder
- R17: renamed from R21; footprint Resistor_THT:R_Axial_DIN0207_L6.3mm_D2.5mm_P7.62mm_Horizontal -> Resistor_SMD:R_1206_3216Metric_Pad1.30x1.75mm_HandSolder
- renumbered U9 to U14
Connections:
- net +5V: now also C43.1, C44.1, C53.1, C67.1, J8.3 (Pin_3), J8.4 (Pin_4), R15.2, U11.16 (VCC), U12.16 (VCC), U13.44 (VCC), U15.20 (VCC), U16.32 (VCC), X3.8 (Vcc)
- net A0: now also U16.12 (A0)
- net A1: now also U13.2 (A1), U16.11 (A1)
- net A10: now also U16.23 (A10)
- net A11: now also U16.25 (A11)
- net A12: now also U16.4 (A12)
- net A13: now also U16.28 (A13)
- net A14: now also U16.3 (A14)
- net A15: now also U16.31 (A15)
- net A16: now also U16.2 (A16)
- net A17: now also U16.30 (A17)
- net A18: now also U16.1 (A18)
- net A2: now also U13.4 (A2), U16.10 (A2)
- net A3: now also U13.6 (A3), U16.9 (A3)
- net A4: now also U13.7 (A4), U16.8 (A4)
- net A5: now also U16.7 (A5)
- net A6: now also U16.6 (A6)
- net A7: now also U16.5 (A7)
- net A8: now also U16.27 (A8)
- net A9: now also U16.26 (A9)
- net D24: now also U15.11 (B7); no longer U14.13 (D0)
- net D25: now also U15.12 (B6); no longer U14.14 (D1)
- net D26: now also U15.13 (B5); no longer U14.15 (D2)
- net D27: now also U15.14 (B4); no longer U14.17 (D3)
- net D28: now also U15.15 (B3); no longer U14.18 (D4)
- net D29: now also U15.16 (B2); no longer U14.19 (D5)
- net D30: now also U15.17 (B1); no longer U14.20 (D6)
- net D31: now also U15.18 (B0); no longer U14.21 (D7)
- net GND: now also C43.2, C44.2, C49.2, C50.1, C51.2, C52.1, C53.2, C67.2, J10.1 (Pin_1), J6.5, J6.SH (PAD), J7.5, J7.SH (PAD), J8.19 (Pin_19), J8.20 (Pin_20), J8.5 (Pin_5), J8.6 (Pin_6), J9.1 (Pin_1), U11.15 (GND), U12.15 (GND), U13.22 (GND), U15.10 (GND), U16.16 (VSS), U16.24 (OE#), X3.4 (GND)
- net R/W: now also U13.9 (/RW), U15.1 (A->B), U16.29 (WE#)
- net /CS_SRAM: now also U16.22 (CE#)
- new net: C51.1, U12.2 (VS+)
- new net: C52.2, U12.6 (VS-)
- new net: C49.1, U11.2 (VS+)
- new net: C47.1, U11.4 (C2+)
- new net: C47.2, U11.5 (C2-)
- new net: C50.2, U11.6 (VS-)
- new net: J6.1, J6.4, J6.6
- new net: J6.2, U12.14 (T1OUT)
- new net: J6.3, U12.13 (R1IN)
- new net: J6.7, U12.8 (R2IN)
- new net: J6.8, U12.7 (T2OUT)
- new net: C45.1, U11.1 (C1+)
- new net: C45.2, U11.3 (C1-)
- new net: J7.2, U11.13 (R1IN)
- new net: J7.3, U11.14 (T1OUT)
- new net: J7.7, U11.7 (T2OUT)
- new net: J7.8, U11.8 (R2IN)
- new net: C46.1, U12.1 (C1+)
- new net: C46.2, U12.3 (C1-)
- new net: C48.1, U12.4 (C2+)
- new net: C48.2, U12.5 (C2-)
- new net: J7.1, J7.4, J7.6
- new net BUF_D24: U13.28 (D0), U14.13 (D0), U15.9 (A7), U16.13 (DQ0)
- new net BUF_D25: U13.18 (D1), U14.14 (D1), U15.8 (A6), U16.14 (DQ1)
- new net BUF_D26: U13.27 (D2), U14.15 (D2), U15.7 (A5), U16.15 (DQ2)
- new net BUF_D27: U13.19 (D3), U14.17 (D3), U15.6 (A4), U16.17 (DQ3)
- new net BUF_D28: U13.26 (D4), U14.18 (D4), U15.5 (A3), U16.18 (DQ4)
- new net BUF_D29: U13.20 (D5), U14.19 (D5), U15.4 (A2), U16.19 (DQ5)
- new net BUF_D30: U13.25 (D6), U14.20 (D6), U15.3 (A1), U16.20 (DQ6)
- new net BUF_D31: U13.21 (D7), U14.21 (D7), U15.2 (A0), U16.21 (DQ7)
- new net CLK_DUART: U13.36 (X1/CLK), X3.5 (OUT)
- new net IP2: J8.11 (Pin_11), U13.40 (IP2)
- new net IP3: J8.13 (Pin_13), U13.3 (IP3)
- new net IP4: J8.15 (Pin_15), U13.43 (IP4)
- new net IP5: J8.17 (Pin_17), U13.42 (IP5)
- new net OP2: J8.8 (Pin_8), U13.31 (OP2)
- new net OP3: J8.10 (Pin_10), U13.15 (OP3)
- new net OP4: J8.12 (Pin_12), U13.30 (OP4)
- new net OP5: J8.14 (Pin_14), U13.16 (OP5)
- new net OP6: J8.16 (Pin_16), U13.29 (OP6)
- new net OP7: J8.18 (Pin_18), U13.17 (OP7)
- new net RXA: J9.4 (Pin_4), U11.12 (R1OUT), U13.35 (RXDA)
- new net RXB: J10.4 (Pin_4), U12.12 (R1OUT), U13.11 (RXDB)
- new net TXA: J9.5 (Pin_5), U11.11 (T1IN), U13.33 (TXDA)
- new net TXB: J10.5 (Pin_5), U12.11 (T1IN), U13.13 (TXDB)
- new net /CS_DUART: U13.39 (CS)
- new net /CTSA: U11.9 (R2OUT), U13.8 (IP0)
- new net /CTSB: U12.9 (R2OUT), U13.5 (IP1)
- new net /DSACK0: U13.10 (/DTACK)
- new net /IACK_DUART: U13.41 (/IACK)
- new net /IRQ_DUART: R15.1, U13.24 (INTR)
- new net /RESET: U13.38 (/RESET)
- new net /RTSA: J9.2 (Pin_2), U11.10 (T2IN), U13.32 (OP0)
- new net /RTSB: J10.2 (Pin_2), U12.10 (T2IN), U13.14 (OP1)
- no-connect marks 0 -> 8
Other:
- note added: "Channel A (Peripheral)"
- note added: "Channel B (Console)"
- moved on the sheet: C54, C55, R16, R17, U14
