File: hardware/mackerel-30-v1/mackerel-30-v1.kicad_pcb (KiCad board)
At the start: 2 copper layers, 26 parts, among them J1 Conn_01x03, J2 Conn_01x07, SW1 SW_Push, U1 ATtiny1614-SS, U2 MCP1700x-330xxTO, U3 74AHCT125, U4 74LVC07A, Y1 Si5351A-B-GT, Y2 Crystal_GND24

Commit message: Mackerel-30: Label the 68030 pinout
Parts:
- added C10: 1u, Capacitor_SMD:C_0805_2012Metric_Pad1.18x1.45mm_HandSolder, F.Cu at (29.3, 74.4)
- added C11: 1u, Capacitor_SMD:C_0805_2012Metric_Pad1.18x1.45mm_HandSolder, F.Cu at (29.3, 77.5)
- added C12: 1u, Capacitor_SMD:C_0805_2012Metric_Pad1.18x1.45mm_HandSolder, F.Cu at (29.3, 80.5)
- added C13: 1u, Capacitor_SMD:C_0805_2012Metric_Pad1.18x1.45mm_HandSolder, F.Cu at (34.1, 68.4)
- added C14: 1u, Capacitor_SMD:C_0805_2012Metric_Pad1.18x1.45mm_HandSolder, F.Cu at (34.1, 71.4)
- added C15: 1u, Capacitor_SMD:C_0805_2012Metric_Pad1.18x1.45mm_HandSolder, F.Cu at (34.1, 74.4)
- added C16: 1u, Capacitor_SMD:C_0805_2012Metric_Pad1.18x1.45mm_HandSolder, F.Cu at (34.1, 77.5)
- added C17: 1u, Capacitor_SMD:C_0805_2012Metric_Pad1.18x1.45mm_HandSolder, F.Cu at (34.1, 80.5)
- added C18: 1u, Capacitor_SMD:C_0805_2012Metric_Pad1.18x1.45mm_HandSolder, F.Cu at (126.0, 117.5)
- added C19: 1u, Capacitor_SMD:C_0805_2012Metric_Pad1.18x1.45mm_HandSolder, F.Cu at (126.0, 120.5)
- added C20: 1u, Capacitor_SMD:C_0805_2012Metric_Pad1.18x1.45mm_HandSolder, F.Cu at (126.0, 123.5)
- added C21: 1u, Capacitor_SMD:C_0805_2012Metric_Pad1.18x1.45mm_HandSolder, F.Cu at (126.0, 126.5)
- added C22: 1u, Capacitor_SMD:C_0805_2012Metric_Pad1.18x1.45mm_HandSolder, F.Cu at (126.0, 129.5)
- added C23: 1u, Capacitor_SMD:C_0805_2012Metric_Pad1.18x1.45mm_HandSolder, F.Cu at (126.0, 132.6)
- added C24: 1u, Capacitor_SMD:C_0805_2012Metric_Pad1.18x1.45mm_HandSolder, F.Cu at (126.0, 135.6)
- added C25: 1u, Capacitor_SMD:C_0805_2012Metric_Pad1.18x1.45mm_HandSolder, F.Cu at (126.0, 138.6)
- added C26: 470u, Capacitor_THT:CP_Radial_D8.0mm_P3.50mm, F.Cu at (44.0, 72.5)
- added C8: 1u, Capacitor_SMD:C_0805_2012Metric_Pad1.18x1.45mm_HandSolder, F.Cu at (29.3, 68.4)
- added C9: 1u, Capacitor_SMD:C_0805_2012Metric_Pad1.18x1.45mm_HandSolder, F.Cu at (29.3, 71.4)
- added J3: Conn_02x05_Odd_Even, Connector_IDC:IDC-Header_2x05_P2.54mm_Vertical, F.Cu at (133.6, 122.1)
- added R10: 4k7, Resistor_SMD:R_0805_2012Metric_Pad1.20x1.40mm_HandSolder, F.Cu at (146.0, 123.0)
- added R11: 4k7, Resistor_SMD:R_0805_2012Metric_Pad1.20x1.40mm_HandSolder, F.Cu at (146.0, 126.0)
- added R12: 4k7, Resistor_SMD:R_0805_2012Metric_Pad1.20x1.40mm_HandSolder, F.Cu at (146.0, 128.9)
- added R13: 4k7, Resistor_SMD:R_0805_2012Metric_Pad1.20x1.40mm_HandSolder, F.Cu at (146.0, 131.8)
- added U5: MC68030RC, mackerel:PGA169, F.Cu at (26.0, 29.5)
- added U6: EPM7128, Package_LCC:PLCC-84_THT-Socket, F.Cu at (104.5, 119.8)
- moved D1 81.9 mm to (259.5, 84.5)
- moved U1 81.9 mm to (260.5, 75.0)
- moved U2 81.9 mm to (188.0, 33.0)
- moved C3 81.9 mm to (226.0, 22.5)
- moved C4 81.9 mm to (193.5, 40.5)
- moved C5 81.9 mm to (187.5, 40.0)
- moved C7 81.9 mm to (249.5, 19.5)
- moved J1 81.9 mm to (244.5, 73.5)
- moved J2 81.9 mm to (272.0, 67.5)
- moved R1 81.9 mm to (245.5, 83.0)
- moved R2 81.9 mm to (218.5, 27.0)
- moved R3 81.9 mm to (218.5, 29.9)
- moved R4 81.9 mm to (218.5, 32.9)
- moved R5 81.9 mm to (251.0, 51.5)
- moved R6 81.9 mm to (251.0, 72.5)
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
Commit message: Mackerel-30: Add low mem, FPU, DRAM, DUART, IDE, power sheets to schematic
Parts:
- removed C4, C5: 1u, Capacitor_SMD:C_0805_2012Metric_Pad1.18x1.45mm_HandSolder
- removed U2: MCP1700x-330xxTO, Package_TO_SOT_THT:TO-92_Inline
- added C27: 10uF, Capacitor_THT:CP_Radial_D5.0mm_P2.00mm, F.Cu at (-43.0, -14.0)
- added C28: 10uF, Capacitor_THT:CP_Radial_D5.0mm_P2.00mm, F.Cu at (-44.0, -4.00)
- added C29: 1000uF, Capacitor_THT:CP_Radial_D10.0mm_P5.00mm, F.Cu at (-72.5, -10.0)
- added C30: 1000uF, Capacitor_THT:CP_Radial_D10.0mm_P5.00mm, F.Cu at (-79.5, 5.00)
- added C31: 1u, Capacitor_SMD:C_0805_2012Metric_Pad1.18x1.45mm_HandSolder, F.Cu at (-120.0, 100.0)
- added C32: 1u, Capacitor_SMD:C_0805_2012Metric_Pad1.18x1.45mm_HandSolder, F.Cu at (-120.0, 103.0)
- added C33: 1u, Capacitor_SMD:C_0805_2012Metric_Pad1.18x1.45mm_HandSolder, F.Cu at (-30.0, 130.2)
- added C34: 1u, Capacitor_SMD:C_0805_2012Metric_Pad1.18x1.45mm_HandSolder, F.Cu at (-30.0, 133.2)
- added C35: 1u, Capacitor_SMD:C_0805_2012Metric_Pad1.18x1.45mm_HandSolder, F.Cu at (-30.0, 136.2)
- added C36: 1u, Capacitor_SMD:C_0805_2012Metric_Pad1.18x1.45mm_HandSolder, F.Cu at (-30.0, 139.2)
- added C37: 1u, Capacitor_SMD:C_0805_2012Metric_Pad1.18x1.45mm_HandSolder, F.Cu at (-30.0, 142.2)
- added C38: 1u, Capacitor_SMD:C_0805_2012Metric_Pad1.18x1.45mm_HandSolder, F.Cu at (-30.0, 145.2)
- added C39: 1u, Capacitor_SMD:C_0805_2012Metric_Pad1.18x1.45mm_HandSolder, F.Cu at (-30.0, 148.2)
- added C40: 1u, Capacitor_SMD:C_0805_2012Metric_Pad1.18x1.45mm_HandSolder, F.Cu at (-30.0, 151.2)
- added C41: 1u, Capacitor_SMD:C_0805_2012Metric_Pad1.18x1.45mm_HandSolder, F.Cu at (128.5, -13.4)
- added D2: 1N5822, Diode_THT:D_DO-27_P15.24mm_Horizontal, F.Cu at (-113.1, 21.0)
- added D3: LED, LED_THT:LED_D5.0mm, F.Cu at (-20.0, 16.0)
- added D4: LED, LED_THT:LED_D5.0mm, F.Cu at (-3.02, 63.6)
- added H1: MountingHole_Pad, MountingHole:MountingHole_3.2mm_M3_Pad_Via, F.Cu at (-1.80, -10.3)
- added H2: MountingHole_Pad, MountingHole:MountingHole_3.2mm_M3_Pad_Via, F.Cu at (292.8, -12.8)
- added H3: MountingHole_Pad, MountingHole:MountingHole_3.2mm_M3_Pad_Via, F.Cu at (-11.0, 213.9)
- added H4: MountingHole_Pad, MountingHole:MountingHole_3.2mm_M3_Pad_Via, F.Cu at (303.7, 230.2)
- added HS1: Heatsink, Heatsink:Heatsink_Stonecold_HS-S02_13.21x9.53mm, F.Cu at (-114.5, -7.50)
- added J10: Conn_02x03_Odd_Even, Connector_PinHeader_2.54mm:PinHeader_2x03_P2.54mm_Vertical, F.Cu at (-47.0, 14.9)
- added J4: Conn_01x06, Connector_PinHeader_2.54mm:PinHeader_1x06_P2.54mm_Vertical, F.Cu at (143.2, -38.2)
- added J5: Conn_01x06, Connector_PinHeader_2.54mm:PinHeader_1x06_P2.54mm_Vertical, F.Cu at (147.8, -38.2)
- added J6: Conn_02x10_Odd_Even, Connector_PinHeader_2.54mm:PinHeader_2x10_P2.54mm_Vertical, F.Cu at (110.5, -38.2)
- added J7: Barrel_Jack_MountingPin, Connector_BarrelJack:BarrelJack_Horizontal, F.Cu at (-83.5, -8.00)
- added J8: Conn_02x03_Odd_Even, Connector_PinHeader_2.54mm:PinHeader_2x03_P2.54mm_Vertical, F.Cu at (-61.3, 14.9)
- added J9: Conn_02x03_Odd_Even, Connector_PinHeader_2.54mm:PinHeader_2x03_P2.54mm_Vertical, F.Cu at (-54.2, 14.9)
- added L1: 100uH, Inductor_THT:L_Radial_D10.0mm_P5.00mm_Fastron_07M, F.Cu at (-95.5, 8.00)
- added R14: 4k7, Resistor_SMD:R_0805_2012Metric_Pad1.20x1.40mm_HandSolder, F.Cu at (67.5, 50.1)
- added R15: 4k7, Resistor_SMD:R_0805_2012Metric_Pad1.20x1.40mm_HandSolder, F.Cu at (67.5, 53.1)
- added R16: 4k7, Resistor_SMD:R_0805_2012Metric_Pad1.20x1.40mm_HandSolder, F.Cu at (67.5, 56.0)
- added R17: 4k7, Resistor_SMD:R_0805_2012Metric_Pad1.20x1.40mm_HandSolder, F.Cu at (67.5, 59.0)
- added R18: 1k, Resistor_THT:R_Axial_DIN0207_L6.3mm_D2.5mm_P7.62mm_Horizontal, F.Cu at (-22.1, 24.5)
- added R19: 1k, Resistor_THT:R_Axial_DIN0207_L6.3mm_D2.5mm_P7.62mm_Horizontal, F.Cu at (-3.92, 57.8)
- added R20: 4k7, Resistor_THT:R_Axial_DIN0207_L6.3mm_D2.5mm_P7.62mm_Horizontal, F.Cu at (-128.6, 45.0)
- added R21: 4k7, Resistor_THT:R_Axial_DIN0207_L6.3mm_D2.5mm_P7.62mm_Horizontal, F.Cu at (-24.1, 130.7)
- added R22: 4k7, Resistor_THT:R_Axial_DIN0207_L6.3mm_D2.5mm_P7.62mm_Horizontal, F.Cu at (116.9, -12.9)
- added R23: 4k7, Resistor_THT:R_Axial_DIN0207_L6.3mm_D2.5mm_P7.62mm_Horizontal, F.Cu at (-63.9, 163.7)
- added R24: 4k7, Resistor_THT:R_Axial_DIN0207_L6.3mm_D2.5mm_P7.62mm_Horizontal, F.Cu at (-63.9, 167.8)
- added R25: 4k7, Resistor_THT:R_Axial_DIN0207_L6.3mm_D2.5mm_P7.62mm_Horizontal, F.Cu at (116.9, -8.84)
- added U10: AS6C4008-55PCN, Package_DIP:DIP-32_W15.24mm_Socket, F.Cu at (-117.0, 54.4)
- added U11: MC68882, Package_LCC:PLCC-68_THT-Socket, F.Cu at (-49.0, 132.5)
- added U12: XR68C681, Package_LCC:PLCC-44_THT-Socket, F.Cu at (129.4, -34.0)
- added U7: AMS1117-3.3, Package_TO_SOT_SMD:SOT-223-3_TabPin2, F.Cu at (-32.5, -11.5)
- added U8: LM2576T-5, Package_TO_SOT_THT:TO-220-5_Vertical, F.Cu at (-116.4, 8.95)
- added U9: SST39SF040, Package_DIP:DIP-32_W15.24mm_Socket, F.Cu at (-136.3, 54.4)
Connections:
- U5 pad C1: unconnected-(U5-FC1-PadC1) -> FC1
- U5 pad D1: unconnected-(U5-FC2-PadD1) -> FC2
- U5 pad D2: unconnected-(U5-FC0-PadD2) -> FC0
- U5 pad E2: unconnected-(U5-/AVEC-PadE2) -> /AVEC
- U5 pad F1: unconnected-(U5-/DSACK0-PadF1) -> /DSACK0
- U5 pad F12: unconnected-(U5-/RESET-PadF12) -> /RESET
- U5 pad F13: unconnected-(U5-/MMUDIS-PadF13) -> Net-(U5-/MMUDIS)
- U5 pad G1: unconnected-(U5-/STERM-PadG1) -> /STERM
- U5 pad G12: unconnected-(U5-/IPL2-PadG12) -> /IPL2
- U5 pad G13: unconnected-(U5-/IPL1-PadG13) -> /IPL1
- U5 pad G2: unconnected-(U5-/DSACK1-PadG2) -> /DSACK1
- U5 pad H1: unconnected-(U5-/BERR-PadH1) -> /BERR
- U5 pad H12: unconnected-(U5-/CDIS-PadH12) -> Net-(U5-/CDIS)
- U5 pad H13: unconnected-(U5-/IPL0-PadH13) -> /IPL0
- U5 pad H2: unconnected-(U5-/HALT-PadH2) -> /HALT
- U5 pad J1: unconnected-(U5-/CBACK-PadJ1) -> /CBACK
- U5 pad J2: unconnected-(U5-/AS-PadJ2) -> /AS
- U5 pad K1: unconnected-(U5-/CBREQ-PadK1) -> /CBREQ
- U5 pad K2: unconnected-(U5-/DS-PadK2) -> /DS
- U5 pad K3: unconnected-(U5-SIZ1-PadK3) -> SIZ1
- U5 pad L1: unconnected-(U5-/CIIN-PadL1) -> /CIIN
- U5 pad L2: unconnected-(U5-SIZ0-PadL2) -> SIZ0
- U5 pad L3: unconnected-(U5-R/W-PadL3) -> R/W

Commit message: SIMM and data buffers mostly routed
Parts:
- removed R23, R24, R25: 4k7, Resistor_THT:R_Axial_DIN0207_L6.3mm_D2.5mm_P7.62mm_Horizontal
- removed Y1: Si5351A-B-GT, Package_SO:MSOP-10_3x3mm_P0.5mm
- removed Y2: Crystal_GND24, Crystal:Crystal_SMD_3225-4Pin_3.2x2.5mm_HandSoldering
- added C4: 0.1uF, Capacitor_SMD:C_1206_3216Metric_Pad1.33x1.80mm_HandSolder, B.Cu at (119.0, 81.7)
- added C42: 0.01uF, Capacitor_SMD:C_1206_3216Metric_Pad1.33x1.80mm_HandSolder, F.Cu at (-48.8, 47.5)
- added C43: 0.1uF, Capacitor_SMD:C_1206_3216Metric_Pad1.33x1.80mm_HandSolder, B.Cu at (183.0, 32.1)
- added C44: 0.1uF, Capacitor_SMD:C_1206_3216Metric_Pad1.33x1.80mm_HandSolder, B.Cu at (199.5, 32.1)
- added C45: 0.1uF, Capacitor_SMD:C_1206_3216Metric_Pad1.33x1.80mm_HandSolder, B.Cu at (180.5, 33.1)
- added C46: 0.1uF, Capacitor_SMD:C_1206_3216Metric_Pad1.33x1.80mm_HandSolder, B.Cu at (197.0, 32.6)
- added C47: 0.1uF, Capacitor_SMD:C_1206_3216Metric_Pad1.33x1.80mm_HandSolder, B.Cu at (180.5, 39.6)
- added C48: 0.1uF, Capacitor_SMD:C_1206_3216Metric_Pad1.33x1.80mm_HandSolder, B.Cu at (197.0, 39.6)
- added C49: 0.1uF, Capacitor_SMD:C_1206_3216Metric_Pad1.33x1.80mm_HandSolder, B.Cu at (175.0, 34.6)
- added C5: 0.1uF, Capacitor_SMD:C_1206_3216Metric_Pad1.33x1.80mm_HandSolder, B.Cu at (120.6, 85.8)
- added C50: 0.1uF, Capacitor_SMD:C_1206_3216Metric_Pad1.33x1.80mm_HandSolder, B.Cu at (175.0, 41.6)
- added C51: 0.1uF, Capacitor_SMD:C_1206_3216Metric_Pad1.33x1.80mm_HandSolder, B.Cu at (191.5, 34.6)
- added C52: 0.1uF, Capacitor_SMD:C_1206_3216Metric_Pad1.33x1.80mm_HandSolder, B.Cu at (191.5, 41.6)
- added C53: 0.1uF, Capacitor_SMD:C_1206_3216Metric_Pad1.33x1.80mm_HandSolder, F.Cu at (-82.6, 125.3)
- added C54: 0.1uF, Capacitor_SMD:C_1206_3216Metric_Pad1.33x1.80mm_HandSolder, F.Cu at (-82.6, 118.6)
- added C55: 0.1uF, Capacitor_SMD:C_1206_3216Metric_Pad1.33x1.80mm_HandSolder, F.Cu at (-82.6, 121.9)
- added C56: 0.1uF, Capacitor_SMD:C_1206_3216Metric_Pad1.33x1.80mm_HandSolder, B.Cu at (129.9, 111.1)
- added C57: 0.1uF, Capacitor_SMD:C_1206_3216Metric_Pad1.33x1.80mm_HandSolder, B.Cu at (120.8, 112.5)
- added C58: 0.1uF, Capacitor_SMD:C_1206_3216Metric_Pad1.33x1.80mm_HandSolder, B.Cu at (115.5, 132.8)
- added C59: 0.1uF, Capacitor_SMD:C_1206_3216Metric_Pad1.33x1.80mm_HandSolder, B.Cu at (127.3, 126.8)
- added C60: 0.1uF, Capacitor_SMD:C_1206_3216Metric_Pad1.33x1.80mm_HandSolder, B.Cu at (135.0, 126.8)
- added C61: 0.1uF, Capacitor_SMD:C_1206_3216Metric_Pad1.33x1.80mm_HandSolder, B.Cu at (127.4, 124.1)
- added C62: 0.1uF, Capacitor_SMD:C_1206_3216Metric_Pad1.33x1.80mm_HandSolder, B.Cu at (136.2, 112.5)
- added C63: 0.1uF, Capacitor_SMD:C_1206_3216Metric_Pad1.33x1.80mm_HandSolder, B.Cu at (137.1, 103.8)
- added C64: 0.1uF, Capacitor_SMD:C_1206_3216Metric_Pad1.33x1.80mm_HandSolder, B.Cu at (85.4, 140.4)
- added C65: 0.1uF, Capacitor_SMD:C_1206_3216Metric_Pad1.33x1.80mm_HandSolder, B.Cu at (115.2, 140.4)
- added C66: 470uF, Capacitor_THT:CP_Radial_D8.0mm_P3.50mm, F.Cu at (65.1, 183.2)
- added C67: 0.1uF, Capacitor_SMD:C_1206_3216Metric_Pad1.33x1.80mm_HandSolder, B.Cu at (85.8, 129.6)
- added J11: Conn_02x20_Odd_Even, Connector_IDC:IDC-Header_2x20_P2.54mm_Vertical, F.Cu at (63.5, 161.0)
- added J12: Conn_02x40_Odd_Even, Connector_PinSocket_2.54mm:PinSocket_2x40_P2.54mm_Vertical, F.Cu at (26.8, 46.4)
- added U13: XR68C681, Package_LCC:PLCC-44_THT-Socket, F.Cu at (81.8, 37.1)
- added U14: SST39SF040, Package_DIP:DIP-32_W15.24mm_Socket, F.Cu at (86.3, 62.9)
- added U15: 74ABT245, Package_DIP:DIP-20_W7.62mm_Socket_LongPads, F.Cu at (84.2, 134.3)
- added U16: AS6C4008-55PCN, Package_DIP:DIP-32_W15.24mm_Socket, F.Cu at (61.8, 62.3)
- added U17: MC68882, Package_LCC:PLCC-68_THT-Socket, F.Cu at (141.3, 118.9)
- added U18: 74HC245, Package_DIP:DIP-20_W7.62mm_Socket, F.Cu at (84.3, 145.5)
- added U19: 74HC245, Package_DIP:DIP-20_W7.62mm_Socket, F.Cu at (114.1, 145.5)
- added U2: EPM7128, Package_LCC:PLCC-84_THT-Socket, F.Cu at (172.6, 62.5)
- added U20: SN74LVC8T245, Package_SO:SOIC-24W_7.5x15.4mm_P1.27mm, F.Cu at (43.9, 58.1)
- added U21: SN74LVC8T245, Package_SO:SOIC-24W_7.5x15.4mm_P1.27mm, F.Cu at (44.0, 71.5)
- added U22: SN74LVC8T245, Package_SO:SOIC-24W_7.5x15.4mm_P1.27mm, F.Cu at (44.2, 84.7)
- added U23: SN74LVC8T245, Package_SO:SOIC-24W_7.5x15.4mm_P1.27mm, F.Cu at (44.3, 98.2)
- added U24: SN74LVC8T245, Package_SO:SOIC-24W_7.5x15.4mm_P1.27mm, F.Cu at (44.4, 113.2)
- added U25: SN74LVC8T245, Package_SO:SOIC-24W_7.5x15.4mm_P1.27mm, F.Cu at (44.3, 127.2)
- added U26: SN74LVC8T245, Package_SO:SOIC-24W_7.5x15.4mm_P1.27mm, F.Cu at (44.4, 142.2)
- added X1: 24 MHz, Oscillator:Oscillator_DIP-14, F.Cu at (126.3, 57.0)
- added X2: 50 MHz, Oscillator:Oscillator_DIP-14, F.Cu at (198.1, 121.1)
- added X3: 3.6864MHz, Oscillator:Oscillator_DIP-8, F.Cu at (98.7, 52.8)
- C1, C2, C3, C6, C7: value 0.1u -> 0.1uF; footprint Capacitor_SMD:C_0805_2012Metric_Pad1.18x1.45mm_HandSolder -> Capacitor_SMD:C_1206_3216Metric_Pad1.33x1.80mm_HandSolder; moved to B.Cu
- C10, C23, C24, C25, C31, C32, C33, C34, C35, C36, C37, C40, C41, C8, C9: value 1u -> 0.1uF; footprint Capacitor_SMD:C_0805_2012Metric_Pad1.18x1.45mm_HandSolder -> Capacitor_SMD:C_1206_3216Metric_Pad1.33x1.80mm_HandSolder; moved to B.Cu
- C11: value 1u -> 470u; footprint Capacitor_SMD:C_0805_2012Metric_Pad1.18x1.45mm_HandSolder -> Capacitor_THT:CP_Radial_D8.0mm_P3.50mm
- C12, C13, C14, C15, C16, C17, C18, C19, C20: value 1u -> 0.1uF; footprint Capacitor_SMD:C_0805_2012Metric_Pad1.18x1.45mm_HandSolder -> Capacitor_SMD:C_1206_3216Metric_Pad1.33x1.80mm_HandSolder
- C21, C22: value 1u -> 470uF; footprint Capacitor_SMD:C_0805_2012Metric_Pad1.18x1.45mm_HandSolder -> Capacitor_THT:CP_Radial_D8.0mm_P3.50mm
- C26: value 470u -> 0.1uF; footprint Capacitor_THT:CP_Radial_D8.0mm_P3.50mm -> Capacitor_SMD:C_1206_3216Metric_Pad1.33x1.80mm_HandSolder; moved to B.Cu
- C27, C28: value 10uF -> 0.1uF; footprint Capacitor_THT:CP_Radial_D5.0mm_P2.00mm -> Capacitor_SMD:C_1206_3216Metric_Pad1.33x1.80mm_HandSolder; moved to B.Cu
- C29, C30: value 1000uF -> 0.1uF; footprint Capacitor_THT:CP_Radial_D10.0mm_P5.00mm -> Capacitor_SMD:C_1206_3216Metric_Pad1.33x1.80mm_HandSolder; moved to B.Cu
- C38, C39: value 1u -> 1000uF; footprint Capacitor_SMD:C_0805_2012Metric_Pad1.18x1.45mm_HandSolder -> Capacitor_THT:CP_Radial_D10.0mm_P5.00mm
- D1: value LED -> 1N5822; footprint LED_SMD:LED_0805_2012Metric_Pad1.15x1.40mm_HandSolder -> Diode_THT:D_DO-27_P15.24mm_Horizontal
- D2: value 1N5822 -> LED; footprint Diode_THT:D_DO-27_P15.24mm_Horizontal -> LED_THT:LED_D5.0mm
- J1: value Conn_01x03 -> Conn_02x05_Odd_Even; footprint Connector_PinHeader_2.54mm:PinHeader_1x03_P2.54mm_Vertical -> Connector_IDC:IDC-Header_2x05_P2.54mm_Vertical
- J10, J9: value Conn_02x03_Odd_Even -> Conn_01x06; footprint Connector_PinHeader_2.54mm:PinHeader_2x03_P2.54mm_Vertical -> Connector_PinHeader_2.54mm:PinHeader_1x06_P2.54mm_Vertical
- J2: value Conn_01x07 -> Conn_02x05_Odd_Even; footprint Connector_PinHeader_2.54mm:PinHeader_1x07_P2.54mm_Vertical -> Connector_IDC:IDC-Header_2x05_P2.54mm_Vertical
- J3: value Conn_02x05_Odd_Even -> Barrel_Jack_MountingPin; footprint Connector_IDC:IDC-Header_2x05_P2.54mm_Vertical -> Connector_BarrelJack:BarrelJack_Horizontal
- J4, J5: value Conn_01x06 -> Conn_02x03_Odd_Even; footprint Connector_PinHeader_2.54mm:PinHeader_1x06_P2.54mm_Vertical -> Connector_PinHeader_2.54mm:PinHeader_2x03_P2.54mm_Vertical
- J6: value Conn_02x10_Odd_Even -> DE9_Socket_MountingHoles; footprint Connector_PinHeader_2.54mm:PinHeader_2x10_P2.54mm_Vertical -> Connector_Dsub:DSUB-9_Socket_Horizontal_P2.77x2.84mm_EdgePinOffset7.70mm_Housed_MountingHolesOffset9.12mm
- J7: value Barrel_Jack_MountingPin -> DE9_Pins_MountingHoles; footprint Connector_BarrelJack:BarrelJack_Horizontal -> Connector_Dsub:DSUB-9_Pins_Horizontal_P2.77x2.84mm_EdgePinOffset7.70mm_Housed_MountingHolesOffset9.12mm
- J8: value Conn_02x03_Odd_Even -> Conn_02x10_Odd_Even; footprint Connector_PinHeader_2.54mm:PinHeader_2x03_P2.54mm_Vertical -> Connector_PinHeader_2.54mm:PinHeader_2x10_P2.54mm_Vertical
- R1, R10, R11, R12, R15, R16, R17, R5, R6, R7, R8: footprint Resistor_SMD:R_0805_2012Metric_Pad1.20x1.40mm_HandSolder -> Resistor_SMD:R_1206_3216Metric_Pad1.30x1.75mm_HandSolder
- R13, R14: value 4k7 -> 1k; footprint Resistor_SMD:R_0805_2012Metric_Pad1.20x1.40mm_HandSolder -> Resistor_SMD:R_1206_3216Metric_Pad1.30x1.75mm_HandSolder
- R18, R19: value 1k -> 4k7; footprint Resistor_THT:R_Axial_DIN0207_L6.3mm_D2.5mm_P7.62mm_Horizontal -> Resistor_SMD:R_1206_3216Metric_Pad1.30x1.75mm_HandSolder
- R2, R3: value 33 -> 10k; footprint Resistor_SMD:R_0805_2012Metric_Pad1.20x1.40mm_HandSolder -> Resistor_SMD:R_1206_3216Metric_Pad1.30x1.75mm_HandSolder
- R20, R21: footprint Resistor_THT:R_Axial_DIN0207_L6.3mm_D2.5mm_P7.62mm_Horizontal -> Resistor_SMD:R_1206_3216Metric_Pad1.30x1.75mm_HandSolder
- R22: value 4k7 -> 1k; footprint Resistor_THT:R_Axial_DIN0207_L6.3mm_D2.5mm_P7.62mm_Horizontal -> Resistor_SMD:R_1206_3216Metric_Pad1.30x1.75mm_HandSolder
- R4: value 33 -> 4k7; footprint Resistor_SMD:R_0805_2012Metric_Pad1.20x1.40mm_HandSolder -> Resistor_SMD:R_1206_3216Metric_Pad1.30x1.75mm_HandSolder
- R9: value 1k -> 4k7; footprint Resistor_SMD:R_0805_2012Metric_Pad1.20x1.40mm_HandSolder -> Resistor_SMD:R_1206_3216Metric_Pad1.30x1.75mm_HandSolder
- U1: value ATtiny1614-SS -> MC68030RC; footprint Package_SO:SOIC-14_3.9x8.7mm_P1.27mm -> mackerel:PGA169
- U10: value AS6C4008-55PCN -> DS1233; footprint Package_DIP:DIP-32_W15.24mm_Socket -> Package_TO_SOT_THT:TO-92L_Wide
- U11: value MC68882 -> MAX232; footprint Package_LCC:PLCC-68_THT-Socket -> Package_DIP:DIP-16_W7.62mm_Socket
- U12: value XR68C681 -> MAX232; footprint Package_LCC:PLCC-44_THT-Socket -> Package_DIP:DIP-16_W7.62mm_Socket
- U3: value 74AHCT125 -> EPM7128; footprint Package_SO:SOIC-14_3.9x8.7mm_P1.27mm -> Package_LCC:PLCC-84_THT-Socket
- U4: value 74LVC07A -> SIMM72; footprint Package_SO:SOIC-14_3.9x8.7mm_P1.27mm -> mackerel:SIMM-72
- U5: value MC68030RC -> 74ABT245; footprint mackerel:PGA169 -> Package_DIP:DIP-20_W7.62mm_Socket_LongPads
- U6: value EPM7128 -> 74ABT245; footprint Package_LCC:PLCC-84_THT-Socket -> Package_DIP:DIP-20_W7.62mm_Socket_LongPads
- U7: value AMS1117-3.3 -> 74ABT245; footprint Package_TO_SOT_SMD:SOT-223-3_TabPin2 -> Package_DIP:DIP-20_W7.62mm_Socket_LongPads
- U8: value LM2576T-5 -> 74ABT245; footprint Package_TO_SOT_THT:TO-220-5_Vertical -> Package_DIP:DIP-20_W7.62mm_Socket_LongPads
- U9: value SST39SF040 -> LM2576T-5; footprint Package_DIP:DIP-32_W15.24mm_Socket -> Package_TO_SOT_THT:TO-220-5_Vertical
- moved R9 349.0 mm to (-94.4, 35.4)
- moved R7 332.6 mm to (-63.5, 153.6)
- moved R8 330.8 mm to (-63.5, 156.9)
- moved R5 328.7 mm to (-63.5, 147.0)
- moved U8 325.6 mm to (173.7, 156.8), turned to 90 degrees
- moved R6 324.0 mm to (-63.5, 150.3)
- moved SW1 321.1 mm to (-54.4, 17.4)
- moved R1 313.1 mm to (-63.5, 133.8)
- moved R4 303.0 mm to (-63.5, 143.7)
- moved R3 302.8 mm to (-63.5, 140.4)
- moved R2 302.7 mm to (-63.5, 137.1)
- moved C29 287.0 mm to (177.1, 131.8), turned to 180 degrees
- moved C32 277.6 mm to (149.9, 167.8), turned to 180 degrees
- moved C30 277.2 mm to (176.6, 111.1), turned to 180 degrees
- moved C27 256.2 mm to (167.7, 131.8), turned to 180 degrees
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Connections:
- net IP0 renamed Net-(U12-R2IN)
- C1 pad 1: +3.3V -> +5V
- C2 pad 1: +3.3V -> +5V
- C28 pad 1: +3.3V -> +5V
- C29 pad 1: +12V -> +5V
- C38 pad 1: +5V -> +12V
- C41 pad 1: +5V -> +12V
- C6 pad 1: +3.3V -> +5V
- C7 pad 1: +3.3V -> +5V
- D1 pad 1: GND -> Net-(D1-K)
- D1 pad 2: Net-(D1-A) -> GND
- D2 pad 1: Net-(D2-K) -> GND
- D2 pad 2: GND -> Net-(D2-A)
- D3 pad 1: GND -> /RESET
- D4 pad 1: /RESET -> unconnected-(D4-K-Pad1)
- J1 pad 1: +3.3V -> TCK
- J1 pad 2: Net-(J1-Pin_2) -> GND
- J1 pad 3: GND -> TDO
- J10 pad 1: +3.3V -> GND
- J10 pad 2: GND -> /RTSB
- J10 pad 3: +3.3V -> unconnected-(J10-Pin_3-Pad3)
- J10 pad 4: GND -> RXB
- J10 pad 5: +3.3V -> TXB
- J10 pad 6: GND -> unconnected-(J10-Pin_6-Pad6)
- J2 pad 1: Net-(J2-Pin_1) -> TCK_DRAM
- J2 pad 2: Net-(J2-Pin_2) -> GND
- J2 pad 3: Net-(J2-Pin_3) -> TDO_DRAM
- J2 pad 4: Net-(J2-Pin_4) -> +5V
- J2 pad 5: Net-(J2-Pin_5) -> TMS_DRAM
- J2 pad 6: +3.3V -> unconnected-(J2-Pin_6-Pad6)
- J2 pad 7: GND -> unconnected-(J2-Pin_7-Pad7)
- J3 pad 1: TCK -> +12V
- J3 pad 3: TDO -> (no net)
- J4 pad 1: GND -> +12V
- J4 pad 2: /RTSA -> GND
- J4 pad 3: unconnected-(J4-Pin_3-Pad3) -> +12V
- J4 pad 4: RXA -> GND
- J4 pad 5: TXA -> +12V
- J4 pad 6: unconnected-(J4-Pin_6-Pad6) -> GND
- J5 pad 1: GND -> +5V
- J5 pad 2: /RTSB -> GND
- J5 pad 3: unconnected-(J5-Pin_3-Pad3) -> +5V
- J5 pad 4: RXB -> GND
- J5 pad 5: TXB -> +5V
- J5 pad 6: unconnected-(J5-Pin_6-Pad6) -> GND
- J6 pad 1: +3.3V -> Net-(J6-Pad1)
- J6 pad 2: +3.3V -> Net-(U12-T1OUT)
- J6 pad 3: +5V -> Net-(U12-R1IN)
- J6 pad 4: +5V -> Net-(J6-Pad1)
- J6 pad 6: GND -> Net-(J6-Pad1)
- J6 pad 8: OP2 -> Net-(U12-T2OUT)
- J6 pad 9: IP1 -> unconnected-(J6-Pad9)
- J7 pad 1: +12V -> Net-(J7-Pad1)
- J7 pad 2: GND -> Net-(U11-R1IN)
- J7 pad 3: (no net) -> Net-(U11-T1OUT)
- J8 pad 1: +12V -> unconnected-(J8-Pin_1-Pad1)
- J8 pad 2: GND -> unconnected-(J8-Pin_2-Pad2)
- J8 pad 3: +12V -> +5V
- J8 pad 4: GND -> +5V
- J8 pad 5: +12V -> GND
- J9 pad 1: +5V -> GND
- J9 pad 2: GND -> /RTSA
- J9 pad 3: +5V -> unconnected-(J9-Pin_3-Pad3)
- J9 pad 4: GND -> RXA
- J9 pad 5: +5V -> TXA
- J9 pad 6: GND -> unconnected-(J9-Pin_6-Pad6)
- L1 pad 1: Net-(D2-K) -> Net-(D1-K)
- R1 pad 1: Net-(U1-~{RESET}/PA0) -> +5V
- R1 pad 2: Net-(J1-Pin_2) -> Net-(U1-/CDIS)
- R10 pad 2: TDO -> TMS_DRAM
- R11 pad 2: TMS -> TDI_DRAM
- R12 pad 1: +5V -> TCK_DRAM
- R12 pad 2: TDI -> GND
- R13 pad 1: TCK -> +5V
- R13 pad 2: GND -> Net-(D2-A)
- R14 pad 2: Net-(U5-/MMUDIS) -> Net-(D3-A)
- R15 pad 1: +5V -> /IRQ_DUART
- R15 pad 2: Net-(U5-/CDIS) -> +5V
- R16 pad 2: /DSACK0 -> /WE_ROM
- R17 pad 2: /DSACK1 -> /OE_ROM
- R18 pad 2: Net-(D3-A) -> Net-(U17-/SIZE)
- R19 pad 2: Net-(D4-A) -> Net-(U17-A0)
- R2 pad 1: Net-(R2-Pad1) -> +5V
- R2 pad 2: CLK_DRAM -> /DSACK1
- R20 pad 1: +5V -> GND
- R20 pad 2: /WE_ROM -> IDE_RDY
- R21 pad 1: +5V -> GND
- R21 pad 2: /OE_ROM -> IDE_INT
- R22 pad 1: /IACK_DUART -> +5V
- R22 pad 2: +5V -> Net-(D4-A)
- R3 pad 1: Net-(R3-Pad1) -> +5V
- R3 pad 2: CLK_CPU -> /DSACK0
- R4 pad 1: Net-(R4-Pad1) -> +5V
- R4 pad 2: CLK_DUART -> Net-(U1-/MMUDIS)
- R5 pad 1: +3.3V -> +5V
- R5 pad 2: Net-(U1-PB0) -> TDO
- R6 pad 1: +3.3V -> +5V
- R6 pad 2: Net-(U1-PB1) -> TMS
- R7 pad 2: /RESET -> TDI
- R8 pad 1: +5V -> TCK
- R8 pad 2: /HALT -> GND
- R9 pad 1: Net-(U1-PA6) -> +5V
- R9 pad 2: Net-(D1-A) -> TDO_DRAM
- SW1 pad 1: GND -> /RESET
- SW1 pad 2: Net-(U1-PA7) -> GND
- U10 pad 1: A18 -> GND
- U10 pad 2: A16 -> /RESET
- U10 pad 3: A14 -> +5V
- U11 pad 1: D2 -> Net-(U11-C1+)
- U11 pad 10: +5V -> /RTSA
- U11 pad 11: CLK_CPU -> TXA
- U11 pad 12: GND -> RXA
- U11 pad 13: /RESET -> Net-(U11-R1IN)
- U11 pad 14: GND -> Net-(U11-T1OUT)
- U11 pad 15: unconnected-(U11-NC-Pad15) -> GND
- U11 pad 2: D1 -> Net-(U11-VS+)
- U11 pad 3: D0 -> Net-(U11-C1-)
- U11 pad 4: GND -> Net-(U11-C2+)
- U11 pad 5: GND -> Net-(U11-C2-)
- U11 pad 6: GND -> Net-(U11-VS-)
- U11 pad 7: GND -> Net-(U11-T2OUT)
- U11 pad 8: GND -> Net-(U11-R2IN)
- U11 pad 9: GND -> /CTSA
- U12 pad 1: unconnected-(U12-NC-Pad1) -> Net-(U12-C1+)
- U12 pad 10: unconnected-(U12-/DTACK-Pad10) -> /RTSB
- U12 pad 11: RXB -> TXB
- U12 pad 12: unconnected-(U12-NC-Pad12) -> RXB
- U12 pad 13: TXB -> Net-(U12-R1IN)
- U12 pad 14: /RTSB -> Net-(U12-T1OUT)
- U12 pad 15: OP3 -> GND
- U12 pad 16: OP5 -> +5V
- U12 pad 2: A1 -> Net-(U12-VS+)
- U12 pad 3: IP3 -> Net-(U12-C1-)
- U12 pad 4: A2 -> Net-(U12-C2+)
- U12 pad 5: IP1 -> Net-(U12-C2-)
- U12 pad 6: A3 -> Net-(U12-VS-)
- U12 pad 7: A4 -> Net-(U12-T2OUT)
- U12 pad 9: R/W -> /CTSB
- U3 pad 10: GND -> unconnected-(U3-IO-Pad10)
- U3 pad 12: GND -> unconnected-(U3-IO-Pad12)
- U3 pad 14: +5V -> TDI_DRAM
- U3 pad 2: Net-(Y1-CLK0) -> GND
- U3 pad 3: Net-(R2-Pad1) -> +5V
- U3 pad 4: GND -> unconnected-(U3-IO-Pad4)
- U3 pad 5: Net-(Y1-CLK1) -> unconnected-(U3-IO-Pad5)
- U3 pad 6: Net-(R3-Pad1) -> unconnected-(U3-IO-Pad6)
- U3 pad 8: Net-(R4-Pad1) -> unconnected-(U3-IO-Pad8)
- U3 pad 9: Net-(Y1-CLK2) -> unconnected-(U3-IO-Pad9)
- U4 pad 1: Net-(U1-PA4) -> GND
- U4 pad 10: unconnected-(U4-Pad10) -> +5V
- U4 pad 11: GND -> unconnected-(U4-NC-Pad11)
- U4 pad 12: unconnected-(U4-Pad12) -> /DRAM/DRAM_A0
- U4 pad 13: GND -> /DRAM/DRAM_A1
- U4 pad 14: +3.3V -> /DRAM/DRAM_A2
- U4 pad 2: /RESET -> /DRAM/SIMM_D0
- U4 pad 3: Net-(U1-PA5) -> /DRAM/SIMM_D16
- U4 pad 4: /HALT -> /DRAM/SIMM_D1
- U4 pad 5: GND -> /DRAM/SIMM_D17
- U4 pad 6: unconnected-(U4-Pad6) -> /DRAM/SIMM_D2
- U4 pad 7: GND -> /DRAM/SIMM_D18
- U4 pad 8: unconnected-(U4-Pad8) -> /DRAM/SIMM_D3
- U4 pad 9: GND -> /DRAM/SIMM_D19
- U6 pad 1: GND -> R/W
- U6 pad 10: unconnected-(U6-IO-Pad10) -> GND
- U6 pad 11: unconnected-(U6-IO-Pad11) -> D8
- U6 pad 12: unconnected-(U6-IO-Pad12) -> D9
- U6 pad 13: +5V -> D10
- U6 pad 14: TDI -> D11
- U6 pad 15: unconnected-(U6-IO-Pad15) -> D12
- U6 pad 16: unconnected-(U6-IO-Pad16) -> D13
- U6 pad 17: unconnected-(U6-IO-Pad17) -> D14
- U6 pad 18: unconnected-(U6-IO-Pad18) -> D15
- U6 pad 19: GND -> /CS_DRAM
- U6 pad 2: unconnected-(U6-OE2/GCLK2-Pad2) -> /DRAM/SIMM_D23
- U6 pad 20: unconnected-(U6-IO-Pad20) -> +5V
- U6 pad 3: +5V -> /DRAM/SIMM_D22
- U6 pad 4: unconnected-(U6-IO-Pad4) -> /DRAM/SIMM_D21
- U6 pad 5: unconnected-(U6-IO-Pad5) -> /DRAM/SIMM_D20
- U6 pad 6: unconnected-(U6-IO-Pad6) -> /DRAM/SIMM_D19
- U6 pad 7: GND -> /DRAM/SIMM_D18
- U6 pad 8: unconnected-(U6-IO-Pad8) -> /DRAM/SIMM_D17
- U6 pad 9: unconnected-(U6-IO-Pad9) -> /DRAM/SIMM_D16
- U7 pad 1: GND -> R/W
- U7 pad 2: +3.3V -> /DRAM/SIMM_D15
- U7 pad 3: +5V -> /DRAM/SIMM_D14
- U8 pad 1: +12V -> R/W
- U8 pad 2: Net-(D2-K) -> /DRAM/SIMM_D7
- U8 pad 3: GND -> /DRAM/SIMM_D6
- U8 pad 4: +5V -> /DRAM/SIMM_D5
- U8 pad 5: GND -> /DRAM/SIMM_D4
- U9 pad 1: A18 -> +12V
- U9 pad 2: A16 -> Net-(D1-K)
- U9 pad 3: A15 -> GND
- U9 pad 4: A12 -> +5V
- U9 pad 5: A7 -> GND
Routing:
- net +5V: track 0.00 -> 105.1 mm, vias 0 -> 4
- net /CS_DRAM: track 0.00 -> 93.7 mm
- net R/W: track 0.00 -> 93.7 mm
- net D0: track 0.00 -> 76.7 mm
- net D1: track 0.00 -> 76.1 mm
- net GND: track 0.00 -> 70.3 mm, vias 0 -> 19
- net D2: track 0.00 -> 69.1 mm
- net D3: track 0.00 -> 69.0 mm
- net D4: track 0.00 -> 62.5 mm
- net D5: track 0.00 -> 62.3 mm
- net /DRAM_WR: track 0.00 -> 56.8 mm
- net /DRAM/DRAM_A11: track 0.00 -> 55.9 mm
- net D6: track 0.00 -> 55.7 mm
- net D30: track 0.00 -> 55.5 mm
- net D31: track 0.00 -> 55.4 mm
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- added copper zone on In1.Cu, net +5V
- added copper zone on In2.Cu, net GND
Other:
- board outline added: 210 x 150 mm
- copper layers 2 -> 4
